Commit message: added a wagon model for testing the vicon system

File: tms_rp/bsen_description/urdf/bsen.urdf (robot description, URDF)
Before this commit: robot environment, 16 links, 15 joints
Links:
- added link wagon; visual mesh filename=package://environmental_model/model/wagon.stl
- link bed: geometry visual mesh filename=package://environmental_model/model/bed.stl
- link drawer: geometry visual mesh filename=package://environmental_model/model/drawer.stl
Joints:
- added joint bsen_room_to_wagon: type fixed, parent bsen_origin, child wagon, origin xyz=0 0 0

Commit message: added joint_state_publisher for control of wagon using vicon data

File: tms_rp/bsen_description/urdf/bsen.urdf (robot description, URDF)
Before this commit: robot environment, 17 links, 16 joints
Links:
- added link wagon_x_link
- added link wagon_y_link
Joints:
- added joint wagon_theta_joint: type continuous, parent wagon_y_link, child wagon, origin xyz=0 0 0 rpy=0 0 -1.57075, axis 0 0 1
- added joint wagon_x_joint: type prismatic, parent origin_position, child wagon_x_link, origin xyz=0 0 0 rpy=0 0 0, limit lower=-5. upper=5. effort=1000.0 velocity=0.5
- added joint wagon_y_joint: type prismatic, parent wagon_x_link, child wagon_y_link, origin xyz=0 0 0 rpy=0 0 1.57075, limit lower=-5. upper=5. effort=1000.0 velocity=0.5

Commit message: added re-position method using vicon pose data

File: tms_rp/bsen_description/urdf/bsen.urdf (robot description, URDF)
Before this commit: robot environment, 19 links, 19 joints
Joints:
- removed joint bsen_room_to_wagon
- joint bsen_origin_joint: origin xyz=4.5 0 0 rpy=0 0 0 -> xyz=0.0 0 0 rpy=0 0 0
- joint wagon_theta_joint: origin xyz=0 0 0 rpy=0 0 -1.57075 -> xyz=0 0 0 rpy=0 0 -1.57079633
- joint wagon_x_joint: limit lower=-5. upper=5. effort=1000.0 velocity=0.5 -> lower=0. upper=15. effort=1000.0 velocity=0.5; parent origin_position -> bsen_origin
- joint wagon_y_joint: limit lower=-5. upper=5. effort=1000.0 velocity=0.5 -> lower=0. upper=7. effort=1000.0 velocity=0.5; origin xyz=0 0 0 rpy=0 0 1.57075 -> xyz=0 0 0 rpy=0 0 1.57079633

Commit message: modified the urdf of bsen for moveable objects

File: tms_rp/bsen_description/urdf/bsen.urdf (robot description, URDF)
Before this commit: robot environment, 19 links, 18 joints
Links:
- removed link origin_position
- added link bsen_celling; visual mesh filename=package://environmental_model/model/bsen_celling.dae
- added link bsen_wall; visual mesh filename=package://environmental_model/model/bsen_wall.dae
- added link carpet; visual mesh filename=package://environmental_model/model/carpet.dae
- added link intelingent_shelf; visual mesh filename=package://environmental_model/model/intelingent_shelf.dae
- added link kitchen; visual mesh filename=package://environmental_model/model/kitchen.dae
- added link recorder; visual mesh filename=package://environmental_model/model/recorder.dae
- added link sofa; visual mesh filename=package://environmental_model/model/sofa.dae
- added link sofa_table; visual mesh filename=package://environmental_model/model/sofa_table.dae
- added link start_position
- added link tv_52; visual mesh filename=package://environmental_model/model/tv_52.dae
- added link tv_multi; visual mesh filename=package://environmental_model/model/tv_multi.dae
- link bed: geometry visual mesh filename=package://environmental_model/model/bed.dae
- link bsen_room: geometry visual mesh filename=package://environmental_model/model/bsen.dae
- link chair: geometry visual mesh filename=package://environmental_model/model/chair.dae
- link drawer: geometry visual mesh filename=package://environmental_model/model/drawer.dae
- link meeting_chair1: geometry visual mesh filename=package://environmental_model/model/meeting_chair.dae
- link meeting_chair2: geometry visual mesh filename=package://environmental_model/model/meeting_chair.dae
- link meeting_chair3: geometry visual mesh filename=package://environmental_model/model/meeting_chair.dae
- link meeting_chair4: geometry visual mesh filename=package://environmental_model/model/meeting_chair.dae
- link meeting_table: geometry visual mesh filename=package://environmental_model/model/meeting_table.dae
- link refrigerator: geometry visual mesh filename=package://environmental_model/model/refrigerator.dae
- link tree: geometry visual mesh filename=package://environmental_model/model/tree.dae
- link tv_table: geometry visual mesh filename=package://environmental_model/model/tv_table.dae
- link wagon: geometry visual mesh filename=package://environmental_model/model/wagon.dae
- link wordrobe: geometry visual mesh filename=package://environmental_model/model/wordrobe.dae
- link workdesk: geometry visual mesh filename=package://environmental_model/model/work_desk.dae
Joints:
- added joint bsen_room_to_carpet: type fixed, parent bsen_origin, child carpet, origin xyz=0 0 0
- added joint bsen_room_to_celling: type fixed, parent bsen_room, child bsen_celling, origin xyz=0 0 0
- added joint bsen_room_to_intelingent_shelf: type fixed, parent bsen_origin, child intelingent_shelf, origin xyz=0 0 0
- added joint bsen_room_to_kitchen: type fixed, parent bsen_origin, child kitchen, origin xyz=0 0 0
- added joint bsen_room_to_recorder: type fixed, parent bsen_origin, child recorder, origin xyz=0 0 0
- added joint bsen_room_to_sofa: type fixed, parent bsen_origin, child sofa, origin xyz=0 0 0
- added joint bsen_room_to_sofa_table: type fixed, parent bsen_origin, child sofa_table, origin xyz=0 0 0
- added joint bsen_room_to_tv_52: type fixed, parent bsen_origin, child tv_52, origin xyz=0 0 0
- added joint bsen_room_to_tv_multi: type fixed, parent bsen_origin, child tv_multi, origin xyz=0 0 0
- added joint bsen_room_to_wagon: type fixed, parent bsen_origin, child wagon, origin xyz=0 0 0
- added joint bsen_room_to_wall: type fixed, parent bsen_room, child bsen_wall, origin xyz=0 0 0
- joint bsen_origin_joint: origin xyz=0.0 0 0 rpy=0 0 0 -> xyz=4.5 0 0 rpy=0 0 0
- joint world_joint: parent origin_position -> start_position

Commit message: added tms_db_state_publisher node for moving the object in RViz

File: tms_rp/bsen_description/urdf/bsen.urdf (robot description, URDF)
Before this commit: robot environment, 29 links, 29 joints
Joints:
- removed joint bsen_room_to_wagon
- joint wagon_theta_joint: origin xyz=0 0 0 rpy=0 0 -1.57079633 -> xyz=0 0 0 rpy=0 0 0
- joint wagon_x_joint: parent bsen_origin -> start_position
