Commit message: added environment_gazebo package for simulation in Gazebo

File: tms_rp/environment_description/urdf/environment.xacro (robot description, xacro)
@@ -1,36 +1,16 @@
 <?xml version="1.0"?>
-<robot name="environment">
-  <!-- ========== basic link ========== -->
-  <link name="start_position"/>
-<!--   <joint name="world_x_joint" type="prismatic">
-    <parent link="origin_position"/>
-    <child link="world_x_link"/>
-    <origin xyz="0 0 0" rpy="0 0 0"/>
-    <limit effort="1000.0" lower="-5." upper="5." velocity="0.5"/>
-  </joint>
-  <link name="world_x_link"/>
-  <joint name="world_y_joint" type="prismatic">
-    <parent link="world_x_link"/>
-    <child link="world_y_link"/>
-    <origin xyz="0 0 0" rpy="0 0 0"/>
-    <limit effort="1000.0" lower="-5." upper="5." velocity="0.5"/>
-  </joint>
-  <link name="world_y_link"/>
-  <joint name="world_theta_joint" type="continuous">
-    <parent link="world_y_link"/>
-    <child link="base_footprint"/>
-    <origin xyz="0 0 0" rpy="0 0 0"/>
-    <axis xyz="0 0 1"/>
-  </joint>
-  <link name="base_footprint"/> -->
-<!--   <joint name="base_footprint_joint" type="fixed">
-    <parent link="base_footprint"/>
-    <child link="base_link"/>
-    <origin xyz="0 0 0" rpy="0 0 0"/>
-  </joint> -->
-  <!-- ========== robots ========== -->
-  <!-- ========== environment ========== -->
+<!-- Environment of B-Sen Project room -->
+<robot name="environment" xmlns:xacro="http://www.ros.org/wiki/xacro">
+  <!-- Constants for robot dimensions -->
+  <xacro:property name="PI" value="3.1415926535897931"/>
+  <!-- Import all Gazebo-customization elements, including Gazebo colors -->
+  <xacro:include filename="$(find environment_description)/urdf/environment.gazebo" />
+  <!-- Import Rviz colors -->
+  <xacro:include filename="$(find environment_description)/urdf/materials.xacro" />
+  <!-- Used for fixing robot to Gazebo 'base_link' -->
+  <link name="world"/>
+  <!--  Environment -->
   <joint name="world_joint" type="fixed">
-    <parent link="start_position"/>
+    <parent link="world"/>
     <child link="bsen_room"/>
     <origin xyz="0 0 0" rpy="0 0 0"/>
@@ -43,4 +23,12 @@
       <origin xyz="0 0 0" rpy="0 0 0"/>
     </visual>
+    <inertial>
+      <origin xyz="0 0 0" rpy="0 0 0"/>
+      <mass value="1"/>
+      <inertia
+        ixx="1.0" ixy="0.0" ixz="0.0"
+        iyy="1.0" iyz="0.0"
+        izz="1.0"/>
+    </inertial>
   </link>
   <joint name="bsen_origin_joint" type="fixed">
@@ -372,5 +360,5 @@
   <link name="wagon_x_link"/>
   <joint name="wagon_x_joint" type="prismatic">
-    <parent link="start_position"/>
+    <parent link="world"/>
     <child link="wagon_x_link"/>
     <origin xyz="0 0 0" rpy="0 0 0"/>
@@ -391,4 +379,2 @@
   </joint>
 </robot>
-<!-- 90  degree to radian 1.57079633 -->
-<!-- 180 degree to radian 3.14159265 -->

Commit message: modifed the description source of B-Sen room

File: tms_rp/environment_description/urdf/environment.xacro (robot description, xacro)
@@ -21,8 +21,8 @@
         <mesh filename="package://environmental_model/model/bsen.dae"/>
       </geometry>
-      <origin xyz="0 0 0" rpy="0 0 0"/>
+      <origin xyz="0 0 0.001" rpy="0 0 0"/>
     </visual>
     <inertial>
-      <origin xyz="0 0 0" rpy="0 0 0"/>
+      <origin xyz="0 0 0.001" rpy="0 0 0"/>
       <mass value="1"/>
       <inertia

Commit message: added viewer for dynamic map using voronoi map

File: tms_rp/environment_description/urdf/environment.xacro (robot description, xacro)
@@ -349,5 +349,5 @@
     <origin xyz="0 0 0"/>
   </joint> -->
-  <link name="wagon">
+<!--   <link name="wagon">
     <visual>
       <geometry>
@@ -356,7 +356,7 @@
       <origin xyz="0. 0. 0.5" rpy="0 0 1.57079633"/>
     </visual>
-  </link>
+  </link> -->
   <!-- ========== Movable object ========== -->
-  <link name="wagon_x_link"/>
+<!--   <link name="wagon_x_link"/>
   <joint name="wagon_x_joint" type="prismatic">
     <parent link="world"/>
@@ -377,4 +377,4 @@
     <origin xyz="0 0 0" rpy="0 0 0"/>
     <axis xyz="0 0 1"/>
-  </joint>
+  </joint> -->
 </robot>

Commit message: modified the urdf files related environment of rostms

File: tms_rp/environment_description/urdf/environment.xacro (robot description, xacro)
@@ -1,11 +1,9 @@
 <?xml version="1.0"?>
 <!-- Environment of B-Sen Project room -->
-<robot name="environment" xmlns:xacro="http://www.ros.org/wiki/xacro">
-  <!-- Constants for robot dimensions -->
-  <xacro:property name="PI" value="3.1415926535897931"/>
+<robot name="rostms" xmlns:xacro="http://www.ros.org/wiki/xacro">
+  <!-- Import common properties -->
+  <xacro:include filename="$(find environment_description)/urdf/common_properties.urdf.xacro" />
   <!-- Import all Gazebo-customization elements, including Gazebo colors -->
   <xacro:include filename="$(find environment_description)/urdf/environment.gazebo" />
-  <!-- Import Rviz colors -->
-  <xacro:include filename="$(find environment_description)/urdf/materials.xacro" />
   <!-- Used for fixing robot to Gazebo 'base_link' -->
   <link name="world"/>

Commit message: change model position kitchen & workdesk & wordrobe

File: tms_rp/environment_description/urdf/environment.xacro (robot description, xacro)
@@ -81,5 +81,5 @@
         <mesh filename="package://environmental_model/model/kitchen.dae"/>
       </geometry>
-      <origin xyz="4.66 5.9 0.4855" rpy="0 0 -1.57079633"/>
+      <origin xyz="4.76 5.9 0.4855" rpy="0 0 -1.57079633"/>
     </visual>
   </link>
@@ -302,5 +302,5 @@
         <mesh filename="package://environmental_model/model/wordrobe.dae"/>
       </geometry>
-      <origin xyz="9.1 5.8 1.3" rpy="0 0 -1.57079633"/>
+      <origin xyz="9.2 5.9 1.3" rpy="0 0 -1.57079633"/>
     </visual>
   </link>
@@ -315,5 +315,5 @@
         <mesh filename="package://environmental_model/model/work_desk.dae"/>
       </geometry>
-      <origin xyz="7.43 5.9 0.5" rpy="0 0 -1.57079633"/>
+      <origin xyz="7.55 5.9 0.5" rpy="0 0 -1.57079633"/>
     </visual>
   </link>
