Commit message: added standalone type of smartpal5

File: tms_rp/smartpal5_description/urdf/smartpal5_standalone.urdf.xacro (robot description, xacro)
@@ -1,7 +1,12 @@
 <?xml version="1.0"?>
-<robot name="smartpal5_standalone" xmlns:xacro="http://www.ros.org/wiki/xacro">
+<robot name="smartpal5" xmlns:xacro="http://www.ros.org/wiki/xacro">
   <!-- Used for fixing all components to 'world' frame of RViz and Gazebo 'world' -->
-  <link name="world"/>
+  <link name="world_link"/>
+  <joint name="world_smartpal5_joint" type="fixed">
+	  <parent link="world_link"/>
+    <child link="smartpal5_link"/>
+    <origin xyz="0 0 0" rpy="0 0 0"/>
+  </joint>
   <!-- Defines the components tags -->
-  <xacro:include filename="$(find rostms_description)/urdf/smartpal5.urdf.xacro" />
+  <xacro:include filename="$(find smartpal5_description)/urdf/smartpal5.urdf.xacro" />
 </robot>
