Commit message: added right_end_effector_joint and left_end_effector_joint into URDF file of smartpal

File: tms_rp/smartpal5_description/urdf/smartpal5.urdf.xacro (robot description, xacro)
@@ -358,4 +358,23 @@
 		</inertial>
 	</link>
+  <joint name="left_end_effector_joint" type="fixed">
+    <origin xyz="0.05 0 0" rpy="-0 0 0"/>
+    <parent link="leftGripper_link"/>
+    <child link="left_end_effector_link"/>
+  </joint>
+  <link name="left_end_effector_link">
+    <visual>
+      <origin rpy="0 0 0" xyz="0 0 0"/>
+      <geometry>
+        <box size="0.001 0.001 0.001"/>
+      </geometry>
+    </visual>
+    <collision>
+      <origin rpy="0 0 0" xyz="0 0 0"/>
+      <geometry>
+        <box size="0.001 0.001 0.001"/>
+      </geometry>
+    </collision>
+  </link>
 	<joint name="leftGripper__leftGripper_thumb_joint" type="revolute">
 		<parent link="leftGripper_link"/>

Commit message: modified the joints and links

File: tms_rp/smartpal5_description/urdf/smartpal5.urdf.xacro (robot description, xacro)
@@ -1,12 +1,11 @@
 <?xml version="1.0"?>
-<!-- SmartPal5 -->
 <robot name="smartpal5" xmlns:xacro="http://www.ros.org/wiki/xacro">
-	<!-- ==================== Planar joint ==================== -->
-    <joint name="world_x_joint" type="prismatic">
-        <parent link="world"/>
-        <child link="world_x_link"/>
-        <origin xyz="0 0 0" rpy="0 0 0"/>
-        <limit effort="1000.0" lower="-5." upper="5." velocity="0.5"/>
-    </joint>
+	<!-- Vehicle -->
+  <joint name="world_x_joint" type="prismatic">
+		<parent link="world"/>
+    <child link="world_x_link"/>
+    <origin xyz="0 0 0" rpy="0 0 0"/>
+    <limit effort="1000.0" lower="-5." upper="5." velocity="0.5"/>
+  </joint>
     <link name="world_x_link"/>
     <joint name="world_y_joint" type="prismatic">
@@ -29,6 +28,5 @@
 		<origin xyz="0 0 0" rpy="0 0 0"/>
 	</joint>
-	<!-- ==================== Vehicle ==================== -->
-	<link name="base_link"> <!-- Vehicle -->
+	<link name="base_link">
 		<visual>
 			<geometry>

Commit message: modified the composition of joints and links

File: tms_rp/smartpal5_description/urdf/smartpal5.urdf.xacro (robot description, xacro)
@@ -1,29 +1,30 @@
 <?xml version="1.0"?>
 <robot name="smartpal5" xmlns:xacro="http://www.ros.org/wiki/xacro">
-	<!-- Vehicle -->
-  <joint name="world_x_joint" type="prismatic">
-		<parent link="world"/>
-    <child link="world_x_link"/>
+	<!-- Base, Vehicle -->
+  <link name="smartpal5_link"/>
+  <joint name="smartpal5_x_joint" type="prismatic">
+	  <parent link="smartpal5_link"/>
+    <child link="smartpal5_x_link"/>
     <origin xyz="0 0 0" rpy="0 0 0"/>
     <limit effort="1000.0" lower="-5." upper="5." velocity="0.5"/>
   </joint>
-    <link name="world_x_link"/>
-    <joint name="world_y_joint" type="prismatic">
-		<parent link="world_x_link"/>
-		<child link="world_y_link"/>
-		<origin xyz="0 0 0" rpy="0 0 1.57075"/>
-        <limit effort="1000.0" lower="-5." upper="5." velocity="0.5"/>
-    </joint>
-    <link name="world_y_link"/>
-    <joint name="world_theta_joint" type="continuous">
-		<parent link="world_y_link"/>
+  <link name="smartpal5_x_link"/>
+  <joint name="smartpal5_y_joint" type="prismatic">
+    <parent link="smartpal5_x_link"/>
+    <child link="smartpal5_y_link"/>
+    <origin xyz="0 0 0" rpy="0 0 1.57075"/>
+    <limit effort="1000.0" lower="-5." upper="5." velocity="0.5"/>
+  </joint>
+  <link name="smartpal5_y_link"/>
+  <joint name="smartpal5_yaw_joint" type="continuous">
+	  <parent link="smartpal5_y_link"/>
 		<child link="base_footprint"/>
 		<origin xyz="0 0 0" rpy="0 0 -1.57075"/>
-        <axis xyz="0 0 1"/>
-	</joint>
-    <link name="base_footprint"/>
+    <axis xyz="0 0 1"/>
+	</joint>
+  <link name="base_footprint"/>
 	<joint name="base_footprint_joint" type="fixed">
-        <parent link="base_footprint"/>
-		<child link="base_link"/>
+    <parent link="base_footprint"/>
+	  <child link="base_link"/>
 		<origin xyz="0 0 0" rpy="0 0 0"/>
 	</joint>
@@ -48,14 +49,13 @@
 		</inertial>
 	</link>
-	<!-- ==================== Vehicle - Lumbar Joint ==================== -->
-	<joint name="vehicle__lumbar_j1_joint" type="revolute">
-		<parent link="base_link"/> <!-- Vehicle -->
-		<child link="lumbar_j1_link"/>
+	<!-- Lumbar -->
+	<joint name="lumbar_lower_joint" type="revolute">
+	  <parent link="base_link"/>
+		<child link="lumbar_lower_link"/>
 		<origin xyz="0 0 0.4365" rpy="-1.57075 0 0"/>
 		<axis xyz="0 0 1"/>
 		<limit lower="-0.2" upper="0.00872664625997165" effort="100.0" velocity="1.0"/>
 	</joint>
-	<!-- ==================== Lumbar ==================== -->
-	<link name="lumbar_j1_link">
+	<link name="lumbar_lower_link">
 		<visual>
 			<geometry>
@@ -77,12 +77,12 @@
 		</inertial>
 	</link>
-	<joint name="lumbar_j1__lumbar_j2_joint" type="revolute">
-		<parent link="lumbar_j1_link"/>
-		<child link="lumbar_j2_link"/>
+	<joint name="lumbar_upper_joint" type="revolute">
+		<parent link="lumbar_lower_link"/>
+		<child link="lumbar_upper_link"/>
 		<origin xyz="0 -0.21 0" rpy="0 0 0"/>
 		<axis xyz="0 0 1"/>
 		<limit lower="-0.00872664625997165" upper="2.10312174865317" effort="100.0" velocity="1.0"/>
 	</joint>
-	<link name="lumbar_j2_link">
+	<link name="lumbar_upper_link">
 		<visual>
 			<geometry>
@@ -104,13 +104,12 @@
 		</inertial>
 	</link>
-    <!-- ==================== Lumbar - RGBD Camera Joint ==================== -->
-    <joint name="lumbar_j2__head_camera_joint" type="fixed">
-		<parent link="lumbar_j2_link"/>
+  <!-- RGB-D Camera -->
+  <joint name="head_camera_joint" type="fixed">
+		<parent link="lumbar_upper_link"/>
 		<child link="camera_link"/>
 		<origin xyz="0.02 -0.7 0" rpy="1.57075 0 0"/>
 	</joint>
-    <!-- ==================== RGBD Camera ==================== -->
-    <link name="camera_link">
-		<visual>
+  <link name="camera_link">
+	  <visual>
 			<geometry>
 				<box size="0.03 0.15 0.05"/>
@@ -131,20 +130,13 @@
 		</inertial>
 	</link>
-    <!--joint name="camera_orientation" type="fixed">
-        <parent link="camera_link"/>
-        <child link="camera_oriented_link"/>
-		<origin xyz="0 0 0" rpy="0 -1.57075 0"/>
-    </joint>
-    <link name="camera_oriented_link"/-->
-	<!-- ==================== Lumbar - Left Arm Joint ==================== -->
-	<joint name="lumbar_j2__leftArm_j1_joint" type="revolute">
-		<parent link="lumbar_j2_link"/>
-		<child link="leftArm_j1_link"/>
+	<!-- Left Arm -->
+  <joint name="l_arm_j1_joint" type="revolute">
+		<parent link="lumbar_upper_link"/>
+		<child link="l_arm_j1_link"/>
 		<origin xyz="-0.025 -0.480 0.200" rpy="3.14159 0 0"/>
 		<axis xyz="0 0 1"/>
 		<limit lower="-0.7679" upper="3.1066" effort="100.0" velocity="1.0"/>
 	</joint>
-	<!-- ==================== Left Arm ==================== -->
-	<link name="leftArm_j1_link">
+	<link name="l_arm_j1_link">
 		<visual>
 			<geometry>
@@ -166,12 +158,12 @@
 		</inertial>
 	</link>
-	<joint name="leftArm_j1__leftArm_j2_joint" type="revolute">
-		<parent link="leftArm_j1_link"/>
-		<child link="leftArm_j2_link"/>
+	<joint name="l_arm_j2_joint" type="revolute">
+		<parent link="l_arm_j1_link"/>
+		<child link="l_arm_j2_link"/>
 		<origin xyz="0 0 0" rpy="1.57075 3.14159 1.57075"/>
 		<axis xyz="0 0 1"/>
 		<limit lower="-0.2443" upper="1.9024" effort="100.0" velocity="1.0"/>
 	</joint>
-	<link name="leftArm_j2_link">
+	<link name="l_arm_j2_link">
 		<visual>
 			<geometry>
@@ -193,12 +185,12 @@
 		</inertial>
 	</link>
-	<joint name="leftArm_j2__leftArm_j3_joint" type="revolute">
-		<parent link="leftArm_j2_link"/>
-		<child link="leftArm_j3_link"/>
+	<joint name="l_arm_j3_joint" type="revolute">
+		<parent link="l_arm_j2_link"/>
+		<child link="l_arm_j3_link"/>
 		<origin xyz="0 0 0" rpy="1.57075 1.57075 1.57075"/>
 		<axis xyz="0 0 1"/>
 		<limit lower="-2.0769" upper="2.0769" effort="100.0" velocity="1.0"/>
 	</joint>
-	<link name="leftArm_j3_link">
+	<link name="l_arm_j3_link">
 		<visual>
 			<geometry>
@@ -220,12 +212,12 @@
 		</inertial>
 	</link>
-	<joint name="leftArm_j3__leftArm_j4_joint" type="revolute">
-		<parent link="leftArm_j3_link"/>
-		<child link="leftArm_j4_link"/>
+	<joint name="l_arm_j4_joint" type="revolute">
+		<parent link="l_arm_j3_link"/>
+		<child link="l_arm_j4_link"/>
 		<origin xyz="-0.02 0.0 0.25" rpy="-1.57075 0 3.14159"/>
 		<axis xyz="0 0 1"/>
 		<limit lower="-0.0174" upper="2.2514" effort="100.0" velocity="1.0"/>
 	</joint>
-	<link name="leftArm_j4_link">
+	<link name="l_arm_j4_link">
 		<visual>
 			<geometry>
@@ -247,12 +239,12 @@
 		</inertial>
 	</link>
-	<joint name="leftArm_j4__leftArm_j5_joint" type="revolute">
-		<parent link="leftArm_j4_link"/>
-		<child link="leftArm_j5_link"/>
+	<joint name="l_arm_j5_joint" type="revolute">
+		<parent link="l_arm_j4_link"/>
+		<child link="l_arm_j5_link"/>
 		<origin xyz="-0.02 0.0 0.0" rpy="1.57075 0 0"/>
 		<axis xyz="0 0 1"/>
 		<limit lower="-2.0769" upper="2.0769" effort="100.0" velocity="1.0"/>
 	</joint>
-	<link name="leftArm_j5_link">
+	<link name="l_arm_j5_link">
 		<visual>
 			<geometry>
@@ -274,12 +266,12 @@
 		</inertial>
 	</link>
-	<joint name="leftArm_j5__leftArm_j6_joint" type="revolute">
-		<parent link="leftArm_j5_link"/>
-		<child link="leftArm_j6_link"/>
+	<joint name="l_arm_j6_joint" type="revolute">
+		<parent link="l_arm_j5_link"/>
+		<child link="l_arm_j6_link"/>
 		<origin xyz="0.0 0.0 0.28" rpy="-1.57075 1.57075 0"/>
 		<axis xyz="0 0 1"/>
 		<limit lower="-0.2617" upper="0.7504" effort="100.0" velocity="1.0"/>
 	</joint>
-	<link name="leftArm_j6_link">
+	<link name="l_arm_j6_link">
 		<visual>
 			<geometry>
@@ -301,12 +293,12 @@
 		</inertial>
 	</link>
-	<joint name="leftArm_j6__leftArm_j7_joint" type="revolute">
-		<parent link="leftArm_j6_link"/>
-		<child link="leftArm_j7_link"/>
+	<joint name="l_arm_j7_joint" type="revolute">
+		<parent link="l_arm_j6_link"/>
+		<child link="l_arm_j7_link"/>
 		<origin xyz="0.0 0.0 0" rpy="1.57075 3.14159 0"/>
 		<axis xyz="0 0 1"/>
 		<limit lower="0" upper="0.5" effort="100.0" velocity="1.0"/>
 	</joint>
-	<link name="leftArm_j7_link">
+	<link name="l_arm_j7_link">
 		<visual>
 			<geometry>
@@ -328,13 +320,12 @@
 		</inertial>
 	</link>
-	<!-- ==================== Left Arm - Left Gripper Joint ==================== -->
-	<joint name="leftArm_j7__leftGripper_joint" type="fixed">
-		<parent link="leftArm_j7_link"/>
-		<child link="leftGripper_link"/>
+	<!-- Left Gripper -->
+	<joint name="l_gripper_joint" type="fixed">
+		<parent link="l_arm_j7_link"/>
+		<child link="l_gripper_link"/>
 		<origin xyz="0.056 0 0" rpy="3.14159 3.14159 1.57075"/>
 		<axis xyz="0 0 1"/>
 	</joint>
-	<!-- ==================== Left Gripper ==================== -->
-	<link name="leftGripper_link">
+	<link name="l_gripper_link">
 		<visual>
 			<geometry>
@@ -356,10 +347,10 @@
 		</inertial>
 	</link>
-  <joint name="left_end_effector_joint" type="fixed">
-    <origin xyz="0.05 0 0" rpy="-0 0 0"/>
-    <parent link="leftGripper_link"/>
-    <child link="left_end_effector_link"/>
+  <joint name="l_end_effector_joint" type="fixed">
+    <origin xyz="0.05 0 0" rpy="0 0 0"/>
+    <parent link="l_gripper_link"/>
+    <child link="l_end_effector_link"/>
   </joint>
-  <link name="left_end_effector_link">
+  <link name="l_end_effector_link">
     <visual>
       <origin rpy="0 0 0" xyz="0 0 0"/>
@@ -375,12 +366,12 @@
     </collision>
   </link>
-	<joint name="leftGripper__leftGripper_thumb_joint" type="revolute">
-		<parent link="leftGripper_link"/>
-		<child link="leftGripper_thumb_link"/>
+	<joint name="l_gripper_thumb_joint" type="revolute">
+		<parent link="l_gripper_link"/>
+		<child link="l_gripper_thumb_link"/>
 		<origin xyz="0.027 0.042 0.0" rpy="0 0 0"/>
 		<axis xyz="0 0 1"/>
 		<limit lower="-1.0122" upper="0.1396" effort="100.0" velocity="1.0"/>
 	</joint>
-	<link name="leftGripper_thumb_link">
+	<link name="l_gripper_thumb_link">
 		<visual>
 			<geometry>
@@ -402,14 +393,13 @@
 		</inertial>
 	</link>
-	<!-- ==================== Lumbar - Right Arm Joint ==================== -->
-	<joint name="lumbar_j2__rightArm_j1_joint" type="revolute">
-		<parent link="lumbar_j2_link"/>
-		<child link="rightArm_j1_link"/>
+	<!-- Right Arm -->
+	<joint name="r_arm_j1_joint" type="revolute">
+		<parent link="lumbar_upper_link"/>
+		<child link="r_arm_j1_link"/>
 		<origin xyz="-0.025 -0.480 -0.200" rpy="3.14159 0 0"/>
 		<axis xyz="0 0 1"/>
 		<limit lower="-0.7679" upper="3.1066" effort="100.0" velocity="1.0"/>
 	</joint>
-	<!-- ==================== Right Arm ==================== -->
-	<link name="rightArm_j1_link">
+	<link name="r_arm_j1_link">
 		<visual>
 			<geometry>
@@ -431,12 +421,12 @@
 		</inertial>
 	</link>
-	<joint name="rightArm_j1__rightArm_j2_joint" type="revolute">
-		<parent link="rightArm_j1_link"/>
-		<child link="rightArm_j2_link"/>
+	<joint name="r_armj2_joint" type="revolute">
+		<parent link="r_arm_j1_link"/>
+		<child link="r_arm_j2_link"/>
 		<origin xyz="0 0 0" rpy="-1.57075 0 -1.57075"/>
 		<axis xyz="0 0 1"/>
 		<limit lower="-1.9024" upper="0.2443" effort="100.0" velocity="1.0"/>
 	</joint>
-	<link name="rightArm_j2_link">
+	<link name="r_arm_j2_link">
 		<visual>
 			<geometry>
@@ -458,12 +448,12 @@
 		</inertial>
 	</link>
-	<joint name="rightArm_j2__rightArm_j3_joint" type="revolute">
-		<parent link="rightArm_j2_link"/>
-		<child link="rightArm_j3_link"/>
+	<joint name="r_arm_j3_joint" type="revolute">
+		<parent link="r_arm_j2_link"/>
+		<child link="r_arm_j3_link"/>
 		<origin xyz="0 0 0" rpy="1.57075 1.57075 1.57075"/>
 		<axis xyz="0 0 1"/>
 		<limit lower="-2.0769" upper="2.0769" effort="100.0" velocity="1.0"/>
 	</joint>
-	<link name="rightArm_j3_link">
+	<link name="r_arm_j3_link">
 		<visual>
 			<geometry>
@@ -485,12 +475,12 @@
 		</inertial>
 	</link>
-	<joint name="rightArm_j3__rightArm_j4_joint" type="revolute">
-		<parent link="rightArm_j3_link"/>
-		<child link="rightArm_j4_link"/>
+	<joint name="r_arm_j4_joint" type="revolute">
+		<parent link="r_arm_j3_link"/>
+		<child link="r_arm_j4_link"/>
 		<origin xyz="-0.02 0.0 0.25" rpy="-1.57075 0 3.14159"/>
 		<axis xyz="0 0 1"/>
 		<limit lower="-0.0174" upper="2.2514" effort="100.0" velocity="1.0"/>
 	</joint>
-	<link name="rightArm_j4_link">
+	<link name="r_arm_j4_link">
 		<visual>
 			<geometry>
@@ -512,12 +502,12 @@
 		</inertial>
 	</link>
-	<joint name="rightArm_j4__rightArm_j5_joint" type="revolute">
-		<parent link="rightArm_j4_link"/>
-		<child link="rightArm_j5_link"/>
+	<joint name="r_arm_j5_joint" type="revolute">
+		<parent link="r_arm_j4_link"/>
+		<child link="r_arm_j5_link"/>
 		<origin xyz="-0.02 0.0 0.0" rpy="1.57075 0 0"/>
 		<axis xyz="0 0 1"/>
 		<limit lower="-2.0769" upper="2.0769" effort="100.0" velocity="1.0"/>
 	</joint>
-	<link name="rightArm_j5_link">
+	<link name="r_arm_j5_link">
 		<visual>
 			<geometry>
@@ -539,12 +529,12 @@
 		</inertial>
 	</link>
-	<joint name="rightArm_j5__rightArm_j6_joint" type="revolute">
-		<parent link="rightArm_j5_link"/>
-		<child link="rightArm_j6_link"/>
+	<joint name="r_arm_j6_joint" type="revolute">
+		<parent link="r_arm_j5_link"/>
+		<child link="r_arm_j6_link"/>
 		<origin xyz="0.0 0.0 0.28" rpy="-1.57075 1.57075 0"/>
 		<axis xyz="0 0 1"/>
 		<limit lower="-0.2617" upper="0.7504" effort="100.0" velocity="1.0"/>
 	</joint>
-	<link name="rightArm_j6_link">
+	<link name="r_arm_j6_link">
 		<visual>
 			<geometry>
@@ -566,12 +556,12 @@
 		</inertial>
 	</link>
-	<joint name="rightArm_j6__rightArm_j7_joint" type="revolute">
-		<parent link="rightArm_j6_link"/>
-		<child link="rightArm_j7_link"/>
+	<joint name="r_arm_j7_joint" type="revolute">
+		<parent link="r_arm_j6_link"/>
+		<child link="r_arm_j7_link"/>
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
Commit message: chaged the position of end effectors

File: tms_rp/smartpal5_description/urdf/smartpal5.urdf.xacro (robot description, xacro)
@@ -348,5 +348,5 @@
 	</link>
   <joint name="l_end_effector_joint" type="fixed">
-    <origin xyz="0.05 0 0" rpy="0 0 0"/>
+    <origin xyz="0.01 0.11 0" rpy="0 0 0"/>
     <parent link="l_gripper_link"/>
     <child link="l_end_effector_link"/>
@@ -611,5 +611,5 @@
 	</link>
   <joint name="r_end_effector_joint" type="fixed">
-    <origin xyz="0 0.05 0" rpy="0 0 0"/>
+    <origin xyz="0.11 0.01 0" rpy="0 0 0"/>
     <parent link="r_gripper_link"/>
     <child link="r_end_effector_link"/>
