Commit message: modify the setting of world joint in accordance with the description package of ROS-TMS's environment

File: tms_rp/smartpal5_description/urdf/smartpal5.urdf (robot description, URDF)
Before this commit: robot ros-tms, 68 links, 67 joints
Links:
- removed link bed_link
- removed link bsen_celling_link
- removed link bsen_room_link
- removed link bsen_wall_link
- removed link carpet_link
- removed link chair
- removed link chair_x_link
- removed link chair_y_link
- removed link drawer_link
- removed link intelingent_shelf_link
- removed link kitchen_link
- removed link meeting_chair1
- removed link meeting_chair1_x_link
- removed link meeting_chair1_y_link
- removed link meeting_chair2
- removed link meeting_chair2_x_link
- removed link meeting_chair2_y_link
- removed link meeting_chair3
- removed link meeting_chair3_x_link
- removed link meeting_chair3_y_link
- removed link meeting_chair4
- removed link meeting_chair4_x_link
- removed link meeting_chair4_y_link
- removed link meeting_table_link
- removed link recorder_link
- removed link refrigerator
- removed link refrigerator_x_link
- removed link refrigerator_y_link
- removed link sofa_link
- removed link sofa_table_link
- removed link tree_link
- removed link tv_52_link
- removed link tv_multi_link
- removed link tv_table_link
- removed link wagon
- removed link wagon_x_link
- removed link wagon_y_link
- removed link wardrobe_link
- removed link workdesk_link
- removed link world_link
Joints:
- removed joint bed_joint
- removed joint carpet_joint
- removed joint celling_joint
- removed joint chair_x_joint
- removed joint chair_y_joint
- removed joint chair_yaw_joint
- removed joint drawer_joint
- removed joint intelingent_shelf_joint
- removed joint kitchen_joint
- removed joint meeting_chair1_x_joint
- removed joint meeting_chair1_y_joint
- removed joint meeting_chair1_yaw_joint
- removed joint meeting_chair2_x_joint
- removed joint meeting_chair2_y_joint
- removed joint meeting_chair2_yaw_joint
- removed joint meeting_chair3_x_joint
- removed joint meeting_chair3_y_joint
- removed joint meeting_chair3_yaw_joint
- removed joint meeting_chair4_x_joint
- removed joint meeting_chair4_y_joint
- removed joint meeting_chair4_yaw_joint
- removed joint meeting_table_joint
- removed joint r_arm_j2_joint
- removed joint recorder_joint
- removed joint refrigerator_x_joint
- removed joint refrigerator_y_joint
- removed joint refrigerator_yaw_joint
- removed joint sofa_joint
- removed joint sofa_table_joint
- removed joint tree_link
- removed joint tv_52_link
- removed joint tv_multi_joint
- removed joint tv_table_joint
- removed joint wagon_x_joint
- removed joint wagon_y_joint
- removed joint wagon_yaw_joint
- removed joint wall_joint
- removed joint wardrobe_joint
- removed joint workdesk_joint
- removed joint world_bsen_room_joint
- removed joint world_smartpal5_joint
- added joint r_armj2_joint: type revolute, parent r_arm_j1_link, child r_arm_j2_link, origin xyz=0 0 0 rpy=-1.57075 0 -1.57075, axis 0 0 1, limit lower=-1.9024 upper=0.2443 effort=100.0 velocity=1.0

File: tms_rp/smartpal5_description/urdf/smartpal5.urdf.xacro (robot description, xacro)
@@ -421,5 +421,5 @@
 		</inertial>
 	</link>
-	<joint name="r_armj2_joint" type="revolute">
+	<joint name="r_arm_j2_joint" type="revolute">
 		<parent link="r_arm_j1_link"/>
 		<child link="r_arm_j2_link"/>

Commit message: modified the setting of smartpal5_moveit_config

File: tms_rp/smartpal5_description/urdf/smartpal5.urdf (robot description, URDF)
Before this commit: robot smartpal5, 28 links, 27 joints
Joints:
- removed joint r_armj2_joint
- added joint r_arm_j2_joint: type revolute, parent r_arm_j1_link, child r_arm_j2_link, origin xyz=0 0 0 rpy=-1.57075 0 -1.57075, axis 0 0 1, limit lower=-1.9024 upper=0.2443 effort=100.0 velocity=1.0

Commit message: chaged the position of end effectors

File: tms_rp/smartpal5_description/urdf/smartpal5.urdf (robot description, URDF)
Before this commit: robot smartpal5, 28 links, 27 joints
Joints:
- joint l_end_effector_joint: origin xyz=0.05 0 0 rpy=0 0 0 -> xyz=0.01 0.11 0 rpy=0 0 0
- joint r_end_effector_joint: origin xyz=0 0.05 0 rpy=0 0 0 -> xyz=0.11 0.01 0 rpy=0 0 0
