Commit message: We can call the models like environments, objects and robots

File: tms_rp/rostms_description/urdf/robots_standalone.urdf.xacro (robot description, xacro)
@@ -9,5 +9,10 @@
   <xacro:include filename="$(find rostms_description)/urdf/common_properties.urdf.xacro" />
   <!-- Used for fixing all components to 'world' frame of RViz and Gazebo 'world' -->
-  <link name="world"/>
+  <link name="world_link"/>
+  <joint name="world_smartpal5_joint" type="fixed">
+	  <parent link="world_link"/>
+    <child link="smartpal5_link"/>
+    <origin xyz="0 0 0" rpy="0 0 0"/>
+  </joint>
   <!-- Defines the component tags -->
   <xacro:include filename="$(find rostms_description)/urdf/robots.urdf.xacro" />
