Commit message: added smartpal_gazebo package

File: tms_rp/rostms_description/urdf/robots.urdf.xacro (robot description, xacro)
@@ -6,5 +6,5 @@
   <xacro:macro name="robots">
     <xacro:include filename="$(find smartpal5_description)/urdf/smartpal5.urdf.xacro" />
-    <xacro:smartpal5_sim/>
+    <xacro:robots_sim/>
   </xacro:macro>
 </robot>

File: tms_rp/smartpal5_description/urdf/smartpal5_gazebo.urdf.xacro (robot description, xacro)
@@ -1,5 +1,58 @@
 <?xml version="1.0"?>
-<robot name="smartpal5_sim" xmlns:xacro="http://ros.org/wiki/xacro">
-  <xacro:macro name="smartpal5_sim">
-  </xacro:macro>
+<robot>
+  <!-- ros_control plugin -->
+  <gazebo>
+    <plugin name="gazebo_ros_control" filename="libgazebo_ros_control.so">
+      <robotNamespace>/smartpal</robotNamespace>
+      <robotSimType>gazebo_ros_control/DefaultRobotHWSim</robotSimType>
+    </plugin>
+  </gazebo>
+  <gazebo reference="base_link">
+  </gazebo>
+  <gazebo reference="lumbar_lower_link">
+  </gazebo>
+  <gazebo reference="lumbar_upper_link">
+  </gazebo>
+  <gazebo reference="camera_link">
+  </gazebo>
+  <gazebo reference="l_arm_j1_link">
+  </gazebo>
+  <gazebo reference="l_arm_j2_link">
+  </gazebo>
+  <gazebo reference="l_arm_j3_link">
+  </gazebo>
+  <gazebo reference="l_arm_j4_link">
+  </gazebo>
+  <gazebo reference="l_arm_j5_link">
+  </gazebo>
+  <gazebo reference="l_arm_j6_link">
+  </gazebo>
+  <gazebo reference="l_arm_j7_link">
+  </gazebo>
+  <gazebo reference="l_gripper_link">
+  </gazebo>
+  <gazebo reference="l_end_effector_link">
+  </gazebo>
+  <gazebo reference="l_gripper_thumb_link">
+  </gazebo>
+  <gazebo reference="r_arm_j1_link">
+  </gazebo>
+  <gazebo reference="r_arm_j2_link">
+  </gazebo>
+  <gazebo reference="r_arm_j3_link">
+  </gazebo>
+  <gazebo reference="r_arm_j4_link">
+  </gazebo>
+  <gazebo reference="r_arm_j5_link">
+  </gazebo>
+  <gazebo reference="r_arm_j6_link">
+  </gazebo>
+  <gazebo reference="r_arm_j7_link">
+  </gazebo>
+  <gazebo reference="r_gripper_link">
+  </gazebo>
+  <gazebo reference="r_end_effector_link">
+  </gazebo>
+  <gazebo reference="r_gripper_thumb_link">
+  </gazebo>
 </robot>
