Commit message: modified hierarchy of models

File: tms_rp/rostms_description/urdf/all_components.urdf.xacro (robot description, xacro)
@@ -1,5 +1,5 @@
 <?xml version="1.0"?>
-<!-- all component of ROS-TMS project -->
-<robot name="all_component"
+<!-- All components of ROS-TMS project -->
+<robot name="all_components"
        xmlns:sensor="http://playerstage.sourceforge.net/gazebo/xmlschema/#sensor"
        xmlns:controller="http://playerstage.sourceforge.net/gazebo/xmlschema/#controller"
@@ -7,7 +7,11 @@
        xmlns:xacro="http://ros.org/wiki/xacro">
   <!-- Import common properties -->
-  <xacro:include filename="$(find environment_description)/urdf/common_properties.urdf.xacro" />
-  <!-- Defines the environment component tag. -->
-  <xacro:include filename="$(find environment_description)/urdf/environment_standalone.urdf.xacro" />
-  <environment/>
+  <xacro:include filename="$(find rostms_description)/urdf/common_properties.urdf.xacro" />
+  <!-- Used for fixing all components to 'world' frame of RViz and Gazebo 'world' -->
+  <link name="world"/>
+  <!-- Defines the components tags -->
+  <xacro:include filename="$(find rostms_description)/urdf/environments.urdf.xacro" />
+  <xacro:include filename="$(find rostms_description)/urdf/objects.urdf.xacro" />
+  <objects/>
+  <environments/>
 </robot>

File: tms_rp/rostms_description/urdf/environments.urdf.xacro (robot description, xacro)
@@ -1,10 +1,8 @@
 <?xml version="1.0"?>
-<!-- Environment of ROS-TMS project room -->
-<robot name="environment" xmlns:xacro="http://www.ros.org/wiki/xacro">
+<!-- Environments of ROS-TMS -->
+<robot name="environments" xmlns:xacro="http://www.ros.org/wiki/xacro">
   <!-- Import all Gazebo-customization elements, including Gazebo colors -->
-  <xacro:include filename="$(find environment_description)/urdf/environment_gazebo.urdf.xacro" />
-  <xacro:macro name="environment">
-    <!-- Used for fixing robot to Gazebo 'base_link' -->
-    <link name="world"/>
+  <xacro:include filename="$(find rostms_description)/urdf/environments_gazebo.urdf.xacro"/>
+  <xacro:macro name="environments">
     <!--  Environment -->
     <joint name="world_joint" type="fixed">
@@ -81,82 +79,4 @@
       </visual>
     </link>
-    <joint name="bsen_room_to_chair" type="fixed">
-      <parent link="bsen_origin"/>
-      <child link="chair"/>
-      <origin xyz="0 0 0"/>
-    </joint>
-    <link name="chair">
-      <visual>
-        <geometry>
-          <mesh filename="package://environmental_model/model/chair.dae"/>
-        </geometry>
-        <origin xyz="7.8 5.62 0.51" rpy="0 0 1.57079633"/>
-      </visual>
-    </link>
-    <joint name="bsen_room_to_refrigerator" type="fixed">
-      <parent link="bsen_origin"/>
-      <child link="refrigerator"/>
-      <origin xyz="0 0 0"/>
-    </joint>
-    <link name="refrigerator">
-      <visual>
-        <geometry>
-          <mesh filename="package://environmental_model/model/refrigerator.dae"/>
-        </geometry>
-        <origin xyz="7.2 4.2 0.56" rpy="0 0 0"/>
-      </visual>
-    </link>
-    <joint name="bsen_room_to_meeting_chair1" type="fixed">
-      <parent link="bsen_origin"/>
-      <child link="meeting_chair1"/>
-      <origin xyz="0 0 0"/>
-    </joint>
-    <link name="meeting_chair1">
-      <visual>
-        <geometry>
-          <mesh filename="package://environmental_model/model/meeting_chair.dae"/>
-        </geometry>
-        <origin xyz="1.2 2.1 0.3978" rpy="0 0 -1.57079633"/>
-      </visual>
-    </link>
-    <joint name="bsen_room_to_meeting_chair2" type="fixed">
-      <parent link="bsen_origin"/>
-      <child link="meeting_chair2"/>
-      <origin xyz="0 0 0"/>
-    </joint>
-    <link name="meeting_chair2">
-      <visual>
-        <geometry>
-          <mesh filename="package://environmental_model/model/meeting_chair.dae"/>
-        </geometry>
-        <origin xyz="0.6 1.5 0.3978" rpy="0 0 0"/>
-      </visual>
-    </link>
-     <joint name="bsen_room_to_meeting_chair3" type="fixed">
-      <parent link="bsen_origin"/>
-      <child link="meeting_chair3"/>
-      <origin xyz="0 0 0"/>
-    </joint>
-    <link name="meeting_chair3">
-      <visual>
-        <geometry>
-          <mesh filename="package://environmental_model/model/meeting_chair.dae"/>
-        </geometry>
-        <origin xyz="1.2 0.9 0.3978" rpy="0 0 1.57079633"/>
-      </visual>
-    </link>
-     <joint name="bsen_room_to_meeting_chair4" type="fixed">
-      <parent link="bsen_origin"/>
-      <child link="meeting_chair4"/>
-      <origin xyz="0 0 0"/>
-    </joint>
-    <link name="meeting_chair4">
-      <visual>
-        <geometry>
-          <mesh filename="package://environmental_model/model/meeting_chair.dae"/>
-        </geometry>
-        <origin xyz="1.8 1.5 0.3978" rpy="0 0 3.14159265"/>
-      </visual>
-    </link>
     <joint name="bsen_room_to_meeting_table" type="fixed">
       <parent link="bsen_origin"/>
@@ -341,5 +261,5 @@
       </visual>
     </link>
-    <environment_sim/>
+    <environments_sim/>
   </xacro:macro>
 </robot>

File: tms_rp/rostms_description/urdf/environments_gazebo.urdf.xacro (robot description, xacro)
@@ -1,5 +1,5 @@
 <?xml version="1.0"?>
-<robot name="environment_sim" xmlns:xacro="http://ros.org/wiki/xacro">
-  <xacro:macro name="environment_sim">
+<robot name="environments_sim" xmlns:xacro="http://ros.org/wiki/xacro">
+  <xacro:macro name="environments_sim">
   </xacro:macro>
 </robot>

File: tms_rp/rostms_description/urdf/environments_standalone.urdf.xacro (robot description, xacro)
@@ -1,5 +1,5 @@
 <?xml version="1.0"?>
-<!-- Environment component of ROS-TMS project -->
-<robot name="environment_standalone"
+<!-- Environments of ROS-TMS project -->
+<robot name="environments_standalone"
        xmlns:sensor="http://playerstage.sourceforge.net/gazebo/xmlschema/#sensor"
        xmlns:controller="http://playerstage.sourceforge.net/gazebo/xmlschema/#controller"
@@ -7,7 +7,9 @@
        xmlns:xacro="http://ros.org/wiki/xacro">
   <!-- Import common properties -->
-  <xacro:include filename="$(find environment_description)/urdf/common_properties.urdf.xacro" />
-  <!-- Defines the environment component tag. -->
-  <xacro:include filename="$(find environment_description)/urdf/environment.urdf.xacro" />
-  <environment/>
+  <xacro:include filename="$(find rostms_description)/urdf/common_properties.urdf.xacro" />
+  <!-- Used for fixing all components to 'world' frame of RViz and Gazebo 'world' -->
+  <link name="world"/>
+  <!-- Defines the component tags -->
+  <xacro:include filename="$(find rostms_description)/urdf/environments.urdf.xacro" />
+  <environments/>
 </robot>

File: tms_rp/rostms_description/urdf/objects.urdf.xacro (robot description, xacro)
@@ -1,40 +1,212 @@
 <?xml version="1.0"?>
-<!-- Environment of B-Sen Project room -->
-<robot name="object" xmlns:xacro="http://www.ros.org/wiki/xacro">
+<!-- Objects of ROS-TMS -->
+<robot name="objects" xmlns:xacro="http://www.ros.org/wiki/xacro">
   <!-- Import all Gazebo-customization elements, including Gazebo colors -->
-  <xacro:include filename="$(find environment_description)/urdf/environment.gazebo" />
-  <!-- Import Rviz colors -->
-  <xacro:include filename="$(find environment_description)/urdf/materials.xacro" />
-  <!-- Used for fixing robot to Gazebo 'base_link' -->
-  <link name="world"/>
-  <!--  Movable object  -->
-  <link name="wagon">
-    <visual>
-      <geometry>
-        <mesh filename="package://environmental_model/model/wagon.dae"/>
-      </geometry>
-      <origin xyz="0. 0. 0.5" rpy="0 0 1.57079633"/>
-    </visual>
-  </link>
-  <!-- ========== Movable object ========== -->
-  <link name="wagon_x_link"/>
-  <joint name="wagon_x_joint" type="prismatic">
-    <parent link="world"/>
-    <child link="wagon_x_link"/>
-    <origin xyz="0 0 0" rpy="0 0 0"/>
-    <limit effort="1000.0" lower="0." upper="15." velocity="0.5"/>
-  </joint>
-  <link name="wagon_y_link"/>
-  <joint name="wagon_y_joint" type="prismatic">
-    <parent link="wagon_x_link"/>
-    <child link="wagon_y_link"/>
-    <origin xyz="0 0 0" rpy="0 0 1.57079633"/>
-    <limit effort="1000.0" lower="0." upper="7." velocity="0.5"/>
-  </joint>
-  <joint name="wagon_theta_joint" type="continuous">
-    <parent link="wagon_y_link"/>
-    <child link="wagon"/>
-    <origin xyz="0 0 0" rpy="0 0 0"/>
-    <axis xyz="0 0 1"/>
-  </joint>
+  <xacro:include filename="$(find rostms_description)/urdf/objects_gazebo.urdf.xacro" />
+  <xacro:macro name="objects">
+    <!-- chair -->
+    <link name="chair">
+      <visual>
+        <geometry>
+          <mesh filename="package://environmental_model/model/chair.dae"/>
+        </geometry>
+        <origin xyz="12.3 5.62 0.51" rpy="0 0 1.57079633"/>
+      </visual>
+    </link>
+    <link name="chair_x_link"/>
+    <joint name="chair_x_joint" type="prismatic">
+      <parent link="world"/>
+      <child link="chair_x_link"/>
+      <origin xyz="0 0 0" rpy="0 0 0"/>
+      <limit effort="1000.0" lower="0." upper="15." velocity="0.5"/>
+    </joint>
+    <link name="chair_y_link"/>
+    <joint name="chair_y_joint" type="prismatic">
+      <parent link="chair_x_link"/>
+      <child link="chair_y_link"/>
+      <origin xyz="0 0 0" rpy="0 0 1.57079633"/>
+      <limit effort="1000.0" lower="0." upper="8." velocity="0.5"/>
+    </joint>
+    <joint name="chair_yaw_joint" type="continuous">
+      <parent link="chair_y_link"/>
+      <child link="chair"/>
+      <origin xyz="0 0 0" rpy="0 0 0"/>
+      <axis xyz="0 0 1"/>
+    </joint>
+    <!-- refrigerator -->
+    <link name="refrigerator">
+      <visual>
+        <geometry>
+          <mesh filename="package://environmental_model/model/refrigerator.dae"/>
+        </geometry>
+        <origin xyz="11.7 4.2 0.56" rpy="0 0 0"/>
+      </visual>
+    </link>
+    <link name="refrigerator_x_link"/>
+    <joint name="refrigerator_x_joint" type="prismatic">
+      <parent link="world"/>
+      <child link="refrigerator_x_link"/>
+      <origin xyz="0 0 0" rpy="0 0 0"/>
+      <limit effort="1000.0" lower="0." upper="15." velocity="0.5"/>
+    </joint>
+    <link name="refrigerator_y_link"/>
+    <joint name="refrigerator_y_joint" type="prismatic">
+      <parent link="refrigerator_x_link"/>
+      <child link="refrigerator_y_link"/>
+      <origin xyz="0 0 0" rpy="0 0 1.57079633"/>
+      <limit effort="1000.0" lower="0." upper="8." velocity="0.5"/>
+    </joint>
+    <joint name="refrigerator_yaw_joint" type="continuous">
+      <parent link="refrigerator_y_link"/>
+      <child link="refrigerator"/>
+      <origin xyz="0 0 0" rpy="0 0 0"/>
+      <axis xyz="0 0 1"/>
+    </joint>
+    <!-- meeting_chair1 -->
+    <link name="meeting_chair1">
+      <visual>
+        <geometry>
+          <mesh filename="package://environmental_model/model/meeting_chair.dae"/>
+        </geometry>
+        <origin xyz="5.7 2.1 0.3978" rpy="0 0 -1.57079633"/>
+      </visual>
+    </link>
+    <link name="meeting_chair1_x_link"/>
+    <joint name="meeting_chair1_x_joint" type="prismatic">
+      <parent link="world"/>
+      <child link="meeting_chair1_x_link"/>
+      <origin xyz="0 0 0" rpy="0 0 0"/>
+      <limit effort="1000.0" lower="0." upper="15." velocity="0.5"/>
+    </joint>
+    <link name="meeting_chair1_y_link"/>
+    <joint name="meeting_chair1_y_joint" type="prismatic">
+      <parent link="meeting_chair1_x_link"/>
+      <child link="meeting_chair1_y_link"/>
+      <origin xyz="0 0 0" rpy="0 0 1.57079633"/>
+      <limit effort="1000.0" lower="0." upper="8." velocity="0.5"/>
+    </joint>
+    <joint name="meeting_chair1_yaw_joint" type="continuous">
+      <parent link="meeting_chair1_y_link"/>
+      <child link="meeting_chair1"/>
+      <origin xyz="0 0 0" rpy="0 0 0"/>
+      <axis xyz="0 0 1"/>
+    </joint>
+    <!--  meeting_chair2 -->
+    <link name="meeting_chair2">
+      <visual>
+        <geometry>
+          <mesh filename="package://environmental_model/model/meeting_chair.dae"/>
+        </geometry>
+        <origin xyz="5.1 1.5 0.3978" rpy="0 0 0"/>
+      </visual>
+    </link>
+    <link name="meeting_chair2_x_link"/>
+    <joint name="meeting_chair2_x_joint" type="prismatic">
+      <parent link="world"/>
+      <child link="meeting_chair2_x_link"/>
+      <origin xyz="0 0 0" rpy="0 0 0"/>
+      <limit effort="1000.0" lower="0." upper="15." velocity="0.5"/>
+    </joint>
+    <link name="meeting_chair2_y_link"/>
+    <joint name="meeting_chair2_y_joint" type="prismatic">
+      <parent link="meeting_chair2_x_link"/>
+      <child link="meeting_chair2_y_link"/>
+      <origin xyz="0 0 0" rpy="0 0 1.57079633"/>
+      <limit effort="1000.0" lower="0." upper="8." velocity="0.5"/>
+    </joint>
+    <joint name="meeting_chair2_yaw_joint" type="continuous">
+      <parent link="meeting_chair2_y_link"/>
+      <child link="meeting_chair2"/>
+      <origin xyz="0 0 0" rpy="0 0 0"/>
+      <axis xyz="0 0 1"/>
+    </joint>
+    <!-- meeting_chair3 -->
+    <link name="meeting_chair3">
+      <visual>
+        <geometry>
+          <mesh filename="package://environmental_model/model/meeting_chair.dae"/>
+        </geometry>
+        <origin xyz="5.7 0.9 0.3978" rpy="0 0 1.57079633"/>
+      </visual>
+    </link>
+    <link name="meeting_chair3_x_link"/>
+    <joint name="meeting_chair3_x_joint" type="prismatic">
+      <parent link="world"/>
+      <child link="meeting_chair3_x_link"/>
+      <origin xyz="0 0 0" rpy="0 0 0"/>
+      <limit effort="1000.0" lower="0." upper="15." velocity="0.5"/>
+    </joint>
+    <link name="meeting_chair3_y_link"/>
+    <joint name="meeting_chair3_y_joint" type="prismatic">
+      <parent link="meeting_chair3_x_link"/>
+      <child link="meeting_chair3_y_link"/>
+      <origin xyz="0 0 0" rpy="0 0 1.57079633"/>
+      <limit effort="1000.0" lower="0." upper="8." velocity="0.5"/>
+    </joint>
+    <joint name="meeting_chair3_yaw_joint" type="continuous">
+      <parent link="meeting_chair3_y_link"/>
+      <child link="meeting_chair3"/>
+      <origin xyz="0 0 0" rpy="0 0 0"/>
+      <axis xyz="0 0 1"/>
+    </joint>
+    <!-- meeting_chair4 -->
+    <link name="meeting_chair4">
+      <visual>
+        <geometry>
+          <mesh filename="package://environmental_model/model/meeting_chair.dae"/>
+        </geometry>
+        <origin xyz="6.3 1.5 0.3978" rpy="0 0 3.14159265"/>
+      </visual>
+    </link>
+    <link name="meeting_chair4_x_link"/>
+    <joint name="meeting_chair4_x_joint" type="prismatic">
+      <parent link="world"/>
+      <child link="meeting_chair4_x_link"/>
+      <origin xyz="0 0 0" rpy="0 0 0"/>
+      <limit effort="1000.0" lower="0." upper="15." velocity="0.5"/>
+    </joint>
+    <link name="meeting_chair4_y_link"/>
+    <joint name="meeting_chair4_y_joint" type="prismatic">
+      <parent link="meeting_chair4_x_link"/>
+      <child link="meeting_chair4_y_link"/>
+      <origin xyz="0 0 0" rpy="0 0 1.57079633"/>
+      <limit effort="1000.0" lower="0." upper="8." velocity="0.5"/>
+    </joint>
+    <joint name="meeting_chair4_yaw_joint" type="continuous">
+      <parent link="meeting_chair4_y_link"/>
+      <child link="meeting_chair4"/>
+      <origin xyz="0 0 0" rpy="0 0 0"/>
+      <axis xyz="0 0 1"/>
+    </joint>
+    <!-- wagon -->
+    <link name="wagon">
+      <visual>
+        <geometry>
+          <mesh filename="package://environmental_model/model/wagon.dae"/>
+        </geometry>
+        <origin xyz="0. 0. 0.5" rpy="0 0 1.57079633"/>
+      </visual>
+    </link>
+    <link name="wagon_x_link"/>
+    <joint name="wagon_x_joint" type="prismatic">
+      <parent link="world"/>
+      <child link="wagon_x_link"/>
+      <origin xyz="0 0 0" rpy="0 0 0"/>
+      <limit effort="1000.0" lower="0." upper="15." velocity="0.5"/>
+    </joint>
+    <link name="wagon_y_link"/>
+    <joint name="wagon_y_joint" type="prismatic">
+      <parent link="wagon_x_link"/>
+      <child link="wagon_y_link"/>
+      <origin xyz="0 0 0" rpy="0 0 1.57079633"/>
+      <limit effort="1000.0" lower="0." upper="8." velocity="0.5"/>
+    </joint>
+    <joint name="wagon_yaw_joint" type="continuous">
+      <parent link="wagon_y_link"/>
+      <child link="wagon"/>
+      <origin xyz="0 0 0" rpy="0 0 0"/>
+      <axis xyz="0 0 1"/>
+    </joint>
+    <objects_sim/>
+  </xacro:macro>
 </robot>

File: tms_rp/rostms_description/urdf/objects_gazebo.urdf.xacro (robot description, xacro)
@@ -1,5 +1,5 @@
 <?xml version="1.0"?>
-<robot name="environment_sim" xmlns:xacro="http://ros.org/wiki/xacro">
-  <xacro:macro name="environment_sim">
+<robot name="objects_sim" xmlns:xacro="http://ros.org/wiki/xacro">
+  <xacro:macro name="objects_sim">
   </xacro:macro>
 </robot>

File: tms_rp/rostms_description/urdf/objects_standalone.urdf.xacro (robot description, xacro)
@@ -1,40 +1,15 @@
 <?xml version="1.0"?>
-<!-- Environment of B-Sen Project room -->
-<robot name="objects" xmlns:xacro="http://www.ros.org/wiki/xacro">
-  <!-- Import all Gazebo-customization elements, including Gazebo colors -->
-  <xacro:include filename="$(find environment_description)/urdf/environment.gazebo" />
-  <!-- Import Rviz colors -->
-  <xacro:include filename="$(find environment_description)/urdf/materials.xacro" />
-  <!-- Used for fixing robot to Gazebo 'base_link' -->
+<!-- Objects of ROS-TMS project -->
+<robot name="objects_standalone"
+       xmlns:sensor="http://playerstage.sourceforge.net/gazebo/xmlschema/#sensor"
+       xmlns:controller="http://playerstage.sourceforge.net/gazebo/xmlschema/#controller"
+       xmlns:interface="http://playerstage.sourceforge.net/gazebo/xmlschema/#interface"
+       xmlns:xacro="http://ros.org/wiki/xacro">
+  <!-- Import common properties -->
+  <xacro:include filename="$(find rostms_description)/urdf/common_properties.urdf.xacro" />
+  <!-- Used for fixing all components to 'world' frame of RViz and Gazebo 'world' -->
   <link name="world"/>
-  <!--  Movable object  -->
-  <link name="wagon">
-    <visual>
-      <geometry>
-        <mesh filename="package://environmental_model/model/wagon.dae"/>
-      </geometry>
-      <origin xyz="0. 0. 0.5" rpy="0 0 1.57079633"/>
-    </visual>
-  </link>
-  <!-- ========== Movable object ========== -->
-  <link name="wagon_x_link"/>
-  <joint name="wagon_x_joint" type="prismatic">
-    <parent link="world"/>
-    <child link="wagon_x_link"/>
-    <origin xyz="0 0 0" rpy="0 0 0"/>
-    <limit effort="1000.0" lower="0." upper="15." velocity="0.5"/>
-  </joint>
-  <link name="wagon_y_link"/>
-  <joint name="wagon_y_joint" type="prismatic">
-    <parent link="wagon_x_link"/>
-    <child link="wagon_y_link"/>
-    <origin xyz="0 0 0" rpy="0 0 1.57079633"/>
-    <limit effort="1000.0" lower="0." upper="7." velocity="0.5"/>
-  </joint>
-  <joint name="wagon_theta_joint" type="continuous">
-    <parent link="wagon_y_link"/>
-    <child link="wagon"/>
-    <origin xyz="0 0 0" rpy="0 0 0"/>
-    <axis xyz="0 0 1"/>
-  </joint>
+  <!-- Defines the component tags -->
+  <xacro:include filename="$(find rostms_description)/urdf/objects.urdf.xacro" />
+  <objects/>
 </robot>
