Commit message: added 4 pattern models configuration

File: tms_rp/rostms_description/urdf/all_components.urdf.xacro (robot description, xacro)
@@ -12,6 +12,8 @@
   <!-- Defines the components tags -->
   <xacro:include filename="$(find rostms_description)/urdf/environments.urdf.xacro" />
+  <environments/>
   <xacro:include filename="$(find rostms_description)/urdf/objects.urdf.xacro" />
   <objects/>
-  <environments/>
+  <xacro:include filename="$(find rostms_description)/urdf/robots.urdf.xacro" />
+  <robots/>
 </robot>

File: tms_rp/rostms_description/urdf/objects.urdf.xacro (robot description, xacro)
@@ -11,5 +11,5 @@
           <mesh filename="package://environmental_model/model/chair.dae"/>
         </geometry>
-        <origin xyz="12.3 5.62 0.51" rpy="0 0 1.57079633"/>
+        <origin xyz="0.0 0.0 0.51" rpy="0.0 0.0 0.0"/>
       </visual>
     </link>
@@ -40,5 +40,5 @@
           <mesh filename="package://environmental_model/model/refrigerator.dae"/>
         </geometry>
-        <origin xyz="11.7 4.2 0.56" rpy="0 0 0"/>
+        <origin xyz="0.0 0.0 0.56" rpy="0 0 0"/>
       </visual>
     </link>
@@ -69,5 +69,5 @@
           <mesh filename="package://environmental_model/model/meeting_chair.dae"/>
         </geometry>
-        <origin xyz="5.7 2.1 0.3978" rpy="0 0 -1.57079633"/>
+        <origin xyz="0.0 0.0 0.3978" rpy="0 0 0"/>
       </visual>
     </link>
@@ -98,5 +98,5 @@
           <mesh filename="package://environmental_model/model/meeting_chair.dae"/>
         </geometry>
-        <origin xyz="5.1 1.5 0.3978" rpy="0 0 0"/>
+        <origin xyz="0.0 0.0 0.3978" rpy="0 0 0"/>
       </visual>
     </link>
@@ -127,5 +127,5 @@
           <mesh filename="package://environmental_model/model/meeting_chair.dae"/>
         </geometry>
-        <origin xyz="5.7 0.9 0.3978" rpy="0 0 1.57079633"/>
+        <origin xyz="0.0 0.0 0.3978" rpy="0 0 0"/>
       </visual>
     </link>
@@ -156,5 +156,5 @@
           <mesh filename="package://environmental_model/model/meeting_chair.dae"/>
         </geometry>
-        <origin xyz="6.3 1.5 0.3978" rpy="0 0 3.14159265"/>
+        <origin xyz="0.0 0.0 0.3978" rpy="0 0 0"/>
       </visual>
     </link>
@@ -185,5 +185,5 @@
           <mesh filename="package://environmental_model/model/wagon.dae"/>
         </geometry>
-        <origin xyz="0. 0. 0.5" rpy="0 0 1.57079633"/>
+        <origin xyz="0. 0. 0.5" rpy="0 0 0"/>
       </visual>
     </link>

File: tms_rp/rostms_description/urdf/robots.urdf.xacro (robot description, xacro)
@@ -1,40 +1,10 @@
 <?xml version="1.0"?>
-<!-- Environment of B-Sen Project room -->
-<robot name="object" xmlns:xacro="http://www.ros.org/wiki/xacro">
+<!-- Robots of ROS-TMS -->
+<robot name="robots" xmlns:xacro="http://www.ros.org/wiki/xacro">
   <!-- Import all Gazebo-customization elements, including Gazebo colors -->
-  <xacro:include filename="$(find environment_description)/urdf/environment.gazebo" />
-  <!-- Import Rviz colors -->
-  <xacro:include filename="$(find environment_description)/urdf/materials.xacro" />
-  <!-- Used for fixing robot to Gazebo 'base_link' -->
-  <link name="world"/>
-  <!--  Movable object  -->
-  <link name="wagon">
-    <visual>
-      <geometry>
-        <mesh filename="package://environmental_model/model/wagon.dae"/>
-      </geometry>
-      <origin xyz="0. 0. 0.5" rpy="0 0 1.57079633"/>
-    </visual>
-  </link>
-  <!-- ========== Movable object ========== -->
-  <link name="wagon_x_link"/>
-  <joint name="wagon_x_joint" type="prismatic">
-    <parent link="world"/>
-    <child link="wagon_x_link"/>
-    <origin xyz="0 0 0" rpy="0 0 0"/>
-    <limit effort="1000.0" lower="0." upper="15." velocity="0.5"/>
-  </joint>
-  <link name="wagon_y_link"/>
-  <joint name="wagon_y_joint" type="prismatic">
-    <parent link="wagon_x_link"/>
-    <child link="wagon_y_link"/>
-    <origin xyz="0 0 0" rpy="0 0 1.57079633"/>
-    <limit effort="1000.0" lower="0." upper="7." velocity="0.5"/>
-  </joint>
-  <joint name="wagon_theta_joint" type="continuous">
-    <parent link="wagon_y_link"/>
-    <child link="wagon"/>
-    <origin xyz="0 0 0" rpy="0 0 0"/>
-    <axis xyz="0 0 1"/>
-  </joint>
+  <xacro:include filename="$(find smartpal5_description)/urdf/smartpal5_gazebo.urdf.xacro" />
+  <xacro:macro name="robots">
+  <xacro:include filename="$(find smartpal5_description)/urdf/smartpal5.urdf.xacro" />
+  <smartpal5_sim/>
+  </xacro:macro>
 </robot>

File: tms_rp/rostms_description/urdf/robots_gazebo.urdf.xacro (robot description, xacro)
@@ -1,5 +1,5 @@
 <?xml version="1.0"?>
-<robot name="environment_sim" xmlns:xacro="http://ros.org/wiki/xacro">
-  <xacro:macro name="environment_sim">
+<robot name="robots_sim" xmlns:xacro="http://ros.org/wiki/xacro">
+  <xacro:macro name="robots_sim">
   </xacro:macro>
 </robot>

File: tms_rp/rostms_description/urdf/robots_standalone.urdf.xacro (robot description, xacro)
@@ -1,40 +1,15 @@
 <?xml version="1.0"?>
-<!-- Environment of B-Sen Project room -->
-<robot name="objects" xmlns:xacro="http://www.ros.org/wiki/xacro">
-  <!-- Import all Gazebo-customization elements, including Gazebo colors -->
-  <xacro:include filename="$(find environment_description)/urdf/environment.gazebo" />
-  <!-- Import Rviz colors -->
-  <xacro:include filename="$(find environment_description)/urdf/materials.xacro" />
-  <!-- Used for fixing robot to Gazebo 'base_link' -->
+<!-- Robots of ROS-TMS project -->
+<robot name="robots_standalone"
+       xmlns:sensor="http://playerstage.sourceforge.net/gazebo/xmlschema/#sensor"
+       xmlns:controller="http://playerstage.sourceforge.net/gazebo/xmlschema/#controller"
+       xmlns:interface="http://playerstage.sourceforge.net/gazebo/xmlschema/#interface"
+       xmlns:xacro="http://ros.org/wiki/xacro">
+  <!-- Import common properties -->
+  <xacro:include filename="$(find rostms_description)/urdf/common_properties.urdf.xacro" />
+  <!-- Used for fixing all components to 'world' frame of RViz and Gazebo 'world' -->
   <link name="world"/>
-  <!--  Movable object  -->
-  <link name="wagon">
-    <visual>
-      <geometry>
-        <mesh filename="package://environmental_model/model/wagon.dae"/>
-      </geometry>
-      <origin xyz="0. 0. 0.5" rpy="0 0 1.57079633"/>
-    </visual>
-  </link>
-  <!-- ========== Movable object ========== -->
-  <link name="wagon_x_link"/>
-  <joint name="wagon_x_joint" type="prismatic">
-    <parent link="world"/>
-    <child link="wagon_x_link"/>
-    <origin xyz="0 0 0" rpy="0 0 0"/>
-    <limit effort="1000.0" lower="0." upper="15." velocity="0.5"/>
-  </joint>
-  <link name="wagon_y_link"/>
-  <joint name="wagon_y_joint" type="prismatic">
-    <parent link="wagon_x_link"/>
-    <child link="wagon_y_link"/>
-    <origin xyz="0 0 0" rpy="0 0 1.57079633"/>
-    <limit effort="1000.0" lower="0." upper="7." velocity="0.5"/>
-  </joint>
-  <joint name="wagon_theta_joint" type="continuous">
-    <parent link="wagon_y_link"/>
-    <child link="wagon"/>
-    <origin xyz="0 0 0" rpy="0 0 0"/>
-    <axis xyz="0 0 1"/>
-  </joint>
+  <!-- Defines the component tags -->
+  <xacro:include filename="$(find rostms_description)/urdf/robots.urdf.xacro" />
+  <robots/>
 </robot>

Commit message: modified the descriptions of environments.urdf.xacro

File: tms_rp/rostms_description/urdf/all_components.urdf.xacro (robot description, xacro)
@@ -1,5 +1,5 @@
 <?xml version="1.0"?>
 <!-- All components of ROS-TMS project -->
-<robot name="all_components"
+<robot name="ros-tms"
        xmlns:sensor="http://playerstage.sourceforge.net/gazebo/xmlschema/#sensor"
        xmlns:controller="http://playerstage.sourceforge.net/gazebo/xmlschema/#controller"
@@ -9,11 +9,21 @@
   <xacro:include filename="$(find rostms_description)/urdf/common_properties.urdf.xacro" />
   <!-- Used for fixing all components to 'world' frame of RViz and Gazebo 'world' -->
-  <link name="world"/>
+  <link name="world_link"/>
+  <joint name="world_bsen_room_joint" type="fixed">
+    <parent link="world_link"/>
+    <child link="bsen_room_link"/>
+    <origin xyz="0 0 0" rpy="0 0 0"/>
+  </joint>
+  <!-- <joint name="world_smartpal5_joint" type="fixed">
+	  <parent link="world_link"/>
+    <child link="smartpal5_link"/>
+    <origin xyz="0 0 0" rpy="0 0 0"/>
+  </joint> -->
   <!-- Defines the components tags -->
   <xacro:include filename="$(find rostms_description)/urdf/environments.urdf.xacro" />
-  <environments/>
-  <xacro:include filename="$(find rostms_description)/urdf/objects.urdf.xacro" />
-  <objects/>
-  <xacro:include filename="$(find rostms_description)/urdf/robots.urdf.xacro" />
-  <robots/>
+  <xacro:environments/>
+  <!-- <xacro:include filename="$(find rostms_description)/urdf/objects.urdf.xacro" />
+  <objects/> -->
+  <!-- <xacro:include filename="$(find rostms_description)/urdf/robots.urdf.xacro" />
+  <robots/> -->
 </robot>

File: tms_rp/rostms_description/urdf/environments.urdf.xacro (robot description, xacro)
@@ -6,10 +6,5 @@
   <xacro:macro name="environments">
     <!--  Environment -->
-    <joint name="world_joint" type="fixed">
-      <parent link="world"/>
-      <child link="bsen_room"/>
-      <origin xyz="0 0 0" rpy="0 0 0"/>
-    </joint>
-    <link name="bsen_room">
+    <link name="bsen_room_link">
       <visual>
         <geometry>
@@ -27,10 +22,10 @@
       </inertial>
     </link>
-    <joint name="bsen_room_to_wall" type="fixed">
-      <parent link="bsen_room"/>
-      <child link="bsen_wall"/>
+    <joint name="wall_joint" type="fixed">
+      <parent link="bsen_room_link"/>
+      <child link="bsen_wall_link"/>
       <origin xyz="0. 0. 0." rpy="0 0 0"/>
     </joint>
-    <link name="bsen_wall">
+    <link name="bsen_wall_link">
       <visual>
         <geometry>
@@ -39,10 +34,10 @@
       </visual>
     </link>
-    <joint name="bsen_room_to_celling" type="fixed">
-      <parent link="bsen_room"/>
-      <child link="bsen_celling"/>
+    <joint name="celling_joint" type="fixed">
+      <parent link="bsen_room_link"/>
+      <child link="bsen_celling_link"/>
       <origin xyz="0. 0. 2.3" rpy="0 0 0"/>
     </joint>
-    <link name="bsen_celling">
+    <link name="bsen_celling_link">
       <visual>
         <geometry>
@@ -51,10 +46,10 @@
       </visual>
     </link>
-    <joint name="bsen_room_to_kitchen" type="fixed">
-      <parent link="bsen_room"/>
-      <child link="kitchen"/>
+    <joint name="kitchen_joint" type="fixed">
+      <parent link="bsen_room_link"/>
+      <child link="kitchen_link"/>
       <origin xyz="9.26 5.9 0.4855" rpy="0 0 -1.57079633"/>
     </joint>
-    <link name="kitchen">
+    <link name="kitchen_link">
       <visual>
         <geometry>
@@ -63,10 +58,10 @@
       </visual>
     </link>
-    <joint name="bsen_room_to_meeting_table" type="fixed">
-      <parent link="bsen_room"/>
-      <child link="meeting_table"/>
+    <joint name="meeting_table_joint" type="fixed">
+      <parent link="bsen_room_link"/>
+      <child link="meeting_table_link"/>
       <origin xyz="5.7 1.5 0.36" rpy="0 0 0"/>
     </joint>
-    <link name="meeting_table">
+    <link name="meeting_table_link">
       <visual>
         <geometry>
@@ -75,10 +70,10 @@
       </visual>
     </link>
-    <joint name="bsen_room_to_tree" type="fixed">
-      <parent link="bsen_room"/>
-      <child link="tree"/>
+    <joint name="tree_link" type="fixed">
+      <parent link="bsen_room_link"/>
+      <child link="tree_link"/>
       <origin xyz="14.3 5.3 0." rpy="0 0 0"/>
     </joint>
-    <link name="tree">
+    <link name="tree_link">
       <visual>
         <geometry>
@@ -87,10 +82,10 @@
       </visual>
     </link>
-    <joint name="bsen_room_to_tv_table" type="fixed">
-      <parent link="bsen_room"/>
-      <child link="tv_table"/>
+    <joint name="tv_table_joint" type="fixed">
+      <parent link="bsen_room_link"/>
+      <child link="tv_table_link"/>
       <origin xyz="11.1 2.9 0.175" rpy="0 0 0"/>
     </joint>
-    <link name="tv_table">
+    <link name="tv_table_link">
       <visual>
         <geometry>
@@ -99,10 +94,10 @@
       </visual>
     </link>
-    <joint name="bsen_room_to_tv_52" type="fixed">
-      <parent link="bsen_room"/>
-      <child link="tv_52"/>
+    <joint name="tv_52_link" type="fixed">
+      <parent link="bsen_room_link"/>
+      <child link="tv_52_link"/>
       <origin xyz="11.2 2.9 0.7085" rpy="0 0 -1.57079633"/>
     </joint>
-    <link name="tv_52">
+    <link name="tv_52_link">
       <visual>
         <geometry>
@@ -111,10 +106,10 @@
       </visual>
     </link>
-    <joint name="bsen_room_to_recorder" type="fixed">
-      <parent link="bsen_room"/>
-      <child link="recorder"/>
+    <joint name="recorder_joint" type="fixed">
+      <parent link="bsen_room_link"/>
+      <child link="recorder_link"/>
       <origin xyz="11.1 2.9 0.3805" rpy="0 0 3.14159265"/>
     </joint>
-    <link name="recorder">
+    <link name="recorder_link">
       <visual>
         <geometry>
@@ -123,10 +118,10 @@
       </visual>
     </link>
-    <joint name="bsen_room_to_sofa" type="fixed">
-      <parent link="bsen_room"/>
-      <child link="sofa"/>
+    <joint name="sofa_joint" type="fixed">
+      <parent link="bsen_room_link"/>
+      <child link="sofa_link"/>
       <origin xyz="9.1 2.9 0.395" rpy="0 0 0"/>
     </joint>
-    <link name="sofa">
+    <link name="sofa_link">
       <visual>
         <geometry>
@@ -135,10 +130,10 @@
       </visual>
     </link>
-    <joint name="bsen_room_to_sofa_table" type="fixed">
-      <parent link="bsen_room"/>
-      <child link="sofa_table"/>
+    <joint name="sofa_table_joint" type="fixed">
+      <parent link="bsen_room_link"/>
+      <child link="sofa_table_link"/>
       <origin xyz="10.2 2.9 0.235" rpy="0 0 0"/>
     </joint>
-    <link name="sofa_table">
+    <link name="sofa_table_link">
       <visual>
         <geometry>
@@ -147,10 +142,10 @@
       </visual>
     </link>
-    <joint name="bsen_room_to_carpet" type="fixed">
-      <parent link="bsen_room"/>
-      <child link="carpet"/>
+    <joint name="carpet_joint" type="fixed">
+      <parent link="bsen_room_link"/>
+      <child link="carpet_link"/>
       <origin xyz="9.9 2.9 0.1" rpy="0 0 0"/>
     </joint>
-    <link name="carpet">
+    <link name="carpet_link">
       <visual>
         <geometry>
@@ -159,10 +154,10 @@
       </visual>
     </link>
-    <joint name="bsen_room_to_drawer" type="fixed">
-      <parent link="bsen_room"/>
-      <child link="drawer"/>
+    <joint name="drawer_joint" type="fixed">
+      <parent link="bsen_room_link"/>
+      <child link="drawer_link"/>
       <origin xyz="12.93 5.8 0.303" rpy="0 0 -1.57079633"/>
     </joint>
-    <link name="drawer">
+    <link name="drawer_link">
       <visual>
         <geometry>
@@ -171,10 +166,10 @@
       </visual>
     </link>
-    <joint name="bsen_room_to_bed" type="fixed">
-      <parent link="bsen_room"/>
-      <child link="bed"/>
+    <joint name="bed_joint" type="fixed">
+      <parent link="bsen_room_link"/>
+      <child link="bed_link"/>
       <origin xyz="12.48 2.3 0.2075" rpy="0 0 0"/>
     </joint>
-    <link name="bed">
+    <link name="bed_link">
       <visual>
         <geometry>
@@ -183,10 +178,10 @@
       </visual>
     </link>
-    <joint name="bsen_room_to_wordrobe" type="fixed">
-      <parent link="bsen_room"/>
-      <child link="wardrobe"/>
+    <joint name="wardrobe_joint" type="fixed">
+      <parent link="bsen_room_link"/>
+      <child link="wardrobe_link"/>
       <origin xyz="13.7 5.9 1.3" rpy="0 0 -1.57079633"/>
     </joint>
-    <link name="wardrobe">
+    <link name="wardrobe_link">
       <visual>
         <geometry>
@@ -195,10 +190,10 @@
       </visual>
     </link>
-    <joint name="bsen_room_to_workdesk" type="fixed">
-      <parent link="bsen_room"/>
-      <child link="workdesk"/>
+    <joint name="workdesk_joint" type="fixed">
+      <parent link="bsen_room_link"/>
+      <child link="workdesk_link"/>
       <origin xyz="12.05 5.9 0.5" rpy="0 0 -1.57079633"/>
     </joint>
-    <link name="workdesk">
+    <link name="workdesk_link">
       <visual>
         <geometry>
@@ -207,10 +202,10 @@
       </visual>
     </link>
-    <joint name="bsen_room_to_tv_multi" type="fixed">
-      <parent link="bsen_room"/>
-      <child link="tv_multi"/>
+    <joint name="tv_multi_joint" type="fixed">
+      <parent link="bsen_room_link"/>
+      <child link="tv_multi_link"/>
       <origin xyz="14.37 2.2 1.0" rpy="0 0 -1.57079633"/>
     </joint>
-    <link name="tv_multi">
+    <link name="tv_multi_link">
       <visual>
         <geometry>
@@ -219,10 +214,10 @@
       </visual>
     </link>
-    <joint name="bsen_room_to_intelingent_shelf" type="fixed">
-      <parent link="bsen_room"/>
-      <child link="intelingent_shelf"/>
+    <joint name="intelingent_shelf_joint" type="fixed">
+      <parent link="bsen_room_link"/>
+      <child link="intelingent_shelf_link"/>
       <origin xyz="11.56 3.520 0.445" rpy="0 0 0"/>
     </joint>
-    <link name="intelingent_shelf">
+    <link name="intelingent_shelf_link">
       <visual>
         <geometry>
@@ -231,5 +226,5 @@
       </visual>
     </link>
-    <environments_sim/>
+    <xacro:environments_sim/>
   </xacro:macro>
 </robot>

File: tms_rp/rostms_description/urdf/environments_standalone.urdf.xacro (robot description, xacro)
@@ -9,7 +9,12 @@
   <xacro:include filename="$(find rostms_description)/urdf/common_properties.urdf.xacro" />
   <!-- Used for fixing all components to 'world' frame of RViz and Gazebo 'world' -->
-  <link name="world"/>
+  <link name="world_link"/>
+  <joint name="world_bsen_room_joint" type="fixed">
+    <parent link="world_link"/>
+    <child link="bsen_room_link"/>
+    <origin xyz="0 0 0" rpy="0 0 0"/>
+  </joint>
   <!-- Defines the component tags -->
   <xacro:include filename="$(find rostms_description)/urdf/environments.urdf.xacro" />
-  <environments/>
+  <xacro:environments/>
 </robot>

File: tms_rp/rostms_description/urdf/objects.urdf.xacro (robot description, xacro)
@@ -16,5 +16,5 @@
     <link name="chair_x_link"/>
     <joint name="chair_x_joint" type="prismatic">
-      <parent link="world"/>
+      <parent link="world_link"/>
       <child link="chair_x_link"/>
       <origin xyz="0 0 0" rpy="0 0 0"/>
@@ -45,5 +45,5 @@
     <link name="refrigerator_x_link"/>
     <joint name="refrigerator_x_joint" type="prismatic">
-      <parent link="world"/>
+      <parent link="world_link"/>
       <child link="refrigerator_x_link"/>
       <origin xyz="0 0 0" rpy="0 0 0"/>
@@ -74,5 +74,5 @@
     <link name="meeting_chair1_x_link"/>
     <joint name="meeting_chair1_x_joint" type="prismatic">
-      <parent link="world"/>
+      <parent link="world_link"/>
       <child link="meeting_chair1_x_link"/>
       <origin xyz="0 0 0" rpy="0 0 0"/>
@@ -103,5 +103,5 @@
     <link name="meeting_chair2_x_link"/>
     <joint name="meeting_chair2_x_joint" type="prismatic">
-      <parent link="world"/>
+      <parent link="world_link"/>
       <child link="meeting_chair2_x_link"/>
       <origin xyz="0 0 0" rpy="0 0 0"/>
@@ -132,5 +132,5 @@
     <link name="meeting_chair3_x_link"/>
     <joint name="meeting_chair3_x_joint" type="prismatic">
-      <parent link="world"/>
+      <parent link="world_link"/>
       <child link="meeting_chair3_x_link"/>
       <origin xyz="0 0 0" rpy="0 0 0"/>
@@ -161,5 +161,5 @@
     <link name="meeting_chair4_x_link"/>
     <joint name="meeting_chair4_x_joint" type="prismatic">
-      <parent link="world"/>
+      <parent link="world_link"/>
       <child link="meeting_chair4_x_link"/>
       <origin xyz="0 0 0" rpy="0 0 0"/>
@@ -190,5 +190,5 @@
     <link name="wagon_x_link"/>
     <joint name="wagon_x_joint" type="prismatic">
-      <parent link="world"/>
+      <parent link="world_link"/>
       <child link="wagon_x_link"/>
       <origin xyz="0 0 0" rpy="0 0 0"/>

File: tms_rp/rostms_description/urdf/robots.urdf.xacro (robot description, xacro)
@@ -5,6 +5,6 @@
   <xacro:include filename="$(find smartpal5_description)/urdf/smartpal5_gazebo.urdf.xacro" />
   <xacro:macro name="robots">
-  <xacro:include filename="$(find smartpal5_description)/urdf/smartpal5.urdf.xacro" />
-  <smartpal5_sim/>
+    <xacro:include filename="$(find smartpal5_description)/urdf/smartpal5.urdf.xacro" />
+    <smartpal5_sim/>
   </xacro:macro>
 </robot>

Commit message: add scripts of demo for simulation test

File: tms_rp/rostms_description/urdf/all_components.urdf.xacro (robot description, xacro)
@@ -1,9 +1,5 @@
 <?xml version="1.0"?>
 <!-- All components of ROS-TMS project -->
-<robot name="rostms"
-       xmlns:sensor="http://playerstage.sourceforge.net/gazebo/xmlschema/#sensor"
-       xmlns:controller="http://playerstage.sourceforge.net/gazebo/xmlschema/#controller"
-       xmlns:interface="http://playerstage.sourceforge.net/gazebo/xmlschema/#interface"
-       xmlns:xacro="http://ros.org/wiki/xacro">
+<robot name="rostms" xmlns:xacro="http://ros.org/wiki/xacro">
   <!-- Import common properties -->
   <xacro:include filename="$(find rostms_description)/urdf/common_properties.urdf.xacro" />

File: tms_rp/rostms_description/urdf/environments.urdf.xacro (robot description, xacro)
@@ -21,5 +21,5 @@
       <inertial>
         <origin xyz="0 0 0.001" rpy="0 0 0"/>
-        <mass value="1"/>
+        <mass value="100"/>
         <inertia
           ixx="1.0" ixy="0.0" ixz="0.0"
@@ -78,4 +78,12 @@
         </geometry>
       </collision>
+      <inertial>
+        <origin xyz="0 0 0.001" rpy="0 0 0"/>
+        <mass value="50"/>
+        <inertia
+          ixx="1.0" ixy="0.0" ixz="0.0"
+          iyy="1.0" iyz="0.0"
+          izz="1.0"/>
+      </inertial>
     </link>
     <joint name="meeting_table_joint" type="fixed">
