Commit message: modified the descriptions of objects.urdf.xacro

File: tms_rp/rostms_description/urdf/all_components.urdf (robot description, URDF)
Before this commit: robot ros-tms, 19 links, 18 joints
Links:
- added link chair; visual mesh filename=package://environmental_model/model/chair.dae
- added link chair_x_link
- added link chair_y_link
- added link meeting_chair1; visual mesh filename=package://environmental_model/model/meeting_chair.dae
- added link meeting_chair1_x_link
- added link meeting_chair1_y_link
- added link meeting_chair2; visual mesh filename=package://environmental_model/model/meeting_chair.dae
- added link meeting_chair2_x_link
- added link meeting_chair2_y_link
- added link meeting_chair3; visual mesh filename=package://environmental_model/model/meeting_chair.dae
- added link meeting_chair3_x_link
- added link meeting_chair3_y_link
- added link meeting_chair4; visual mesh filename=package://environmental_model/model/meeting_chair.dae
- added link meeting_chair4_x_link
- added link meeting_chair4_y_link
- added link refrigerator; visual mesh filename=package://environmental_model/model/refrigerator.dae
- added link refrigerator_x_link
- added link refrigerator_y_link
- added link wagon; visual mesh filename=package://environmental_model/model/wagon.dae
- added link wagon_x_link
- added link wagon_y_link
Joints:
- added joint chair_x_joint: type prismatic, parent world_link, child chair_x_link, origin xyz=0 0 0 rpy=0 0 0, limit lower=0. upper=15. effort=1000.0 velocity=0.5
- added joint chair_y_joint: type prismatic, parent chair_x_link, child chair_y_link, origin xyz=0 0 0 rpy=0 0 1.57079633, limit lower=0. upper=8. effort=1000.0 velocity=0.5
- added joint chair_yaw_joint: type continuous, parent chair_y_link, child chair, origin xyz=0 0 0 rpy=0 0 0, axis 0 0 1
- added joint meeting_chair1_x_joint: type prismatic, parent world_link, child meeting_chair1_x_link, origin xyz=0 0 0 rpy=0 0 0, limit lower=0. upper=15. effort=1000.0 velocity=0.5
- added joint meeting_chair1_y_joint: type prismatic, parent meeting_chair1_x_link, child meeting_chair1_y_link, origin xyz=0 0 0 rpy=0 0 1.57079633, limit lower=0. upper=8. effort=1000.0 velocity=0.5
- added joint meeting_chair1_yaw_joint: type continuous, parent meeting_chair1_y_link, child meeting_chair1, origin xyz=0 0 0 rpy=0 0 0, axis 0 0 1
- added joint meeting_chair2_x_joint: type prismatic, parent world_link, child meeting_chair2_x_link, origin xyz=0 0 0 rpy=0 0 0, limit lower=0. upper=15. effort=1000.0 velocity=0.5
- added joint meeting_chair2_y_joint: type prismatic, parent meeting_chair2_x_link, child meeting_chair2_y_link, origin xyz=0 0 0 rpy=0 0 1.57079633, limit lower=0. upper=8. effort=1000.0 velocity=0.5
- added joint meeting_chair2_yaw_joint: type continuous, parent meeting_chair2_y_link, child meeting_chair2, origin xyz=0 0 0 rpy=0 0 0, axis 0 0 1
- added joint meeting_chair3_x_joint: type prismatic, parent world_link, child meeting_chair3_x_link, origin xyz=0 0 0 rpy=0 0 0, limit lower=0. upper=15. effort=1000.0 velocity=0.5
- added joint meeting_chair3_y_joint: type prismatic, parent meeting_chair3_x_link, child meeting_chair3_y_link, origin xyz=0 0 0 rpy=0 0 1.57079633, limit lower=0. upper=8. effort=1000.0 velocity=0.5
- added joint meeting_chair3_yaw_joint: type continuous, parent meeting_chair3_y_link, child meeting_chair3, origin xyz=0 0 0 rpy=0 0 0, axis 0 0 1
- added joint meeting_chair4_x_joint: type prismatic, parent world_link, child meeting_chair4_x_link, origin xyz=0 0 0 rpy=0 0 0, limit lower=0. upper=15. effort=1000.0 velocity=0.5
- added joint meeting_chair4_y_joint: type prismatic, parent meeting_chair4_x_link, child meeting_chair4_y_link, origin xyz=0 0 0 rpy=0 0 1.57079633, limit lower=0. upper=8. effort=1000.0 velocity=0.5
- added joint meeting_chair4_yaw_joint: type continuous, parent meeting_chair4_y_link, child meeting_chair4, origin xyz=0 0 0 rpy=0 0 0, axis 0 0 1
- added joint refrigerator_x_joint: type prismatic, parent world_link, child refrigerator_x_link, origin xyz=0 0 0 rpy=0 0 0, limit lower=0. upper=15. effort=1000.0 velocity=0.5
- added joint refrigerator_y_joint: type prismatic, parent refrigerator_x_link, child refrigerator_y_link, origin xyz=0 0 0 rpy=0 0 1.57079633, limit lower=0. upper=8. effort=1000.0 velocity=0.5
- added joint refrigerator_yaw_joint: type continuous, parent refrigerator_y_link, child refrigerator, origin xyz=0 0 0 rpy=0 0 0, axis 0 0 1
- added joint wagon_x_joint: type prismatic, parent world_link, child wagon_x_link, origin xyz=0 0 0 rpy=0 0 0, limit lower=0. upper=15. effort=1000.0 velocity=0.5
- added joint wagon_y_joint: type prismatic, parent wagon_x_link, child wagon_y_link, origin xyz=0 0 0 rpy=0 0 1.57079633, limit lower=0. upper=8. effort=1000.0 velocity=0.5
- added joint wagon_yaw_joint: type continuous, parent wagon_y_link, child wagon, origin xyz=0 0 0 rpy=0 0 0, axis 0 0 1

File: tms_rp/rostms_description/urdf/all_components.urdf.xacro (robot description, xacro)
@@ -23,6 +23,6 @@
   <xacro:include filename="$(find rostms_description)/urdf/environments.urdf.xacro" />
   <xacro:environments/>
-  <!-- <xacro:include filename="$(find rostms_description)/urdf/objects.urdf.xacro" />
-  <objects/> -->
+  <xacro:include filename="$(find rostms_description)/urdf/objects.urdf.xacro" />
+  <xacro:objects/>
   <!-- <xacro:include filename="$(find rostms_description)/urdf/robots.urdf.xacro" />
   <robots/> -->

File: tms_rp/rostms_description/urdf/objects.urdf.xacro (robot description, xacro)
@@ -4,14 +4,37 @@
   <!-- Import all Gazebo-customization elements, including Gazebo colors -->
   <xacro:include filename="$(find rostms_description)/urdf/objects_gazebo.urdf.xacro" />
+  <!-- meeting_chair -->
+  <xacro:macro name="meeting_chair" params="num">
+    <link name="meeting_chair${num}_x_link"/>
+    <joint name="meeting_chair${num}_x_joint" type="prismatic">
+      <parent link="world_link"/>
+      <child link="meeting_chair${num}_x_link"/>
+      <origin xyz="0 0 0" rpy="0 0 0"/>
+      <limit effort="1000.0" lower="0." upper="15." velocity="0.5"/>
+    </joint>
+    <link name="meeting_chair${num}_y_link"/>
+    <joint name="meeting_chair${num}_y_joint" type="prismatic">
+      <parent link="meeting_chair${num}_x_link"/>
+      <child link="meeting_chair${num}_y_link"/>
+      <origin xyz="0 0 0" rpy="0 0 1.57079633"/>
+      <limit effort="1000.0" lower="0." upper="8." velocity="0.5"/>
+    </joint>
+    <joint name="meeting_chair${num}_yaw_joint" type="continuous">
+      <parent link="meeting_chair${num}_y_link"/>
+      <child link="meeting_chair${num}"/>
+      <origin xyz="0 0 0" rpy="0 0 0"/>
+      <axis xyz="0 0 1"/>
+    </joint>
+    <link name="meeting_chair${num}">
+      <visual>
+        <geometry>
+          <mesh filename="package://environmental_model/model/meeting_chair.dae"/>
+        </geometry>
+        <origin xyz="0.0 0.0 0.3978" rpy="0 0 0"/>
+      </visual>
+    </link>
+  </xacro:macro>
   <xacro:macro name="objects">
     <!-- chair -->
-    <link name="chair">
-      <visual>
-        <geometry>
-          <mesh filename="package://environmental_model/model/chair.dae"/>
-        </geometry>
-        <origin xyz="0.0 0.0 0.51" rpy="0.0 0.0 0.0"/>
-      </visual>
-    </link>
     <link name="chair_x_link"/>
     <joint name="chair_x_joint" type="prismatic">
@@ -34,13 +57,13 @@
       <axis xyz="0 0 1"/>
     </joint>
-    <!-- refrigerator -->
-    <link name="refrigerator">
+    <link name="chair">
       <visual>
         <geometry>
-          <mesh filename="package://environmental_model/model/refrigerator.dae"/>
+          <mesh filename="package://environmental_model/model/chair.dae"/>
         </geometry>
-        <origin xyz="0.0 0.0 0.56" rpy="0 0 0"/>
+        <origin xyz="0.0 0.0 0.51" rpy="0.0 0.0 0.0"/>
       </visual>
     </link>
+    <!-- refrigerator -->
     <link name="refrigerator_x_link"/>
     <joint name="refrigerator_x_joint" type="prismatic">
@@ -63,129 +86,18 @@
       <axis xyz="0 0 1"/>
     </joint>
-    <!-- meeting_chair1 -->
-    <link name="meeting_chair1">
+    <link name="refrigerator">
       <visual>
         <geometry>
-          <mesh filename="package://environmental_model/model/meeting_chair.dae"/>
+          <mesh filename="package://environmental_model/model/refrigerator.dae"/>
         </geometry>
-        <origin xyz="0.0 0.0 0.3978" rpy="0 0 0"/>
+        <origin xyz="0.0 0.0 0.56" rpy="0 0 0"/>
       </visual>
     </link>
-    <link name="meeting_chair1_x_link"/>
-    <joint name="meeting_chair1_x_joint" type="prismatic">
-      <parent link="world_link"/>
-      <child link="meeting_chair1_x_link"/>
-      <origin xyz="0 0 0" rpy="0 0 0"/>
-      <limit effort="1000.0" lower="0." upper="15." velocity="0.5"/>
-    </joint>
-    <link name="meeting_chair1_y_link"/>
-    <joint name="meeting_chair1_y_joint" type="prismatic">
-      <parent link="meeting_chair1_x_link"/>
-      <child link="meeting_chair1_y_link"/>
-      <origin xyz="0 0 0" rpy="0 0 1.57079633"/>
-      <limit effort="1000.0" lower="0." upper="8." velocity="0.5"/>
-    </joint>
-    <joint name="meeting_chair1_yaw_joint" type="continuous">
-      <parent link="meeting_chair1_y_link"/>
-      <child link="meeting_chair1"/>
-      <origin xyz="0 0 0" rpy="0 0 0"/>
-      <axis xyz="0 0 1"/>
-    </joint>
-    <!--  meeting_chair2 -->
-    <link name="meeting_chair2">
-      <visual>
-        <geometry>
-          <mesh filename="package://environmental_model/model/meeting_chair.dae"/>
-        </geometry>
-        <origin xyz="0.0 0.0 0.3978" rpy="0 0 0"/>
-      </visual>
-    </link>
-    <link name="meeting_chair2_x_link"/>
-    <joint name="meeting_chair2_x_joint" type="prismatic">
-      <parent link="world_link"/>
-      <child link="meeting_chair2_x_link"/>
-      <origin xyz="0 0 0" rpy="0 0 0"/>
-      <limit effort="1000.0" lower="0." upper="15." velocity="0.5"/>
-    </joint>
-    <link name="meeting_chair2_y_link"/>
-    <joint name="meeting_chair2_y_joint" type="prismatic">
-      <parent link="meeting_chair2_x_link"/>
-      <child link="meeting_chair2_y_link"/>
-      <origin xyz="0 0 0" rpy="0 0 1.57079633"/>
-      <limit effort="1000.0" lower="0." upper="8." velocity="0.5"/>
-    </joint>
-    <joint name="meeting_chair2_yaw_joint" type="continuous">
-      <parent link="meeting_chair2_y_link"/>
-      <child link="meeting_chair2"/>
-      <origin xyz="0 0 0" rpy="0 0 0"/>
-      <axis xyz="0 0 1"/>
-    </joint>
-    <!-- meeting_chair3 -->
-    <link name="meeting_chair3">
-      <visual>
-        <geometry>
-          <mesh filename="package://environmental_model/model/meeting_chair.dae"/>
-        </geometry>
-        <origin xyz="0.0 0.0 0.3978" rpy="0 0 0"/>
-      </visual>
-    </link>
-    <link name="meeting_chair3_x_link"/>
-    <joint name="meeting_chair3_x_joint" type="prismatic">
-      <parent link="world_link"/>
-      <child link="meeting_chair3_x_link"/>
-      <origin xyz="0 0 0" rpy="0 0 0"/>
-      <limit effort="1000.0" lower="0." upper="15." velocity="0.5"/>
-    </joint>
-    <link name="meeting_chair3_y_link"/>
-    <joint name="meeting_chair3_y_joint" type="prismatic">
-      <parent link="meeting_chair3_x_link"/>
-      <child link="meeting_chair3_y_link"/>
-      <origin xyz="0 0 0" rpy="0 0 1.57079633"/>
-      <limit effort="1000.0" lower="0." upper="8." velocity="0.5"/>
-    </joint>
-    <joint name="meeting_chair3_yaw_joint" type="continuous">
-      <parent link="meeting_chair3_y_link"/>
-      <child link="meeting_chair3"/>
-      <origin xyz="0 0 0" rpy="0 0 0"/>
-      <axis xyz="0 0 1"/>
-    </joint>
-    <!-- meeting_chair4 -->
-    <link name="meeting_chair4">
-      <visual>
-        <geometry>
-          <mesh filename="package://environmental_model/model/meeting_chair.dae"/>
-        </geometry>
-        <origin xyz="0.0 0.0 0.3978" rpy="0 0 0"/>
-      </visual>
-    </link>
-    <link name="meeting_chair4_x_link"/>
-    <joint name="meeting_chair4_x_joint" type="prismatic">
-      <parent link="world_link"/>
-      <child link="meeting_chair4_x_link"/>
-      <origin xyz="0 0 0" rpy="0 0 0"/>
-      <limit effort="1000.0" lower="0." upper="15." velocity="0.5"/>
-    </joint>
-    <link name="meeting_chair4_y_link"/>
-    <joint name="meeting_chair4_y_joint" type="prismatic">
-      <parent link="meeting_chair4_x_link"/>
-      <child link="meeting_chair4_y_link"/>
-      <origin xyz="0 0 0" rpy="0 0 1.57079633"/>
-      <limit effort="1000.0" lower="0." upper="8." velocity="0.5"/>
-    </joint>
-    <joint name="meeting_chair4_yaw_joint" type="continuous">
-      <parent link="meeting_chair4_y_link"/>
-      <child link="meeting_chair4"/>
-      <origin xyz="0 0 0" rpy="0 0 0"/>
-      <axis xyz="0 0 1"/>
-    </joint>
+    <!-- Add meeting_chair -->
+    <xacro:meeting_chair num="1"/>
+    <xacro:meeting_chair num="2"/>
+    <xacro:meeting_chair num="3"/>
+    <xacro:meeting_chair num="4"/>
     <!-- wagon -->
-    <link name="wagon">
-      <visual>
-        <geometry>
-          <mesh filename="package://environmental_model/model/wagon.dae"/>
-        </geometry>
-        <origin xyz="0. 0. 0.5" rpy="0 0 0"/>
-      </visual>
-    </link>
     <link name="wagon_x_link"/>
     <joint name="wagon_x_joint" type="prismatic">
@@ -208,4 +120,12 @@
       <axis xyz="0 0 1"/>
     </joint>
+    <link name="wagon">
+      <visual>
+        <geometry>
+          <mesh filename="package://environmental_model/model/wagon.dae"/>
+        </geometry>
+        <origin xyz="0. 0. 0.5" rpy="0 0 0"/>
+      </visual>
+    </link>
     <objects_sim/>
   </xacro:macro>

File: tms_rp/rostms_description/urdf/objects_standalone.urdf.xacro (robot description, xacro)
@@ -9,5 +9,5 @@
   <xacro:include filename="$(find rostms_description)/urdf/common_properties.urdf.xacro" />
   <!-- Used for fixing all components to 'world' frame of RViz and Gazebo 'world' -->
-  <link name="world"/>
+  <link name="world_link"/>
   <!-- Defines the component tags -->
   <xacro:include filename="$(find rostms_description)/urdf/objects.urdf.xacro" />
