Commit message: modified the descriptions of smartpal with environmental setting

File: tms_rp/rostms_description/urdf/all_components.urdf (robot description, URDF)
Before this commit: robot ros-tms, 40 links, 39 joints
Links:
- added link base_footprint
- added link base_link, mass 27; collision mesh filename=package://smartpal5_description/meshes/collision/Pal5_body_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; visual mesh filename=package://smartpal5_description/meshes/visual/Pal5_body_veh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
- added link camera_link, mass 0.5; collision box size=0.05 0.2 0.08; visual box size=0.03 0.15 0.05
- added link l_arm_j1_link, mass 0.6; collision mesh filename=package://smartpal5_description/meshes/collision/Pal5_leftA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; visual mesh filename=package://smartpal5_description/meshes/visual/Pal5_leftArm_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
- added link l_arm_j2_link, mass 0.6; collision mesh filename=package://smartpal5_description/meshes/collision/Pal5_leftA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; visual mesh filename=package://smartpal5_description/meshes/visual/Pal5_leftArm_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
- added link l_arm_j3_link, mass 1; collision mesh filename=package://smartpal5_description/meshes/collision/Pal5_leftA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; visual mesh filename=package://smartpal5_description/meshes/visual/Pal5_leftArm_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
- added link l_arm_j4_link, mass 0.6; collision mesh filename=package://smartpal5_description/meshes/collision/Pal5_leftA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; visual mesh filename=package://smartpal5_description/meshes/visual/Pal5_leftArm_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
- added link l_arm_j5_link, mass 0.4; collision mesh filename=package://smartpal5_description/meshes/collision/Pal5_leftA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; visual mesh filename=package://smartpal5_description/meshes/visual/Pal5_leftArm_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
- added link l_arm_j6_link, mass 0.4; collision mesh filename=package://smartpal5_description/meshes/collision/Pal5_leftA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; visual mesh filename=package://smartpal5_description/meshes/visual/Pal5_leftArm_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
- added link l_arm_j7_link, mass 0.4; collision mesh filename=package://smartpal5_description/meshes/collision/Pal5_leftA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; visual mesh filename=package://smartpal5_description/meshes/visual/Pal5_leftArm_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
- added link l_end_effector_link; collision box size=0.001 0.001 0.001; visual box size=0.001 0.001 0.001
- added link l_gripper_link, mass 0.6; collision mesh filename=package://smartpal5_description/meshes/collision/Pal5_leftG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; visual mesh filename=package://smartpal5_description/meshes/visual/Pal5_leftGrip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
- added link l_gripper_thumb_link, mass 0.4; collision mesh filename=package://smartpal5_description/meshes/collision/Pal5_leftG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; visual mesh filename=package://smartpal5_description/meshes/visual/Pal5_leftGrip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
- added link lumbar_lower_link, mass 6; collision mesh filename=package://smartpal5_description/meshes/collision/Pal5_body_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; visual mesh filename=package://smartpal5_description/meshes/visual/Pal5_body_lum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
- added link lumbar_upper_link, mass 30; collision mesh filename=package://smartpal5_description/meshes/collision/Pal5_body_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; visual mesh filename=package://smartpal5_description/meshes/visual/Pal5_body_lum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
- added link r_arm_j1_link, mass 0.6; collision mesh filename=package://smartpal5_description/meshes/collision/Pal5_right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; visual mesh filename=package://smartpal5_description/meshes/visual/Pal5_rightArm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
- added link r_arm_j2_link, mass 0.6; collision mesh filename=package://smartpal5_description/meshes/collision/Pal5_right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; visual mesh filename=package://smartpal5_description/meshes/visual/Pal5_rightArm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
- added link r_arm_j3_link, mass 1; collision mesh filename=package://smartpal5_description/meshes/collision/Pal5_right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; visual mesh filename=package://smartpal5_description/meshes/visual/Pal5_rightArm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
- added link r_arm_j4_link, mass 0.6; collision mesh filename=package://smartpal5_description/meshes/collision/Pal5_right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; visual mesh filename=package://smartpal5_description/meshes/visual/Pal5_rightArm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
- added link r_arm_j5_link, mass 0.4; collision mesh filename=package://smartpal5_description/meshes/collision/Pal5_right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; visual mesh filename=package://smartpal5_description/meshes/visual/Pal5_rightArm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
- added link r_arm_j6_link, mass 0.4; collision mesh filename=package://smartpal5_description/meshes/collision/Pal5_right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; visual mesh filename=package://smartpal5_description/meshes/visual/Pal5_rightArm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
- added link r_arm_j7_link, mass 0.4; collision mesh filename=package://smartpal5_description/meshes/collision/Pal5_right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; visual mesh filename=package://smartpal5_description/meshes/visual/Pal5_rightArm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
- added link r_end_effector_link; collision box size=0.001 0.001 0.001; visual box size=0.001 0.001 0.001
- added link r_gripper_link, mass 0.6; collision mesh filename=package://smartpal5_description/meshes/collision/Pal5_right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; visual mesh filename=package://smartpal5_description/meshes/visual/Pal5_rightGri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
- added link r_gripper_thumb_link, mass 0.4; collision mesh filename=package://smartpal5_description/meshes/collision/Pal5_right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; visual mesh filename=package://smartpal5_description/meshes/visual/Pal5_rightGri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
- added link smartpal5_link
- added link smartpal5_x_link
- added link smartpal5_y_link
Joints:
- added joint base_footprint_joint: type fixed, parent base_footprint, child base_link, origin xyz=0 0 0 rpy=0 0 0
- added joint head_camera_joint: type fixed, parent lumbar_upper_link, child camera_link, origin xyz=0.02 -0.7 0 rpy=1.57075 0 0
- added joint l_arm_j1_joint: type revolute, parent lumbar_upper_link, child l_arm_j1_link, origin xyz=-0.025 -0.480 0.200 rpy=3.14159 0 0, axis 0 0 1, limit lower=-0.7679 upper=3.1066 effort=100.0 velocity=1.0
- added joint l_arm_j2_joint: type revolute, parent l_arm_j1_link, child l_arm_j2_link, origin xyz=0 0 0 rpy=1.57075 3.14159 1.57075, axis 0 0 1, limit lower=-0.2443 upper=1.9024 effort=100.0 velocity=1.0
- added joint l_arm_j3_joint: type revolute, parent l_arm_j2_link, child l_arm_j3_link, origin xyz=0 0 0 rpy=1.57075 1.57075 1.57075, axis 0 0 1, limit lower=-2.0769 upper=2.0769 effort=100.0 velocity=1.0
- added joint l_arm_j4_joint: type revolute, parent l_arm_j3_link, child l_arm_j4_link, origin xyz=-0.02 0.0 0.25 rpy=-1.57075 0 3.14159, axis 0 0 1, limit lower=-0.0174 upper=2.2514 effort=100.0 velocity=1.0
- added joint l_arm_j5_joint: type revolute, parent l_arm_j4_link, child l_arm_j5_link, origin xyz=-0.02 0.0 0.0 rpy=1.57075 0 0, axis 0 0 1, limit lower=-2.0769 upper=2.0769 effort=100.0 velocity=1.0
- added joint l_arm_j6_joint: type revolute, parent l_arm_j5_link, child l_arm_j6_link, origin xyz=0.0 0.0 0.28 rpy=-1.57075 1.57075 0, axis 0 0 1, limit lower=-0.2617 upper=0.7504 effort=100.0 velocity=1.0
- added joint l_arm_j7_joint: type revolute, parent l_arm_j6_link, child l_arm_j7_link, origin xyz=0.0 0.0 0 rpy=1.57075 3.14159 0, axis 0 0 1, limit lower=0 upper=0.5 effort=100.0 velocity=1.0
- added joint l_end_effector_joint: type fixed, parent l_gripper_link, child l_end_effector_link, origin xyz=0.05 0 0 rpy=0 0 0
- added joint l_gripper_joint: type fixed, parent l_arm_j7_link, child l_gripper_link, origin xyz=0.056 0 0 rpy=3.14159 3.14159 1.57075, axis 0 0 1
- added joint l_gripper_thumb_joint: type revolute, parent l_gripper_link, child l_gripper_thumb_link, origin xyz=0.027 0.042 0.0 rpy=0 0 0, axis 0 0 1, limit lower=-1.0122 upper=0.1396 effort=100.0 velocity=1.0
- added joint lumbar_lower_joint: type revolute, parent base_link, child lumbar_lower_link, origin xyz=0 0 0.4365 rpy=-1.57075 0 0, axis 0 0 1, limit lower=-0.2 upper=0.00872664625997165 effort=100.0 velocity=1.0
- added joint lumbar_upper_joint: type revolute, parent lumbar_lower_link, child lumbar_upper_link, origin xyz=0 -0.21 0 rpy=0 0 0, axis 0 0 1, limit lower=-0.00872664625997165 upper=2.10312174865317 effort=100.0 velocity=1.0
- added joint r_arm_j1_joint: type revolute, parent lumbar_upper_link, child r_arm_j1_link, origin xyz=-0.025 -0.480 -0.200 rpy=3.14159 0 0, axis 0 0 1, limit lower=-0.7679 upper=3.1066 effort=100.0 velocity=1.0
- added joint r_arm_j3_joint: type revolute, parent r_arm_j2_link, child r_arm_j3_link, origin xyz=0 0 0 rpy=1.57075 1.57075 1.57075, axis 0 0 1, limit lower=-2.0769 upper=2.0769 effort=100.0 velocity=1.0
- added joint r_arm_j4_joint: type revolute, parent r_arm_j3_link, child r_arm_j4_link, origin xyz=-0.02 0.0 0.25 rpy=-1.57075 0 3.14159, axis 0 0 1, limit lower=-0.0174 upper=2.2514 effort=100.0 velocity=1.0
- added joint r_arm_j5_joint: type revolute, parent r_arm_j4_link, child r_arm_j5_link, origin xyz=-0.02 0.0 0.0 rpy=1.57075 0 0, axis 0 0 1, limit lower=-2.0769 upper=2.0769 effort=100.0 velocity=1.0
- added joint r_arm_j6_joint: type revolute, parent r_arm_j5_link, child r_arm_j6_link, origin xyz=0.0 0.0 0.28 rpy=-1.57075 1.57075 0, axis 0 0 1, limit lower=-0.2617 upper=0.7504 effort=100.0 velocity=1.0
- added joint r_arm_j7_joint: type revolute, parent r_arm_j6_link, child r_arm_j7_link, origin xyz=0.0 0.0 0 rpy=1.57075 3.14159 0, axis 0 0 1, limit lower=-1.0122 upper=1.0 effort=100.0 velocity=1.0
- added joint r_armj2_joint: type revolute, parent r_arm_j1_link, child r_arm_j2_link, origin xyz=0 0 0 rpy=-1.57075 0 -1.57075, axis 0 0 1, limit lower=-1.9024 upper=0.2443 effort=100.0 velocity=1.0
- added joint r_end_effector_joint: type fixed, parent r_gripper_link, child r_end_effector_link, origin xyz=0 0.05 0 rpy=0 0 0
- added joint r_gripper_joint: type fixed, parent r_arm_j7_link, child r_gripper_link, origin xyz=0.056 0 0 rpy=3.14159 3.14159 3.14159, axis 0 0 1
- added joint r_gripper_thumb_joint: type revolute, parent r_gripper_link, child r_gripper_thumb_link, origin xyz=0.042 0.027 0.0 rpy=0 0 -1.57075, axis 0 0 1, limit lower=-0.1396 upper=1.0122 effort=100.0 velocity=1.0
- added joint smartpal5_x_joint: type prismatic, parent smartpal5_link, child smartpal5_x_link, origin xyz=0 0 0 rpy=0 0 0, limit lower=-5. upper=5. effort=1000.0 velocity=0.5
- added joint smartpal5_y_joint: type prismatic, parent smartpal5_x_link, child smartpal5_y_link, origin xyz=0 0 0 rpy=0 0 1.57075, limit lower=-5. upper=5. effort=1000.0 velocity=0.5
- added joint smartpal5_yaw_joint: type continuous, parent smartpal5_y_link, child base_footprint, origin xyz=0 0 0 rpy=0 0 -1.57075, axis 0 0 1
- added joint world_smartpal5_joint: type fixed, parent world_link, child smartpal5_link, origin xyz=0 0 0 rpy=0 0 0

File: tms_rp/rostms_description/urdf/all_components.urdf.xacro (robot description, xacro)
@@ -15,9 +15,9 @@
     <origin xyz="0 0 0" rpy="0 0 0"/>
   </joint>
-  <!-- <joint name="world_smartpal5_joint" type="fixed">
+  <joint name="world_smartpal5_joint" type="fixed">
 	  <parent link="world_link"/>
     <child link="smartpal5_link"/>
     <origin xyz="0 0 0" rpy="0 0 0"/>
-  </joint> -->
+  </joint>
   <!-- Defines the components tags -->
   <xacro:include filename="$(find rostms_description)/urdf/environments.urdf.xacro" />
@@ -25,5 +25,5 @@
   <xacro:include filename="$(find rostms_description)/urdf/objects.urdf.xacro" />
   <xacro:objects/>
-  <!-- <xacro:include filename="$(find rostms_description)/urdf/robots.urdf.xacro" />
-  <robots/> -->
+  <xacro:include filename="$(find rostms_description)/urdf/robots.urdf.xacro" />
+  <xacro:robots/>
 </robot>

File: tms_rp/rostms_description/urdf/robots.urdf.xacro (robot description, xacro)
@@ -6,5 +6,5 @@
   <xacro:macro name="robots">
     <xacro:include filename="$(find smartpal5_description)/urdf/smartpal5.urdf.xacro" />
-    <smartpal5_sim/>
+    <xacro:smartpal5_sim/>
   </xacro:macro>
 </robot>

Commit message: added rostms_moveit_config package

File: tms_rp/rostms_description/urdf/all_components.urdf (robot description, URDF)
Before this commit: robot rostms, 68 links, 67 joints
Links:
- removed link chair
- removed link meeting_chair1
- removed link meeting_chair2
- removed link meeting_chair3
- removed link meeting_chair4
- removed link refrigerator
- removed link wagon
- added link chair_link; visual mesh filename=package://environmental_model/model/chair.dae
- added link meeting_chair1_link; visual mesh filename=package://environmental_model/model/meeting_chair.dae
- added link meeting_chair2_link; visual mesh filename=package://environmental_model/model/meeting_chair.dae
- added link meeting_chair3_link; visual mesh filename=package://environmental_model/model/meeting_chair.dae
- added link meeting_chair4_link; visual mesh filename=package://environmental_model/model/meeting_chair.dae
- added link refrigerator_link; visual mesh filename=package://environmental_model/model/refrigerator.dae
- added link wagon_link; visual mesh filename=package://environmental_model/model/wagon.dae
Joints:
- joint chair_yaw_joint: child chair -> chair_link
- joint meeting_chair1_yaw_joint: child meeting_chair1 -> meeting_chair1_link
- joint meeting_chair2_yaw_joint: child meeting_chair2 -> meeting_chair2_link
- joint meeting_chair3_yaw_joint: child meeting_chair3 -> meeting_chair3_link
- joint meeting_chair4_yaw_joint: child meeting_chair4 -> meeting_chair4_link
- joint refrigerator_yaw_joint: child refrigerator -> refrigerator_link
- joint wagon_yaw_joint: child wagon -> wagon_link

File: tms_rp/rostms_description/urdf/objects.urdf.xacro (robot description, xacro)
@@ -5,5 +5,5 @@
   <xacro:include filename="$(find rostms_description)/urdf/objects_gazebo.urdf.xacro" />
   <!-- meeting_chair -->
-  <xacro:macro name="meeting_chair" params="num">
+  <xacro:macro name="meeting_chair_link" params="num">
     <link name="meeting_chair${num}_x_link"/>
     <joint name="meeting_chair${num}_x_joint" type="prismatic">
@@ -22,9 +22,9 @@
     <joint name="meeting_chair${num}_yaw_joint" type="continuous">
       <parent link="meeting_chair${num}_y_link"/>
-      <child link="meeting_chair${num}"/>
+      <child link="meeting_chair${num}_link"/>
       <origin xyz="0 0 0" rpy="0 0 0"/>
       <axis xyz="0 0 1"/>
     </joint>
-    <link name="meeting_chair${num}">
+    <link name="meeting_chair${num}_link">
       <visual>
         <geometry>
@@ -53,9 +53,9 @@
     <joint name="chair_yaw_joint" type="continuous">
       <parent link="chair_y_link"/>
-      <child link="chair"/>
+      <child link="chair_link"/>
       <origin xyz="0 0 0" rpy="0 0 0"/>
       <axis xyz="0 0 1"/>
     </joint>
-    <link name="chair">
+    <link name="chair_link">
       <visual>
         <geometry>
@@ -82,9 +82,9 @@
     <joint name="refrigerator_yaw_joint" type="continuous">
       <parent link="refrigerator_y_link"/>
-      <child link="refrigerator"/>
+      <child link="refrigerator_link"/>
       <origin xyz="0 0 0" rpy="0 0 0"/>
       <axis xyz="0 0 1"/>
     </joint>
-    <link name="refrigerator">
+    <link name="refrigerator_link">
       <visual>
         <geometry>
@@ -95,8 +95,8 @@
     </link>
     <!-- Add meeting_chair -->
-    <xacro:meeting_chair num="1"/>
-    <xacro:meeting_chair num="2"/>
-    <xacro:meeting_chair num="3"/>
-    <xacro:meeting_chair num="4"/>
+    <xacro:meeting_chair_link num="1"/>
+    <xacro:meeting_chair_link num="2"/>
+    <xacro:meeting_chair_link num="3"/>
+    <xacro:meeting_chair_link num="4"/>
     <!-- wagon -->
     <link name="wagon_x_link"/>
@@ -116,9 +116,9 @@
     <joint name="wagon_yaw_joint" type="continuous">
       <parent link="wagon_y_link"/>
-      <child link="wagon"/>
+      <child link="wagon_link"/>
       <origin xyz="0 0 0" rpy="0 0 0"/>
       <axis xyz="0 0 1"/>
     </joint>
-    <link name="wagon">
+    <link name="wagon_link">
       <visual>
         <geometry>

Commit message: added rostms_bringup package and modified sources related the moveit

File: tms_rp/rostms_description/urdf/all_components.urdf (robot description, URDF)
Before this commit: robot rostms, 68 links, 67 joints
Links:
- link bed_link: geometry collision box size=2.2 1.88 0.2; visual mesh filename=package://environmental_model/model/bed.dae
- link bsen_celling_link: geometry collision mesh filename=package://environmental_model/model/bsen_celling.dae; visual mesh filename=package://environmental_model/model/bsen_celling.dae
- link bsen_room_link: geometry collision box size=15.0 7.0 0.001; visual mesh filename=package://environmental_model/model/bsen.dae
- link bsen_wall_link: geometry collision mesh filename=package://environmental_model/model/bsen_wall.dae; visual mesh filename=package://environmental_model/model/bsen_wall.dae
- link carpet_link: geometry collision box size=1.76 2.55 0.01; visual mesh filename=package://environmental_model/model/carpet.dae
- link chair_link: geometry collision cylinder length=1.1 radius=0.35; visual mesh filename=package://environmental_model/model/chair.dae
- link drawer_link: geometry collision box size=0.6 0.4 0.6; visual mesh filename=package://environmental_model/model/drawer.dae
- link intelingent_shelf_link: geometry collision box size=0.3 0.5 0.9; visual mesh filename=package://environmental_model/model/intelingent_shelf.dae
- link kitchen_link: geometry collision box size=0.65 3.12 0.65; visual mesh filename=package://environmental_model/model/kitchen.dae
- link meeting_chair1_link: geometry collision cylinder length=0.8 radius=0.35; visual mesh filename=package://environmental_model/model/meeting_chair.dae
- link meeting_chair2_link: geometry collision cylinder length=0.8 radius=0.35; visual mesh filename=package://environmental_model/model/meeting_chair.dae
- link meeting_chair3_link: geometry collision cylinder length=0.8 radius=0.35; visual mesh filename=package://environmental_model/model/meeting_chair.dae
- link meeting_chair4_link: geometry collision cylinder length=0.8 radius=0.35; visual mesh filename=package://environmental_model/model/meeting_chair.dae
- link meeting_table_link: geometry collision cylinder length=0.73 radius=0.66; visual mesh filename=package://environmental_model/model/meeting_table.dae
- link recorder_link: geometry collision box size=0.25 0.45 0.1; visual mesh filename=package://environmental_model/model/recorder.dae
- link refrigerator_link: geometry collision box size=0.6 0.5 1.1; visual mesh filename=package://environmental_model/model/refrigerator.dae
- link sofa_link: geometry collision box size=0.8 2.35 0.77; visual mesh filename=package://environmental_model/model/sofa.dae
- link sofa_table_link: geometry collision box size=0.5 1.3 0.43; visual mesh filename=package://environmental_model/model/sofa_table.dae
- link tree_link: geometry collision cylinder length=1.0 radius=0.2; visual mesh filename=package://environmental_model/model/tree.dae
- link tv_52_link: geometry collision box size=1.2 0.1 0.7; visual mesh filename=package://environmental_model/model/tv_52.dae
- link tv_multi_link: geometry collision box size=2.5 0.2 1.4; visual mesh filename=package://environmental_model/model/tv_multi.dae
- link tv_table_link: geometry collision box size=0.35 2.7 0.35; visual mesh filename=package://environmental_model/model/tv_table.dae
- link wagon_link: geometry collision box size=0.6 0.4 0.7; visual mesh filename=package://environmental_model/model/wagon.dae
- link wardrobe_link: geometry collision box size=0.7 0.95 2.56; visual mesh filename=package://environmental_model/model/wardrobe.dae
- link workdesk_link: geometry collision box size=0.65 2.44 0.7; visual mesh filename=package://environmental_model/model/work_desk.dae
Joints:
- joint carpet_joint: origin xyz=9.9 2.9 0.1 rpy=0 0 0 -> xyz=9.9 2.9 0.01 rpy=0 0 0
