Commit message: modified subtask grasp

File: tms_rp/rostms_description/urdf/all_components.urdf (robot description, URDF)
Before this commit: robot rostms, 68 links, 67 joints
Links:
- added link chipstar_red_link; collision cylinder length=0.001 radius=0.001; visual mesh filename=package://environmental_model/model/chipstar_red.dae
- added link chipstar_red_x_link
- added link chipstar_red_y_link
- added link chipstar_red_z_link
Joints:
- removed joint l_arm_j5_joint
- added joint chipstar_red_x_joint: type prismatic, parent world_link, child chipstar_red_x_link, origin xyz=0 0 0 rpy=0 0 0, limit lower=0. upper=15. effort=1000.0 velocity=0.5
- added joint chipstar_red_y_joint: type prismatic, parent chipstar_red_x_link, child chipstar_red_y_link, origin xyz=0 0 0 rpy=0 0 1.57079633, limit lower=0. upper=8. effort=1000.0 velocity=0.5
- added joint chipstar_red_yaw_joint: type continuous, parent chipstar_red_z_link, child chipstar_red_link, origin xyz=0 0 0 rpy=0 1.57079633 0, axis 0 0 1
- added joint chipstar_red_z_joint: type prismatic, parent chipstar_red_y_link, child chipstar_red_z_link, origin xyz=0 0 0 rpy=0 -1.57079633 0, limit lower=0. upper=3. effort=1000.0 velocity=0.5
- added joint l_a     rm_j5_joint: type revolute, parent l_arm_j4_link, child l_arm_j5_link, origin xyz=-0.02 0.0 0.0 rpy=1.57075 0 0, axis 0 0 1, limit lower=-2.0769 upper=2.0769 effort=100.0 velocity=1.0

File: tms_rp/rostms_description/urdf/all_components_with_moveit.urdf (robot description, URDF)
Before this commit: robot rostms, 68 links, 67 joints
Links:
- added link chipstar_red_link; collision cylinder length=0.001 radius=0.001; visual mesh filename=package://environmental_model/model/chipstar_red.dae
- added link chipstar_red_x_link
- added link chipstar_red_y_link
- added link chipstar_red_z_link
Joints:
- added joint chipstar_red_x_joint: type prismatic, parent world_link, child chipstar_red_x_link, origin xyz=0 0 0 rpy=0 0 0, limit lower=0. upper=15. effort=1000.0 velocity=0.5
- added joint chipstar_red_y_joint: type prismatic, parent chipstar_red_x_link, child chipstar_red_y_link, origin xyz=0 0 0 rpy=0 0 1.57079633, limit lower=0. upper=8. effort=1000.0 velocity=0.5
- added joint chipstar_red_yaw_joint: type continuous, parent chipstar_red_z_link, child chipstar_red_link, origin xyz=0 0 0 rpy=0 1.57079633 0, axis 0 0 1
- added joint chipstar_red_z_joint: type prismatic, parent chipstar_red_y_link, child chipstar_red_z_link, origin xyz=0 0 0 rpy=0 -1.57079633 0, limit lower=0. upper=3. effort=1000.0 velocity=0.5

File: tms_rp/rostms_description/urdf/objects.urdf.xacro (robot description, xacro)
@@ -152,4 +152,46 @@
       </collision>
     </link>
+    <!-- object -->
+    <link name="chipstar_red_x_link"/>
+    <joint name="chipstar_red_x_joint" type="prismatic">
+      <parent link="world_link"/>
+      <child link="chipstar_red_x_link"/>
+      <origin rpy="0 0 0" xyz="0 0 0"/>
+      <limit effort="1000.0" lower="0." upper="15." velocity="0.5"/>
+    </joint>
+    <link name="chipstar_red_y_link"/>
+    <joint name="chipstar_red_y_joint" type="prismatic">
+      <parent link="chipstar_red_x_link"/>
+      <child link="chipstar_red_y_link"/>
+      <origin rpy="0 0 1.57079633" xyz="0 0 0"/>
+      <limit effort="1000.0" lower="0." upper="8." velocity="0.5"/>
+    </joint>
+    <link name="chipstar_red_z_link"/>
+    <joint name="chipstar_red_z_joint" type="prismatic">
+      <parent link="chipstar_red_y_link"/>
+      <child link="chipstar_red_z_link"/>
+      <origin rpy="0 -1.57079633 0" xyz="0 0 0"/>
+      <limit effort="1000.0" lower="0." upper="3." velocity="0.5"/>
+    </joint>
+    <joint name="chipstar_red_yaw_joint" type="continuous">
+      <parent link="chipstar_red_z_link"/>
+      <child link="chipstar_red_link"/>
+      <origin rpy="0 1.57079633 0" xyz="0 0 0"/>
+      <axis xyz="0 0 1"/>
+    </joint>
+    <link name="chipstar_red_link">
+      <visual>
+        <geometry>
+          <mesh filename="package://environmental_model/model/chipstar_red.dae"/>
+        </geometry>
+        <origin rpy="0 0 0" xyz="0. 0. 0."/>
+      </visual>
+    <collision>
+        <geometry>
+          <cylinder length="0.001" radius="0.001"/>
+        </geometry>
+        <origin rpy="0 0 0" xyz="0. 0. 0."/>
+      </collision>
+    </link>
     <objects_sim/>
   </xacro:macro>

Commit message: added roll pitch axis and changed chipstar_red model

File: tms_rp/rostms_description/urdf/all_components.urdf (robot description, URDF)
Before this commit: robot rostms, 72 links, 71 joints
Links:
- added link chipstar_red_pitch_link
- added link chipstar_red_yaw_link
- link chipstar_red_link: geometry visual mesh filename=package://environmental_model/model/chipstar_red.dae
Joints:
- added joint chipstar_red_pitch_joint: type continuous, parent chipstar_red_yaw_link, child chipstar_red_pitch_link, origin xyz=0 0 0 rpy=0 0 0, axis 0 1 0
- added joint chipstar_red_roll_joint: type continuous, parent chipstar_red_pitch_link, child chipstar_red_link, origin xyz=0 0 0 rpy=0 0 0, axis 1 0 0
- joint chipstar_red_yaw_joint: child chipstar_red_link -> chipstar_red_yaw_link; origin xyz=0 0 0 rpy=0 1.57079633 0 -> xyz=0 0 0 rpy=-1.57079633 0 -1.57079633

File: tms_rp/rostms_description/urdf/all_components_with_moveit.urdf (robot description, URDF)
Before this commit: robot rostms, 72 links, 71 joints
Links:
- added link chipstar_red_pitch_link
- added link chipstar_red_yaw_link
- link chipstar_red_link: geometry visual mesh filename=package://environmental_model/model/chipstar_red.dae
Joints:
- added joint chipstar_red_pitch_joint: type continuous, parent chipstar_red_yaw_link, child chipstar_red_pitch_link, origin xyz=0 0 0 rpy=0 0 0, axis 0 1 0
- added joint chipstar_red_roll_joint: type continuous, parent chipstar_red_pitch_link, child chipstar_red_link, origin xyz=0 0 0 rpy=0 0 0, axis 1 0 0
- joint chipstar_red_yaw_joint: child chipstar_red_link -> chipstar_red_yaw_link; origin xyz=0 0 0 rpy=0 1.57079633 0 -> xyz=0 0 0 rpy=-1.57079633 0 -1.57079633

File: tms_rp/rostms_description/urdf/objects.urdf.xacro (robot description, xacro)
@@ -174,9 +174,23 @@
       <limit effort="1000.0" lower="0." upper="3." velocity="0.5"/>
     </joint>
+    <link name="chipstar_red_yaw_link"/>
     <joint name="chipstar_red_yaw_joint" type="continuous">
       <parent link="chipstar_red_z_link"/>
+      <child link="chipstar_red_yaw_link"/>
+      <origin rpy="-1.57079633 0 -1.57079633" xyz="0 0 0"/>
+      <axis xyz="0 0 1"/>
+    </joint>
+    <link name="chipstar_red_pitch_link"/>
+    <joint name="chipstar_red_pitch_joint" type="continuous">
+      <parent link="chipstar_red_yaw_link"/>
+      <child link="chipstar_red_pitch_link"/>
+      <origin rpy="0 0 0" xyz="0 0 0"/>
+      <axis xyz="0 1 0"/>
+    </joint>
+    <joint name="chipstar_red_roll_joint" type="continuous">
+      <parent link="chipstar_red_pitch_link"/>
       <child link="chipstar_red_link"/>
-      <origin rpy="0 1.57079633 0" xyz="0 0 0"/>
-      <axis xyz="0 0 1"/>
+      <origin rpy="0 0 0" xyz="0 0 0"/>
+      <axis xyz="1 0 0"/>
     </joint>
     <link name="chipstar_red_link">
@@ -187,10 +201,4 @@
         <origin rpy="0 0 0" xyz="0. 0. 0."/>
       </visual>
-    <collision>
-        <geometry>
-          <cylinder length="0.001" radius="0.001"/>
-        </geometry>
-        <origin rpy="0 0 0" xyz="0. 0. 0."/>
-      </collision>
     </link>
     <objects_sim/>

Commit message: modified smartpalV model

File: tms_rp/rostms_description/urdf/all_components.urdf (robot description, URDF)
Before this commit: robot rostms, 74 links, 73 joints
Links:
- link bsen_celling_link: geometry collision mesh filename=package://environmental_model/model/bsen_celling.dae; visual mesh filename=package://environmental_model/model/bsen_celling.dae
- link bsen_room_link: mass 1 -> 100
- link bsen_wall_link: geometry collision mesh filename=package://environmental_model/model/bsen_wall.dae; visual mesh filename=package://environmental_model/model/bsen_wall.dae
- link kitchen_link: mass None -> 50
Joints:
- removed joint l_a     rm_j5_joint
- added joint l_arm_j5_joint: type revolute, parent l_arm_j4_link, child l_arm_j5_link, origin xyz=-0.02 0.0 0.0 rpy=1.57075 0 0, axis 0 0 -1, limit lower=-2.0769 upper=2.0769 effort=100.0 velocity=1.0
- joint l_arm_j2_joint: axis 0 0 1 -> 0 0 -1; limit lower=-0.2443 upper=1.9024 effort=100.0 velocity=1.0 -> lower=-1.9024 upper=0.2443 effort=100.0 velocity=1.0
- joint l_arm_j3_joint: axis 0 0 1 -> 0 0 -1
- joint r_arm_j7_joint: axis 0 0 1 -> 0 0 -1; limit lower=-1.0122 upper=1.0 effort=100.0 velocity=1.0 -> lower=-1.0 upper=1.0122 effort=100.0 velocity=1.0
- joint r_gripper_thumb_joint: axis 0 0 1 -> 0 0 -1; limit lower=-0.1396 upper=1.0122 effort=100.0 velocity=1.0 -> lower=-1.0122 upper=0.1396 effort=100.0 velocity=1.0

File: tms_rp/rostms_description/urdf/all_components_with_moveit.urdf (robot description, URDF)
Before this commit: robot rostms, 74 links, 73 joints
Links:
- link bsen_room_link: mass None -> 100
- link bsen_wall_link: geometry collision mesh filename=package://environmental_model/model/bsen_wall.dae; visual mesh filename=package://environmental_model/model/bsen_wall.dae
- link kitchen_link: mass None -> 50
Joints:
- joint l_arm_j2_joint: axis 0 0 1 -> 0 0 -1; limit lower=-0.2443 upper=1.9024 effort=100.0 velocity=1.0 -> lower=-1.9024 upper=0.2443 effort=100.0 velocity=1.0
- joint l_arm_j3_joint: axis 0 0 1 -> 0 0 -1
- joint l_arm_j5_joint: axis 0 0 1 -> 0 0 -1
- joint r_arm_j7_joint: axis 0 0 1 -> 0 0 -1; limit lower=-1.0122 upper=1.0 effort=100.0 velocity=1.0 -> lower=-1.0 upper=1.0122 effort=100.0 velocity=1.0
- joint r_gripper_thumb_joint: axis 0 0 1 -> 0 0 -1; limit lower=-0.1396 upper=1.0122 effort=100.0 velocity=1.0 -> lower=-1.0122 upper=0.1396 effort=100.0 velocity=1.0
- joint wall_joint: origin xyz=0 0 0 rpy=0 0 0 -> xyz=0. 0. 0. rpy=0 0 0

File: tms_rp/smartpal5_description/urdf/smartpal5.urdf (robot description, URDF)
Before this commit: robot smartpal5, 28 links, 27 joints
Joints:
- joint l_arm_j2_joint: axis 0 0 1 -> 0 0 -1; limit lower=-0.2443 upper=1.9024 effort=100.0 velocity=1.0 -> lower=-1.9024 upper=0.2443 effort=100.0 velocity=1.0
- joint l_arm_j3_joint: axis 0 0 1 -> 0 0 -1
- joint l_arm_j5_joint: axis 0 0 1 -> 0 0 -1
- joint r_arm_j7_joint: axis 0 0 1 -> 0 0 -1; limit lower=-1.0122 upper=1.0 effort=100.0 velocity=1.0 -> lower=-1.0 upper=1.0122 effort=100.0 velocity=1.0
- joint r_gripper_thumb_joint: axis 0 0 1 -> 0 0 -1; limit lower=-0.1396 upper=1.0122 effort=100.0 velocity=1.0 -> lower=-1.0122 upper=0.1396 effort=100.0 velocity=1.0

File: tms_rp/smartpal5_description/urdf/smartpal5.urdf.xacro (robot description, xacro)
@@ -162,6 +162,6 @@
 		<child link="l_arm_j2_link"/>
 		<origin xyz="0 0 0" rpy="1.57075 3.14159 1.57075"/>
-		<axis xyz="0 0 1"/>
-		<limit lower="-0.2443" upper="1.9024" effort="100.0" velocity="1.0"/>
+		<axis xyz="0 0 -1"/>
+		<limit lower="-1.9024" upper="0.2443" effort="100.0" velocity="1.0"/>
 	</joint>
 	<link name="l_arm_j2_link">
@@ -189,5 +189,5 @@
 		<child link="l_arm_j3_link"/>
 		<origin xyz="0 0 0" rpy="1.57075 1.57075 1.57075"/>
-		<axis xyz="0 0 1"/>
+		<axis xyz="0 0 -1"/>
 		<limit lower="-2.0769" upper="2.0769" effort="100.0" velocity="1.0"/>
 	</joint>
@@ -243,5 +243,5 @@
 		<child link="l_arm_j5_link"/>
 		<origin xyz="-0.02 0.0 0.0" rpy="1.57075 0 0"/>
-		<axis xyz="0 0 1"/>
+		<axis xyz="0 0 -1"/>
 		<limit lower="-2.0769" upper="2.0769" effort="100.0" velocity="1.0"/>
 	</joint>
@@ -560,6 +560,6 @@
 		<child link="r_arm_j7_link"/>
 		<origin xyz="0.0 0.0 0" rpy="1.57075 3.14159 0"/>
-		<axis xyz="0 0 1"/>
-		<limit lower="-1.0122" upper="1.0" effort="100.0" velocity="1.0"/>
+		<axis xyz="0 0 -1"/>
+		<limit lower="-1.0" upper="1.0122" effort="100.0" velocity="1.0"/>
 	</joint>
 	<link name="r_arm_j7_link">
@@ -633,6 +633,6 @@
 		<child link="r_gripper_thumb_link"/>
 		<origin xyz="0.042 0.027 0.0" rpy="0 0 -1.57075"/>
-		<axis xyz="0 0 1"/>
-		<limit lower="-0.1396" upper="1.0122" effort="100.0" velocity="1.0"/>
+		<axis xyz="0 0 -1"/>
+		<limit lower="-1.0122" upper="0.1396" effort="100.0" velocity="1.0"/>
   </joint>
 	<link name="r_gripper_thumb_link">

File: tms_rp/smartpal5_description/urdf/smartpal5_standalone.urdf (robot description, URDF)
Before this commit: robot smartpal5, 29 links, 28 joints
Joints:
- removed joint r_armj2_joint
- added joint r_arm_j2_joint: type revolute, parent r_arm_j1_link, child r_arm_j2_link, origin xyz=0 0 0 rpy=-1.57075 0 -1.57075, axis 0 0 1, limit lower=-1.9024 upper=0.2443 effort=100.0 velocity=1.0
- joint l_arm_j2_joint: axis 0 0 1 -> 0 0 -1; limit lower=-0.2443 upper=1.9024 effort=100.0 velocity=1.0 -> lower=-1.9024 upper=0.2443 effort=100.0 velocity=1.0
- joint l_arm_j3_joint: axis 0 0 1 -> 0 0 -1
- joint l_arm_j5_joint: axis 0 0 1 -> 0 0 -1
- joint l_end_effector_joint: origin xyz=0.05 0 0 rpy=0 0 0 -> xyz=0.01 0.11 0 rpy=0 0 0
- joint r_arm_j7_joint: axis 0 0 1 -> 0 0 -1; limit lower=-1.0122 upper=1.0 effort=100.0 velocity=1.0 -> lower=-1.0 upper=1.0122 effort=100.0 velocity=1.0
- joint r_end_effector_joint: origin xyz=0 0.05 0 rpy=0 0 0 -> xyz=0.11 0.01 0 rpy=0 0 0
- joint r_gripper_thumb_joint: axis 0 0 1 -> 0 0 -1; limit lower=-0.1396 upper=1.0122 effort=100.0 velocity=1.0 -> lower=-1.0122 upper=0.1396 effort=100.0 velocity=1.0
