Commit message: modified limit of smartpalV model

File: tms_rp/rostms_description/urdf/all_components.urdf (robot description, URDF)
Before this commit: robot rostms, 74 links, 73 joints
Joints:
- joint l_arm_j1_joint: limit lower=-0.7679 upper=3.1066 effort=100.0 velocity=1.0 -> lower=-0.76 upper=3.12 effort=100.0 velocity=1.0
- joint l_arm_j2_joint: limit lower=-1.9024 upper=0.2443 effort=100.0 velocity=1.0 -> lower=-1.8 upper=0.21 effort=100.0 velocity=1.0
- joint l_arm_j3_joint: limit lower=-2.0769 upper=2.0769 effort=100.0 velocity=1.0 -> lower=-2.0 upper=2.0 effort=100.0 velocity=1.0
- joint l_arm_j4_joint: limit lower=-0.0174 upper=2.2514 effort=100.0 velocity=1.0 -> lower=-0.0 upper=2.2 effort=100.0 velocity=1.0
- joint l_arm_j5_joint: limit lower=-2.0769 upper=2.0769 effort=100.0 velocity=1.0 -> lower=-2.0 upper=2.0 effort=100.0 velocity=1.0
- joint l_arm_j6_joint: limit lower=-0.2617 upper=0.7504 effort=100.0 velocity=1.0 -> lower=-0.25 upper=0.75 effort=100.0 velocity=1.0
- joint l_arm_j7_joint: limit lower=0 upper=0.5 effort=100.0 velocity=1.0 -> lower=-1.5 upper=0.8 effort=100.0 velocity=1.0
- joint r_arm_j1_joint: limit lower=-0.7679 upper=3.1066 effort=100.0 velocity=1.0 -> lower=-0.76 upper=3.12 effort=100.0 velocity=1.0
- joint r_arm_j2_joint: limit lower=-1.9024 upper=0.2443 effort=100.0 velocity=1.0 -> lower=-1.8 upper=0.21 effort=100.0 velocity=1.0
- joint r_arm_j3_joint: limit lower=-2.0769 upper=2.0769 effort=100.0 velocity=1.0 -> lower=-2.0 upper=2.0 effort=100.0 velocity=1.0
- joint r_arm_j4_joint: limit lower=-0.0174 upper=2.2514 effort=100.0 velocity=1.0 -> lower=-0.0 upper=2.2 effort=100.0 velocity=1.0
- joint r_arm_j5_joint: limit lower=-2.0769 upper=2.0769 effort=100.0 velocity=1.0 -> lower=-2.0 upper=2.0 effort=100.0 velocity=1.0
- joint r_arm_j6_joint: limit lower=-0.2617 upper=0.7504 effort=100.0 velocity=1.0 -> lower=-0.25 upper=0.75 effort=100.0 velocity=1.0
- joint r_arm_j7_joint: limit lower=-1.0 upper=1.0122 effort=100.0 velocity=1.0 -> lower=-1.5 upper=0.8 effort=100.0 velocity=1.0

File: tms_rp/rostms_description/urdf/all_components_with_moveit.urdf (robot description, URDF)
Before this commit: robot rostms, 74 links, 73 joints
Joints:
- joint l_arm_j1_joint: limit lower=-0.7679 upper=3.1066 effort=100.0 velocity=1.0 -> lower=-0.76 upper=3.12 effort=100.0 velocity=1.0
- joint l_arm_j2_joint: limit lower=-1.9024 upper=0.2443 effort=100.0 velocity=1.0 -> lower=-1.8 upper=0.21 effort=100.0 velocity=1.0
- joint l_arm_j3_joint: limit lower=-2.0769 upper=2.0769 effort=100.0 velocity=1.0 -> lower=-2.0 upper=2.0 effort=100.0 velocity=1.0
- joint l_arm_j4_joint: limit lower=-0.0174 upper=2.2514 effort=100.0 velocity=1.0 -> lower=-0.0 upper=2.2 effort=100.0 velocity=1.0
- joint l_arm_j5_joint: limit lower=-2.0769 upper=2.0769 effort=100.0 velocity=1.0 -> lower=-2.0 upper=2.0 effort=100.0 velocity=1.0
- joint l_arm_j6_joint: limit lower=-0.2617 upper=0.7504 effort=100.0 velocity=1.0 -> lower=-0.25 upper=0.75 effort=100.0 velocity=1.0
- joint l_arm_j7_joint: limit lower=0 upper=0.5 effort=100.0 velocity=1.0 -> lower=-1.5 upper=0.8 effort=100.0 velocity=1.0
- joint r_arm_j1_joint: limit lower=-0.7679 upper=3.1066 effort=100.0 velocity=1.0 -> lower=-0.76 upper=3.12 effort=100.0 velocity=1.0
- joint r_arm_j2_joint: limit lower=-1.9024 upper=0.2443 effort=100.0 velocity=1.0 -> lower=-1.8 upper=0.21 effort=100.0 velocity=1.0
- joint r_arm_j3_joint: limit lower=-2.0769 upper=2.0769 effort=100.0 velocity=1.0 -> lower=-2.0 upper=2.0 effort=100.0 velocity=1.0
- joint r_arm_j4_joint: limit lower=-0.0174 upper=2.2514 effort=100.0 velocity=1.0 -> lower=-0.0 upper=2.2 effort=100.0 velocity=1.0
- joint r_arm_j5_joint: limit lower=-2.0769 upper=2.0769 effort=100.0 velocity=1.0 -> lower=-2.0 upper=2.0 effort=100.0 velocity=1.0
- joint r_arm_j6_joint: limit lower=-0.2617 upper=0.7504 effort=100.0 velocity=1.0 -> lower=-0.25 upper=0.75 effort=100.0 velocity=1.0
- joint r_arm_j7_joint: limit lower=-1.0 upper=1.0122 effort=100.0 velocity=1.0 -> lower=-1.5 upper=0.8 effort=100.0 velocity=1.0

File: tms_rp/smartpal5_description/urdf/smartpal5.urdf (robot description, URDF)
Before this commit: robot smartpal5, 28 links, 27 joints
Joints:
- joint l_arm_j1_joint: limit lower=-0.7679 upper=3.1066 effort=100.0 velocity=1.0 -> lower=-0.76 upper=3.12 effort=100.0 velocity=1.0
- joint l_arm_j2_joint: limit lower=-1.9024 upper=0.2443 effort=100.0 velocity=1.0 -> lower=-1.8 upper=0.21 effort=100.0 velocity=1.0
- joint l_arm_j3_joint: limit lower=-2.0769 upper=2.0769 effort=100.0 velocity=1.0 -> lower=-2.0 upper=2.0 effort=100.0 velocity=1.0
- joint l_arm_j4_joint: limit lower=-0.0174 upper=2.2514 effort=100.0 velocity=1.0 -> lower=-0.0 upper=2.2 effort=100.0 velocity=1.0
- joint l_arm_j5_joint: limit lower=-2.0769 upper=2.0769 effort=100.0 velocity=1.0 -> lower=-2.0 upper=2.0 effort=100.0 velocity=1.0
- joint l_arm_j6_joint: limit lower=-0.2617 upper=0.7504 effort=100.0 velocity=1.0 -> lower=-0.25 upper=0.75 effort=100.0 velocity=1.0
- joint l_arm_j7_joint: limit lower=0 upper=0.5 effort=100.0 velocity=1.0 -> lower=-1.5 upper=0.8 effort=100.0 velocity=1.0
- joint r_arm_j1_joint: limit lower=-0.7679 upper=3.1066 effort=100.0 velocity=1.0 -> lower=-0.76 upper=3.12 effort=100.0 velocity=1.0
- joint r_arm_j2_joint: limit lower=-1.9024 upper=0.2443 effort=100.0 velocity=1.0 -> lower=-1.8 upper=0.21 effort=100.0 velocity=1.0
- joint r_arm_j3_joint: limit lower=-2.0769 upper=2.0769 effort=100.0 velocity=1.0 -> lower=-2.0 upper=2.0 effort=100.0 velocity=1.0
- joint r_arm_j4_joint: limit lower=-0.0174 upper=2.2514 effort=100.0 velocity=1.0 -> lower=-0.0 upper=2.2 effort=100.0 velocity=1.0
- joint r_arm_j5_joint: limit lower=-2.0769 upper=2.0769 effort=100.0 velocity=1.0 -> lower=-2.0 upper=2.0 effort=100.0 velocity=1.0
- joint r_arm_j6_joint: limit lower=-0.2617 upper=0.7504 effort=100.0 velocity=1.0 -> lower=-0.25 upper=0.75 effort=100.0 velocity=1.0
- joint r_arm_j7_joint: limit lower=-1.0 upper=1.0122 effort=100.0 velocity=1.0 -> lower=-1.5 upper=0.8 effort=100.0 velocity=1.0

File: tms_rp/smartpal5_description/urdf/smartpal5.urdf.xacro (robot description, xacro)
@@ -136,5 +136,5 @@
 		<origin xyz="-0.025 -0.480 0.200" rpy="3.14159 0 0"/>
 		<axis xyz="0 0 1"/>
-		<limit lower="-0.7679" upper="3.1066" effort="100.0" velocity="1.0"/>
+		<limit lower="-0.76" upper="3.12" effort="100.0" velocity="1.0"/>
 	</joint>
 	<link name="l_arm_j1_link">
@@ -163,5 +163,5 @@
 		<origin xyz="0 0 0" rpy="1.57075 3.14159 1.57075"/>
 		<axis xyz="0 0 -1"/>
-		<limit lower="-1.9024" upper="0.2443" effort="100.0" velocity="1.0"/>
+		<limit lower="-1.8" upper="0.21" effort="100.0" velocity="1.0"/>
 	</joint>
 	<link name="l_arm_j2_link">
@@ -190,5 +190,5 @@
 		<origin xyz="0 0 0" rpy="1.57075 1.57075 1.57075"/>
 		<axis xyz="0 0 -1"/>
-		<limit lower="-2.0769" upper="2.0769" effort="100.0" velocity="1.0"/>
+		<limit lower="-2.0" upper="2.0" effort="100.0" velocity="1.0"/>
 	</joint>
 	<link name="l_arm_j3_link">
@@ -217,5 +217,5 @@
 		<origin xyz="-0.02 0.0 0.25" rpy="-1.57075 0 3.14159"/>
 		<axis xyz="0 0 1"/>
-		<limit lower="-0.0174" upper="2.2514" effort="100.0" velocity="1.0"/>
+		<limit lower="-0.0" upper="2.2" effort="100.0" velocity="1.0"/>
 	</joint>
 	<link name="l_arm_j4_link">
@@ -244,5 +244,5 @@
 		<origin xyz="-0.02 0.0 0.0" rpy="1.57075 0 0"/>
 		<axis xyz="0 0 -1"/>
-		<limit lower="-2.0769" upper="2.0769" effort="100.0" velocity="1.0"/>
+		<limit lower="-2.0" upper="2.0" effort="100.0" velocity="1.0"/>
 	</joint>
 	<link name="l_arm_j5_link">
@@ -271,5 +271,5 @@
 		<origin xyz="0.0 0.0 0.28" rpy="-1.57075 1.57075 0"/>
 		<axis xyz="0 0 1"/>
-		<limit lower="-0.2617" upper="0.7504" effort="100.0" velocity="1.0"/>
+		<limit lower="-0.25" upper="0.75" effort="100.0" velocity="1.0"/>
 	</joint>
 	<link name="l_arm_j6_link">
@@ -298,5 +298,5 @@
 		<origin xyz="0.0 0.0 0" rpy="1.57075 3.14159 0"/>
 		<axis xyz="0 0 1"/>
-		<limit lower="0" upper="0.5" effort="100.0" velocity="1.0"/>
+		<limit lower="-1.5" upper="0.8" effort="100.0" velocity="1.0"/>
 	</joint>
 	<link name="l_arm_j7_link">
@@ -399,5 +399,5 @@
 		<origin xyz="-0.025 -0.480 -0.200" rpy="3.14159 0 0"/>
 		<axis xyz="0 0 1"/>
-		<limit lower="-0.7679" upper="3.1066" effort="100.0" velocity="1.0"/>
+		<limit lower="-0.76" upper="3.12" effort="100.0" velocity="1.0"/>
 	</joint>
 	<link name="r_arm_j1_link">
@@ -426,5 +426,5 @@
 		<origin xyz="0 0 0" rpy="-1.57075 0 -1.57075"/>
 		<axis xyz="0 0 1"/>
-		<limit lower="-1.9024" upper="0.2443" effort="100.0" velocity="1.0"/>
+		<limit lower="-1.8" upper="0.21" effort="100.0" velocity="1.0"/>
 	</joint>
 	<link name="r_arm_j2_link">
@@ -453,5 +453,5 @@
 		<origin xyz="0 0 0" rpy="1.57075 1.57075 1.57075"/>
 		<axis xyz="0 0 1"/>
-		<limit lower="-2.0769" upper="2.0769" effort="100.0" velocity="1.0"/>
+		<limit lower="-2.0" upper="2.0" effort="100.0" velocity="1.0"/>
 	</joint>
 	<link name="r_arm_j3_link">
@@ -480,5 +480,5 @@
 		<origin xyz="-0.02 0.0 0.25" rpy="-1.57075 0 3.14159"/>
 		<axis xyz="0 0 1"/>
-		<limit lower="-0.0174" upper="2.2514" effort="100.0" velocity="1.0"/>
+		<limit lower="-0.0" upper="2.2" effort="100.0" velocity="1.0"/>
 	</joint>
 	<link name="r_arm_j4_link">
@@ -507,5 +507,5 @@
 		<origin xyz="-0.02 0.0 0.0" rpy="1.57075 0 0"/>
 		<axis xyz="0 0 1"/>
-		<limit lower="-2.0769" upper="2.0769" effort="100.0" velocity="1.0"/>
+		<limit lower="-2.0" upper="2.0" effort="100.0" velocity="1.0"/>
 	</joint>
 	<link name="r_arm_j5_link">
@@ -534,5 +534,5 @@
 		<origin xyz="0.0 0.0 0.28" rpy="-1.57075 1.57075 0"/>
 		<axis xyz="0 0 1"/>
-		<limit lower="-0.2617" upper="0.7504" effort="100.0" velocity="1.0"/>
+		<limit lower="-0.25" upper="0.75" effort="100.0" velocity="1.0"/>
 	</joint>
 	<link name="r_arm_j6_link">
@@ -561,5 +561,5 @@
 		<origin xyz="0.0 0.0 0" rpy="1.57075 3.14159 0"/>
 		<axis xyz="0 0 -1"/>
-		<limit lower="-1.0" upper="1.0122" effort="100.0" velocity="1.0"/>
+		<limit lower="-1.5" upper="0.8" effort="100.0" velocity="1.0"/>
 	</joint>
 	<link name="r_arm_j7_link">

File: tms_rp/smartpal5_description/urdf/smartpal5_standalone.urdf (robot description, URDF)
Before this commit: robot smartpal5, 29 links, 28 joints
Joints:
- joint l_arm_j1_joint: limit lower=-0.7679 upper=3.1066 effort=100.0 velocity=1.0 -> lower=-0.76 upper=3.12 effort=100.0 velocity=1.0
- joint l_arm_j2_joint: limit lower=-1.9024 upper=0.2443 effort=100.0 velocity=1.0 -> lower=-1.8 upper=0.21 effort=100.0 velocity=1.0
- joint l_arm_j3_joint: limit lower=-2.0769 upper=2.0769 effort=100.0 velocity=1.0 -> lower=-2.0 upper=2.0 effort=100.0 velocity=1.0
- joint l_arm_j4_joint: limit lower=-0.0174 upper=2.2514 effort=100.0 velocity=1.0 -> lower=-0.0 upper=2.2 effort=100.0 velocity=1.0
- joint l_arm_j5_joint: limit lower=-2.0769 upper=2.0769 effort=100.0 velocity=1.0 -> lower=-2.0 upper=2.0 effort=100.0 velocity=1.0
- joint l_arm_j6_joint: limit lower=-0.2617 upper=0.7504 effort=100.0 velocity=1.0 -> lower=-0.25 upper=0.75 effort=100.0 velocity=1.0
- joint l_arm_j7_joint: limit lower=0 upper=0.5 effort=100.0 velocity=1.0 -> lower=-1.5 upper=0.8 effort=100.0 velocity=1.0
- joint r_arm_j1_joint: limit lower=-0.7679 upper=3.1066 effort=100.0 velocity=1.0 -> lower=-0.76 upper=3.12 effort=100.0 velocity=1.0
- joint r_arm_j2_joint: limit lower=-1.9024 upper=0.2443 effort=100.0 velocity=1.0 -> lower=-1.8 upper=0.21 effort=100.0 velocity=1.0
- joint r_arm_j3_joint: limit lower=-2.0769 upper=2.0769 effort=100.0 velocity=1.0 -> lower=-2.0 upper=2.0 effort=100.0 velocity=1.0
- joint r_arm_j4_joint: limit lower=-0.0174 upper=2.2514 effort=100.0 velocity=1.0 -> lower=-0.0 upper=2.2 effort=100.0 velocity=1.0
- joint r_arm_j5_joint: limit lower=-2.0769 upper=2.0769 effort=100.0 velocity=1.0 -> lower=-2.0 upper=2.0 effort=100.0 velocity=1.0
- joint r_arm_j6_joint: limit lower=-0.2617 upper=0.7504 effort=100.0 velocity=1.0 -> lower=-0.25 upper=0.75 effort=100.0 velocity=1.0
- joint r_arm_j7_joint: limit lower=-1.0 upper=1.0122 effort=100.0 velocity=1.0 -> lower=-1.5 upper=0.8 effort=100.0 velocity=1.0

Commit message: [add]: show mimamorukun by vicon. but mesh data is refrigetor now :(

File: tms_rp/rostms_description/urdf/all_components.urdf (robot description, URDF)
Before this commit: robot rostms, 68 links, 67 joints
Links:
- added link wheelchair_link; collision box size=0.6 0.5 1.1; visual mesh filename=package://environmental_model/model/refrigerator.dae
- added link wheelchair_x_link
- added link wheelchair_y_link
- link bsen_celling_link: geometry collision mesh filename=package://environmental_model/model/bsen_celling.dae; visual mesh filename=package://environmental_model/model/bsen_celling.dae
- link bsen_room_link: mass 1 -> 100
- link bsen_wall_link: geometry collision mesh filename=package://environmental_model/model/bsen_wall.dae; visual mesh filename=package://environmental_model/model/bsen_wall.dae
- link kitchen_link: mass None -> 50
Joints:
- added joint wheelchair_x_joint: type prismatic, parent world_link, child wheelchair_x_link, origin xyz=0 0 0 rpy=0 0 0, limit lower=0. upper=15. effort=1000.0 velocity=5.0
- added joint wheelchair_y_joint: type prismatic, parent wheelchair_x_link, child wheelchair_y_link, origin xyz=0 0 0 rpy=0 0 1.57079633, limit lower=0. upper=8. effort=1000.0 velocity=5.0
- added joint wheelchair_yaw_joint: type continuous, parent wheelchair_y_link, child wheelchair_link, origin xyz=0 0 0 rpy=0 0 0, axis 0 0 1

File: tms_rp/rostms_description/urdf/robots.urdf.xacro (robot description, xacro)
@@ -4,7 +4,8 @@
   <!-- Import all Gazebo-customization elements, including Gazebo colors -->
   <xacro:include filename="$(find smartpal5_description)/urdf/smartpal5_gazebo.urdf.xacro" />
+    <xacro:robots_sim/>
   <xacro:macro name="robots">
     <xacro:include filename="$(find smartpal5_description)/urdf/smartpal5.urdf.xacro" />
-    <xacro:robots_sim/>
+    <xacro:include filename="$(find tms_rc_mimamorukun_control)/urdf/wheelchair.urdf.xacro" />
   </xacro:macro>
 </robot>
