Commit message: [add] greentea_bottle,cancoffee,soysauce_bottle_black but dont appear now ;(

File: tms_rp/rostms_description/urdf/all_components.urdf (robot description, URDF)
Before this commit: robot rostms, 74 links, 73 joints
Links:
- removed link recorder_link
- removed link tv_52_link
- added link cancoffee_link; visual mesh filename=package://environmental_model/model/cancoffee.dae
- added link cancoffee_pitch_link
- added link cancoffee_x_link
- added link cancoffee_y_link
- added link cancoffee_yaw_link
- added link cancoffee_z_link
- added link greentea_bottle_link; visual mesh filename=package://environmental_model/model/greentea_bottle.dae
- added link greentea_bottle_pitch_link
- added link greentea_bottle_x_link
- added link greentea_bottle_y_link
- added link greentea_bottle_yaw_link
- added link greentea_bottle_z_link
- added link soysauce_bottle_black_link; visual mesh filename=package://environmental_model/model/soysauce_bottle_black.d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
- added link soysauce_bottle_black_pitch_link
- added link soysauce_bottle_black_x_link
- added link soysauce_bottle_black_y_link
- added link soysauce_bottle_black_yaw_link
- added link soysauce_bottle_black_z_link
- link bed_link: geometry collision box size=0.5 1.3 0.43; visual mesh filename=package://environmental_model/model/paramount_bed.dae
Joints:
- removed joint recorder_joint
- removed joint tv_52_link
- added joint cancoffee_pitch_joint: type continuous, parent cancoffee_yaw_link, child cancoffee_pitch_link, origin xyz=0 0 0 rpy=0 0 0, axis 0 1 0
- added joint cancoffee_roll_joint: type continuous, parent cancoffee_pitch_link, child cancoffee_link, origin xyz=0 0 0 rpy=0 0 0, axis 1 0 0
- added joint cancoffee_x_joint: type prismatic, parent world_link, child cancoffee_x_link, origin xyz=0 0 0 rpy=0 0 0, limit lower=0. upper=15. effort=1000.0 velocity=0.5
- added joint cancoffee_y_joint: type prismatic, parent cancoffee_x_link, child cancoffee_y_link, origin xyz=0 0 0 rpy=0 0 1.57079633, limit lower=0. upper=8. effort=1000.0 velocity=0.5
- added joint cancoffee_yaw_joint: type continuous, parent cancoffee_z_link, child cancoffee_yaw_link, origin xyz=0 0 0 rpy=-1.57079633 0 -1.57079633, axis 0 0 1
- added joint cancoffee_z_joint: type prismatic, parent cancoffee_y_link, child cancoffee_z_link, origin xyz=0 0 0 rpy=0 -1.57079633 0, limit lower=0. upper=3. effort=1000.0 velocity=0.5
- added joint greentea_bottle_pitch_joint: type continuous, parent greentea_bottle_yaw_link, child greentea_bottle_pitch_link, origin xyz=0 0 0 rpy=0 0 0, axis 0 1 0
- added joint greentea_bottle_roll_joint: type continuous, parent greentea_bottle_pitch_link, child greentea_bottle_link, origin xyz=0 0 0 rpy=0 0 0, axis 1 0 0
- added joint greentea_bottle_x_joint: type prismatic, parent world_link, child greentea_bottle_x_link, origin xyz=0 0 0 rpy=0 0 0, limit lower=0. upper=15. effort=1000.0 velocity=0.5
- added joint greentea_bottle_y_joint: type prismatic, parent greentea_bottle_x_link, child greentea_bottle_y_link, origin xyz=0 0 0 rpy=0 0 1.57079633, limit lower=0. upper=8. effort=1000.0 velocity=0.5
- added joint greentea_bottle_yaw_joint: type continuous, parent greentea_bottle_z_link, child greentea_bottle_yaw_link, origin xyz=0 0 0 rpy=-1.57079633 0 -1.57079633, axis 0 0 1
- added joint greentea_bottle_z_joint: type prismatic, parent greentea_bottle_y_link, child greentea_bottle_z_link, origin xyz=0 0 0 rpy=0 -1.57079633 0, limit lower=0. upper=3. effort=1000.0 velocity=0.5
- added joint soysauce_bottle_black_pitch_joint: type continuous, parent soysauce_bottle_black_yaw_link, child soysauce_bottle_black_pitch_link, origin xyz=0 0 0 rpy=0 0 0, axis 0 1 0
- added joint soysauce_bottle_black_roll_joint: type continuous, parent soysauce_bottle_black_pitch_link, child soysauce_bottle_black_link, origin xyz=0 0 0 rpy=0 0 0, axis 1 0 0
- added joint soysauce_bottle_black_x_joint: type prismatic, parent world_link, child soysauce_bottle_black_x_link, origin xyz=0 0 0 rpy=0 0 0, limit lower=0. upper=15. effort=1000.0 velocity=0.5
- added joint soysauce_bottle_black_y_joint: type prismatic, parent soysauce_bottle_black_x_link, child soysauce_bottle_black_y_link, origin xyz=0 0 0 rpy=0 0 1.57079633, limit lower=0. upper=8. effort=1000.0 velocity=0.5
- added joint soysauce_bottle_black_yaw_joint: type continuous, parent soysauce_bottle_black_z_link, child soysauce_bottle_black_yaw_link, origin xyz=0 0 0 rpy=-1.57079633 0 -1.57079633, axis 0 0 1
- added joint soysauce_bottle_black_z_joint: type prismatic, parent soysauce_bottle_black_y_link, child soysauce_bottle_black_z_link, origin xyz=0 0 0 rpy=0 -1.57079633 0, limit lower=0. upper=3. effort=1000.0 velocity=0.5
- joint bed_joint: origin xyz=12.48 2.3 0.2075 rpy=0 0 0 -> xyz=10.35 2.7 0.235 rpy=0 0 0
- joint carpet_joint: origin xyz=9.9 2.9 0.01 rpy=0 0 0 -> xyz=12.3 2.6 0.01 rpy=0 0 0
- joint drawer_joint: origin xyz=12.93 5.8 0.303 rpy=0 0 -1.57079633 -> xyz=12.72 5.8 0.303 rpy=0 0 -1.57079633
- joint intelingent_shelf_joint: origin xyz=11.56 3.520 0.445 rpy=0 0 0 -> xyz=11.48 4.220 0.445 rpy=0 0 0
- joint kitchen_joint: origin xyz=9.26 5.9 0.4855 rpy=0 0 -1.57079633 -> xyz=9.05 5.87 0.4855 rpy=0 0 -1.57079633
- joint sofa_joint: origin xyz=9.1 2.9 0.395 rpy=0 0 0 -> xyz=11.75 2.6 0.395 rpy=0 0 0
- joint sofa_table_joint: origin xyz=10.2 2.9 0.235 rpy=0 0 0 -> xyz=12.7 2.5 0.235 rpy=0 0 0
- joint tv_multi_joint: origin xyz=14.37 2.2 1.0 rpy=0 0 -1.57079633 -> xyz=14.37 2.2 1.45 rpy=0 0 -1.57079633
- joint tv_table_joint: origin xyz=11.1 2.9 0.175 rpy=0 0 0 -> xyz=14.25 2.5 0.175 rpy=0 0 0
- joint wardrobe_joint: origin xyz=13.7 5.9 1.3 rpy=0 0 -1.57079633 -> xyz=13.46 5.9 1.3 rpy=0 0 -1.57079633
- joint workdesk_joint: origin xyz=12.05 5.9 0.5 rpy=0 0 -1.57079633 -> xyz=11.80 5.9 0.5 rpy=0 0 -1.57079633

File: tms_rp/rostms_description/urdf/objects.urdf.xacro (robot description, xacro)
@@ -153,4 +153,5 @@
     </link>
     <!-- object -->
+    <!-- chipstar_red -->
     <link name="chipstar_red_x_link"/>
     <joint name="chipstar_red_x_joint" type="prismatic">
@@ -202,4 +203,154 @@
       </visual>
     </link>
+    <!-- greentea_bottle -->
+    <link name="greentea_bottle_x_link"/>
+    <joint name="greentea_bottle_x_joint" type="prismatic">
+      <parent link="world_link"/>
+      <child link="greentea_bottle_x_link"/>
+      <origin rpy="0 0 0" xyz="0 0 0"/>
+      <limit effort="1000.0" lower="0." upper="15." velocity="0.5"/>
+    </joint>
+    <link name="greentea_bottle_y_link"/>
+    <joint name="greentea_bottle_y_joint" type="prismatic">
+      <parent link="greentea_bottle_x_link"/>
+      <child link="greentea_bottle_y_link"/>
+      <origin rpy="0 0 1.57079633" xyz="0 0 0"/>
+      <limit effort="1000.0" lower="0." upper="8." velocity="0.5"/>
+    </joint>
+    <link name="greentea_bottle_z_link"/>
+    <joint name="greentea_bottle_z_joint" type="prismatic">
+      <parent link="greentea_bottle_y_link"/>
+      <child link="greentea_bottle_z_link"/>
+      <origin rpy="0 -1.57079633 0" xyz="0 0 0"/>
+      <limit effort="1000.0" lower="0." upper="3." velocity="0.5"/>
+    </joint>
+    <link name="greentea_bottle_yaw_link"/>
+    <joint name="greentea_bottle_yaw_joint" type="continuous">
+      <parent link="greentea_bottle_z_link"/>
+      <child link="greentea_bottle_yaw_link"/>
+      <origin rpy="-1.57079633 0 -1.57079633" xyz="0 0 0"/>
+      <axis xyz="0 0 1"/>
+    </joint>
+    <link name="greentea_bottle_pitch_link"/>
+    <joint name="greentea_bottle_pitch_joint" type="continuous">
+      <parent link="greentea_bottle_yaw_link"/>
+      <child link="greentea_bottle_pitch_link"/>
+      <origin rpy="0 0 0" xyz="0 0 0"/>
+      <axis xyz="0 1 0"/>
+    </joint>
+    <joint name="greentea_bottle_roll_joint" type="continuous">
+      <parent link="greentea_bottle_pitch_link"/>
+      <child link="greentea_bottle_link"/>
+      <origin rpy="0 0 0" xyz="0 0 0"/>
+      <axis xyz="1 0 0"/>
+    </joint>
+    <link name="greentea_bottle_link">
+      <visual>
+        <geometry>
+          <mesh filename="package://environmental_model/model/greentea_bottle.dae"/>
+        </geometry>
+        <origin rpy="0 0 0" xyz="0. 0. 0."/>
+      </visual>
+    </link>
+    <!-- cancoffee -->
+    <link name="cancoffee_x_link"/>
+    <joint name="cancoffee_x_joint" type="prismatic">
+      <parent link="world_link"/>
+      <child link="cancoffee_x_link"/>
+      <origin rpy="0 0 0" xyz="0 0 0"/>
+      <limit effort="1000.0" lower="0." upper="15." velocity="0.5"/>
+    </joint>
+    <link name="cancoffee_y_link"/>
+    <joint name="cancoffee_y_joint" type="prismatic">
+      <parent link="cancoffee_x_link"/>
+      <child link="cancoffee_y_link"/>
+      <origin rpy="0 0 1.57079633" xyz="0 0 0"/>
+      <limit effort="1000.0" lower="0." upper="8." velocity="0.5"/>
+    </joint>
+    <link name="cancoffee_z_link"/>
+    <joint name="cancoffee_z_joint" type="prismatic">
+      <parent link="cancoffee_y_link"/>
+      <child link="cancoffee_z_link"/>
+      <origin rpy="0 -1.57079633 0" xyz="0 0 0"/>
+      <limit effort="1000.0" lower="0." upper="3." velocity="0.5"/>
+    </joint>
+    <link name="cancoffee_yaw_link"/>
+    <joint name="cancoffee_yaw_joint" type="continuous">
+      <parent link="cancoffee_z_link"/>
+      <child link="cancoffee_yaw_link"/>
+      <origin rpy="-1.57079633 0 -1.57079633" xyz="0 0 0"/>
+      <axis xyz="0 0 1"/>
+    </joint>
+    <link name="cancoffee_pitch_link"/>
+    <joint name="cancoffee_pitch_joint" type="continuous">
+      <parent link="cancoffee_yaw_link"/>
+      <child link="cancoffee_pitch_link"/>
+      <origin rpy="0 0 0" xyz="0 0 0"/>
+      <axis xyz="0 1 0"/>
+    </joint>
+    <joint name="cancoffee_roll_joint" type="continuous">
+      <parent link="cancoffee_pitch_link"/>
+      <child link="cancoffee_link"/>
+      <origin rpy="0 0 0" xyz="0 0 0"/>
+      <axis xyz="1 0 0"/>
+    </joint>
+    <link name="cancoffee_link">
+      <visual>
+        <geometry>
+          <mesh filename="package://environmental_model/model/cancoffee.dae"/>
+        </geometry>
+        <origin rpy="0 0 0" xyz="0. 0. 0."/>
+      </visual>
+    </link>
+    <!-- soysauce_bottle_black -->
+    <link name="soysauce_bottle_black_x_link"/>
+    <joint name="soysauce_bottle_black_x_joint" type="prismatic">
+      <parent link="world_link"/>
+      <child link="soysauce_bottle_black_x_link"/>
+      <origin rpy="0 0 0" xyz="0 0 0"/>
+      <limit effort="1000.0" lower="0." upper="15." velocity="0.5"/>
+    </joint>
+    <link name="soysauce_bottle_black_y_link"/>
+    <joint name="soysauce_bottle_black_y_joint" type="prismatic">
+      <parent link="soysauce_bottle_black_x_link"/>
+      <child link="soysauce_bottle_black_y_link"/>
+      <origin rpy="0 0 1.57079633" xyz="0 0 0"/>
+      <limit effort="1000.0" lower="0." upper="8." velocity="0.5"/>
+    </joint>
+    <link name="soysauce_bottle_black_z_link"/>
+    <joint name="soysauce_bottle_black_z_joint" type="prismatic">
+      <parent link="soysauce_bottle_black_y_link"/>
+      <child link="soysauce_bottle_black_z_link"/>
+      <origin rpy="0 -1.57079633 0" xyz="0 0 0"/>
+      <limit effort="1000.0" lower="0." upper="3." velocity="0.5"/>
+    </joint>
+    <link name="soysauce_bottle_black_yaw_link"/>
+    <joint name="soysauce_bottle_black_yaw_joint" type="continuous">
+      <parent link="soysauce_bottle_black_z_link"/>
+      <child link="soysauce_bottle_black_yaw_link"/>
+      <origin rpy="-1.57079633 0 -1.57079633" xyz="0 0 0"/>
+      <axis xyz="0 0 1"/>
+    </joint>
+    <link name="soysauce_bottle_black_pitch_link"/>
+    <joint name="soysauce_bottle_black_pitch_joint" type="continuous">
+      <parent link="soysauce_bottle_black_yaw_link"/>
+      <child link="soysauce_bottle_black_pitch_link"/>
+      <origin rpy="0 0 0" xyz="0 0 0"/>
+      <axis xyz="0 1 0"/>
+    </joint>
+    <joint name="soysauce_bottle_black_roll_joint" type="continuous">
+      <parent link="soysauce_bottle_black_pitch_link"/>
+      <child link="soysauce_bottle_black_link"/>
+      <origin rpy="0 0 0" xyz="0 0 0"/>
+      <axis xyz="1 0 0"/>
+    </joint>
+    <link name="soysauce_bottle_black_link">
+      <visual>
+        <geometry>
+          <mesh filename="package://environmental_model/model/soysauce_bottle_black.dae"/>
+        </geometry>
+        <origin rpy="0 0 0" xyz="0. 0. 0."/>
+      </visual>
+    </link>
     <objects_sim/>
   </xacro:macro>

Commit message: update get_object task

File: tms_rp/rostms_description/urdf/all_components.urdf (robot description, URDF)
Before this commit: robot rostms, 93 links, 92 joints
Links:
- removed link refrigerator_x_link
- removed link refrigerator_y_link
- link bed_link: geometry collision box size=1.95 0.82 0.38; visual mesh filename=package://environmental_model/model/paramount_bed.dae
- link refrigerator_link: geometry collision box size=0.3 0.5 0.9; visual mesh filename=package://environmental_model/model/refrigerator.dae
- link wheelchair_link: geometry collision box size=0.6 0.5 1.1; visual mesh filename=package://environmental_model/model/wheelchair.dae
Joints:
- removed joint refrigerator_x_joint
- removed joint refrigerator_y_joint
- removed joint refrigerator_yaw_joint
- added joint refrigerator_joint: type fixed, parent bsen_room_link, child refrigerator_link, origin xyz=7.0 5.52 0.0 rpy=0 0 -1.57079633
- joint intelingent_shelf_joint: origin xyz=11.48 4.220 0.445 rpy=0 0 0 -> xyz=11.65 3.970 0.005 rpy=0 0 0
- joint kitchen_joint: origin xyz=9.05 5.87 0.4855 rpy=0 0 -1.57079633 -> xyz=9.03 5.87 0.4855 rpy=0 0 -1.57079633
- joint workdesk_joint: origin xyz=11.80 5.9 0.5 rpy=0 0 -1.57079633 -> xyz=11.80 5.9 0.35 rpy=0 0 -1.57079633

File: tms_rp/rostms_description/urdf/all_components_with_moveit.urdf (robot description, URDF)
Before this commit: robot rostms, 91 links, 90 joints
Links:
- link bed_link: geometry collision box size=1.95 0.82 0.38; visual mesh filename=package://environmental_model/model/paramount_bed.dae

File: tms_rp/rostms_description/urdf/environments.urdf.xacro (robot description, xacro)
@@ -186,5 +186,5 @@
       <collision>
         <geometry>
-          <box size="0.5 1.3 0.43"/>
+          <box size="1.95 0.82 0.38"/>
         </geometry>
       </collision>

Commit message: get_object from refrigerator

File: tms_rp/rostms_description/urdf/all_components.urdf (robot description, URDF)
Before this commit: robot rostms, 91 links, 90 joints
Links:
- link refrigerator_link: geometry visual mesh filename=package://environmental_model/model/refrigerator.dae

File: tms_rp/rostms_description/urdf/all_components_with_moveit.urdf (robot description, URDF)
Before this commit: robot rostms, 91 links, 90 joints
Links:
- link refrigerator_link: geometry visual mesh filename=package://environmental_model/model/refrigerator.dae

File: tms_rp/rostms_description/urdf/environments.urdf.xacro (robot description, xacro)
@@ -303,9 +303,4 @@
         </geometry>
       </visual>
-      <collision>
-        <geometry>
-          <box size="0.3 0.5 0.9"/>
-        </geometry>
-      </collision>
     </link>
     <xacro:environments_sim/>
