Commit message: cleanup the rostms_description package

File: tms_rp/rostms_description/urdf/environments.urdf.xacro (robot description, xacro)
@@ -2,6 +2,4 @@
 <!-- Environment of ROS-TMS project room -->
 <robot name="environment" xmlns:xacro="http://www.ros.org/wiki/xacro">
-  <!-- Import common properties -->
-  <xacro:include filename="$(find environment_description)/urdf/common_properties.urdf.xacro" />
   <!-- Import all Gazebo-customization elements, including Gazebo colors -->
   <xacro:include filename="$(find environment_description)/urdf/environment_gazebo.urdf.xacro" />

File: tms_rp/rostms_description/urdf/environments_standalone.urdf.xacro (robot description, xacro)
@@ -1,3 +1,4 @@
 <?xml version="1.0"?>
+<!-- Environment component of ROS-TMS project -->
 <robot name="environment_standalone"
        xmlns:sensor="http://playerstage.sourceforge.net/gazebo/xmlschema/#sensor"
@@ -5,4 +6,6 @@
        xmlns:interface="http://playerstage.sourceforge.net/gazebo/xmlschema/#interface"
        xmlns:xacro="http://ros.org/wiki/xacro">
+  <!-- Import common properties -->
+  <xacro:include filename="$(find environment_description)/urdf/common_properties.urdf.xacro" />
   <!-- Defines the environment component tag. -->
   <xacro:include filename="$(find environment_description)/urdf/environment.urdf.xacro" />

File: tms_rp/rostms_description/urdf/objects.urdf.xacro (robot description, xacro)
@@ -1,7 +1,5 @@
 <?xml version="1.0"?>
 <!-- Environment of B-Sen Project room -->
-<robot name="objects" xmlns:xacro="http://www.ros.org/wiki/xacro">
-  <!-- Constants for robot dimensions -->
-  <xacro:property name="PI" value="3.1415926535897931"/>
+<robot name="object" xmlns:xacro="http://www.ros.org/wiki/xacro">
   <!-- Import all Gazebo-customization elements, including Gazebo colors -->
   <xacro:include filename="$(find environment_description)/urdf/environment.gazebo" />

Commit message: deleted the bsen_origin joint and use the bsen_room joint for making the one focus point

File: tms_rp/rostms_description/urdf/environments.urdf.xacro (robot description, xacro)
@@ -27,21 +27,8 @@
       </inertial>
     </link>
-    <joint name="bsen_origin_joint" type="fixed">
-      <parent link="bsen_room"/>
-      <child link="bsen_origin"/>
-      <origin xyz="4.5 0 0" rpy="0 0 0"/>
-    </joint>
-    <link name="bsen_origin">
-      <visual>
-        <geometry>
-          <box size="0.1 0.1 0.1"/>
-        </geometry>
-        <origin xyz="0 0 0" rpy="0 0 0"/>
-      </visual>
-    </link>
     <joint name="bsen_room_to_wall" type="fixed">
       <parent link="bsen_room"/>
       <child link="bsen_wall"/>
-      <origin xyz="0 0 0"/>
+      <origin xyz="0. 0. 0." rpy="0 0 0"/>
     </joint>
     <link name="bsen_wall">
@@ -50,5 +37,4 @@
           <mesh filename="package://environmental_model/model/bsen_wall.dae"/>
         </geometry>
-        <origin xyz="0. 0. 0." rpy="0 0 0"/>
       </visual>
     </link>
@@ -56,5 +42,5 @@
       <parent link="bsen_room"/>
       <child link="bsen_celling"/>
-      <origin xyz="0 0 0"/>
+      <origin xyz="0. 0. 2.3" rpy="0 0 0"/>
     </joint>
     <link name="bsen_celling">
@@ -63,11 +49,10 @@
           <mesh filename="package://environmental_model/model/bsen_celling.dae"/>
         </geometry>
-        <origin xyz="0. 0. 2.3" rpy="0 0 0"/>
       </visual>
     </link>
     <joint name="bsen_room_to_kitchen" type="fixed">
-      <parent link="bsen_origin"/>
+      <parent link="bsen_room"/>
       <child link="kitchen"/>
-      <origin xyz="0 0 0"/>
+      <origin xyz="9.16 5.9 0.4855" rpy="0 0 -1.57079633"/>
     </joint>
     <link name="kitchen">
@@ -76,11 +61,10 @@
           <mesh filename="package://environmental_model/model/kitchen.dae"/>
         </geometry>
-        <origin xyz="4.66 5.9 0.4855" rpy="0 0 -1.57079633"/>
       </visual>
     </link>
     <joint name="bsen_room_to_meeting_table" type="fixed">
-      <parent link="bsen_origin"/>
+      <parent link="bsen_room"/>
       <child link="meeting_table"/>
-      <origin xyz="0 0 0"/>
+      <origin xyz="5.7 1.5 0.36" rpy="0 0 0"/>
     </joint>
     <link name="meeting_table">
@@ -89,11 +73,10 @@
           <mesh filename="package://environmental_model/model/meeting_table.dae"/>
         </geometry>
-        <origin xyz="1.2 1.5 0.36" rpy="0 0 0"/>
       </visual>
     </link>
     <joint name="bsen_room_to_tree" type="fixed">
-      <parent link="bsen_origin"/>
+      <parent link="bsen_room"/>
       <child link="tree"/>
-      <origin xyz="0 0 0"/>
+      <origin xyz="14.3 5.3 0." rpy="0 0 0"/>
     </joint>
     <link name="tree">
@@ -102,11 +85,10 @@
           <mesh filename="package://environmental_model/model/tree.dae"/>
         </geometry>
-        <origin xyz="9.8 5.3 0." rpy="0 0 0"/>
       </visual>
     </link>
     <joint name="bsen_room_to_tv_table" type="fixed">
-      <parent link="bsen_origin"/>
+      <parent link="bsen_room"/>
       <child link="tv_table"/>
-      <origin xyz="0 0 0"/>
+      <origin xyz="11.1 2.9 0.175" rpy="0 0 0"/>
     </joint>
     <link name="tv_table">
@@ -115,11 +97,10 @@
           <mesh filename="package://environmental_model/model/tv_table.dae"/>
         </geometry>
-        <origin xyz="6.6 2.9 0.175" rpy="0 0 0"/>
       </visual>
     </link>
     <joint name="bsen_room_to_tv_52" type="fixed">
-      <parent link="bsen_origin"/>
+      <parent link="bsen_room"/>
       <child link="tv_52"/>
-      <origin xyz="0 0 0"/>
+      <origin xyz="11.2 2.9 0.7085" rpy="0 0 -1.57079633"/>
     </joint>
     <link name="tv_52">
@@ -128,11 +109,10 @@
           <mesh filename="package://environmental_model/model/tv_52.dae"/>
         </geometry>
-        <origin xyz="6.7 2.9 0.7085" rpy="0 0 -1.57079633"/>
       </visual>
     </link>
     <joint name="bsen_room_to_recorder" type="fixed">
-      <parent link="bsen_origin"/>
+      <parent link="bsen_room"/>
       <child link="recorder"/>
-      <origin xyz="0 0 0"/>
+      <origin xyz="11.1 2.9 0.3805" rpy="0 0 3.14159265"/>
     </joint>
     <link name="recorder">
@@ -141,11 +121,10 @@
           <mesh filename="package://environmental_model/model/recorder.dae"/>
         </geometry>
-        <origin xyz="6.6 2.9 0.3805" rpy="0 0 3.14159265"/>
       </visual>
     </link>
     <joint name="bsen_room_to_sofa" type="fixed">
-      <parent link="bsen_origin"/>
+      <parent link="bsen_room"/>
       <child link="sofa"/>
-      <origin xyz="0 0 0"/>
+      <origin xyz="9.1 2.9 0.395" rpy="0 0 0"/>
     </joint>
     <link name="sofa">
@@ -154,11 +133,10 @@
           <mesh filename="package://environmental_model/model/sofa.dae"/>
         </geometry>
-        <origin xyz="4.6 2.9 0.395" rpy="0 0 0"/>
       </visual>
     </link>
     <joint name="bsen_room_to_sofa_table" type="fixed">
-      <parent link="bsen_origin"/>
+      <parent link="bsen_room"/>
       <child link="sofa_table"/>
-      <origin xyz="0 0 0"/>
+      <origin xyz="10.2 2.9 0.235" rpy="0 0 0"/>
     </joint>
     <link name="sofa_table">
@@ -167,11 +145,10 @@
           <mesh filename="package://environmental_model/model/sofa_table.dae"/>
         </geometry>
-        <origin xyz="5.7 2.9 0.235" rpy="0 0 0"/>
       </visual>
     </link>
     <joint name="bsen_room_to_carpet" type="fixed">
-      <parent link="bsen_origin"/>
+      <parent link="bsen_room"/>
       <child link="carpet"/>
-      <origin xyz="0 0 0"/>
+      <origin xyz="9.9 2.9 0.1" rpy="0 0 0"/>
     </joint>
     <link name="carpet">
@@ -180,11 +157,10 @@
           <mesh filename="package://environmental_model/model/carpet.dae"/>
         </geometry>
-        <origin xyz="5.4 2.9 0.1" rpy="0 0 0"/>
       </visual>
     </link>
     <joint name="bsen_room_to_drawer" type="fixed">
-      <parent link="bsen_origin"/>
+      <parent link="bsen_room"/>
       <child link="drawer"/>
-      <origin xyz="0 0 0"/>
+      <origin xyz="12.93 5.8 0.303" rpy="0 0 -1.57079633"/>
     </joint>
     <link name="drawer">
@@ -193,11 +169,10 @@
           <mesh filename="package://environmental_model/model/drawer.dae"/>
         </geometry>
-        <origin xyz="8.43 5.8 0.303" rpy="0 0 -1.57079633"/>
       </visual>
     </link>
     <joint name="bsen_room_to_bed" type="fixed">
-      <parent link="bsen_origin"/>
+      <parent link="bsen_room"/>
       <child link="bed"/>
-      <origin xyz="0 0 0"/>
+      <origin xyz="12.48 2.3 0.2075" rpy="0 0 0"/>
     </joint>
     <link name="bed">
@@ -206,11 +181,10 @@
           <mesh filename="package://environmental_model/model/bed.dae"/>
         </geometry>
-        <origin xyz="7.98 2.3 0.2075" rpy="0 0 0"/>
       </visual>
     </link>
     <joint name="bsen_room_to_wordrobe" type="fixed">
-      <parent link="bsen_origin"/>
+      <parent link="bsen_room"/>
       <child link="wordrobe"/>
-      <origin xyz="0 0 0"/>
+      <origin xyz="13.6 5.8 1.3" rpy="0 0 -1.57079633"/>
     </joint>
     <link name="wordrobe">
@@ -219,11 +193,10 @@
           <mesh filename="package://environmental_model/model/wordrobe.dae"/>
         </geometry>
-        <origin xyz="9.1 5.8 1.3" rpy="0 0 -1.57079633"/>
       </visual>
     </link>
     <joint name="bsen_room_to_workdesk" type="fixed">
-      <parent link="bsen_origin"/>
+      <parent link="bsen_room"/>
       <child link="workdesk"/>
-      <origin xyz="0 0 0"/>
+      <origin xyz="11.93 5.9 0.5" rpy="0 0 -1.57079633"/>
     </joint>
     <link name="workdesk">
@@ -232,11 +205,10 @@
           <mesh filename="package://environmental_model/model/work_desk.dae"/>
         </geometry>
-        <origin xyz="7.43 5.9 0.5" rpy="0 0 -1.57079633"/>
       </visual>
     </link>
     <joint name="bsen_room_to_tv_multi" type="fixed">
-      <parent link="bsen_origin"/>
+      <parent link="bsen_room"/>
       <child link="tv_multi"/>
-      <origin xyz="0 0 0"/>
+      <origin xyz="14.37 2.2 1.0" rpy="0 0 -1.57079633"/>
     </joint>
     <link name="tv_multi">
@@ -245,11 +217,10 @@
           <mesh filename="package://environmental_model/model/tv_multi.dae"/>
         </geometry>
-        <origin xyz="9.87 2.2 1.0" rpy="0 0 -1.57079633"/>
       </visual>
     </link>
     <joint name="bsen_room_to_intelingent_shelf" type="fixed">
-      <parent link="bsen_origin"/>
+      <parent link="bsen_room"/>
       <child link="intelingent_shelf"/>
-      <origin xyz="0 0 0"/>
+      <origin xyz="11.56 3.520 0.445" rpy="0 0 0"/>
     </joint>
     <link name="intelingent_shelf">
@@ -258,5 +229,4 @@
           <mesh filename="package://environmental_model/model/intelingent_shelf.dae"/>
         </geometry>
-        <origin xyz="7.06 3.520 0.445" rpy="0 0 0"/>
       </visual>
     </link>

Commit message: change wordrobe & workdesk & kitchen model position on the rviz

File: tms_rp/rostms_description/urdf/environments.urdf.xacro (robot description, xacro)
@@ -54,5 +54,5 @@
       <parent link="bsen_room"/>
       <child link="kitchen"/>
-      <origin xyz="9.16 5.9 0.4855" rpy="0 0 -1.57079633"/>
+      <origin xyz="9.26 5.9 0.4855" rpy="0 0 -1.57079633"/>
     </joint>
     <link name="kitchen">
@@ -186,5 +186,5 @@
       <parent link="bsen_room"/>
       <child link="wordrobe"/>
-      <origin xyz="13.6 5.8 1.3" rpy="0 0 -1.57079633"/>
+      <origin xyz="13.7 5.9 1.3" rpy="0 0 -1.57079633"/>
     </joint>
     <link name="wordrobe">
@@ -198,5 +198,5 @@
       <parent link="bsen_room"/>
       <child link="workdesk"/>
-      <origin xyz="11.93 5.9 0.5" rpy="0 0 -1.57079633"/>
+      <origin xyz="12.05 5.9 0.5" rpy="0 0 -1.57079633"/>
     </joint>
     <link name="workdesk">

Commit message: changed the unit used in tms_rp_action package of ros-tms system

File: tms_rp/rostms_description/urdf/environments.urdf.xacro (robot description, xacro)
@@ -185,11 +185,11 @@
     <joint name="bsen_room_to_wordrobe" type="fixed">
       <parent link="bsen_room"/>
-      <child link="wordrobe"/>
+      <child link="wardrobe"/>
       <origin xyz="13.7 5.9 1.3" rpy="0 0 -1.57079633"/>
     </joint>
-    <link name="wordrobe">
-      <visual>
-        <geometry>
-          <mesh filename="package://environmental_model/model/wordrobe.dae"/>
+    <link name="wardrobe">
+      <visual>
+        <geometry>
+          <mesh filename="package://environmental_model/model/wardrobe.dae"/>
         </geometry>
       </visual>

Commit message: added collision information of models in our environment for planning

File: tms_rp/rostms_description/urdf/environments.urdf.xacro (robot description, xacro)
@@ -13,4 +13,10 @@
         <origin xyz="0 0 0.001" rpy="0 0 0"/>
       </visual>
+      <collision>
+        <geometry>
+          <box size="15.0 7.0 0.001"/>
+        </geometry>
+        <origin xyz="7.5 3.5 -0.001" rpy="0 0 0"/>
+      </collision>
       <inertial>
         <origin xyz="0 0 0.001" rpy="0 0 0"/>
@@ -33,4 +39,9 @@
         </geometry>
       </visual>
+      <collision>
+        <geometry>
+          <mesh filename="package://environmental_model/model/bsen_wall.dae"/>
+        </geometry>
+      </collision>
     </link>
     <joint name="celling_joint" type="fixed">
@@ -45,4 +56,9 @@
         </geometry>
       </visual>
+      <collision>
+        <geometry>
+          <mesh filename="package://environmental_model/model/bsen_celling.dae"/>
+        </geometry>
+      </collision>
     </link>
     <joint name="kitchen_joint" type="fixed">
@@ -57,4 +73,9 @@
         </geometry>
       </visual>
+      <collision>
+        <geometry>
+          <box size="0.65 3.12 0.65"/>
+        </geometry>
+      </collision>
     </link>
     <joint name="meeting_table_joint" type="fixed">
@@ -69,4 +90,9 @@
         </geometry>
       </visual>
+      <collision>
+        <geometry>
+          <cylinder radius="0.66" length="0.73"/>
+        </geometry>
+      </collision>
     </link>
     <joint name="tree_link" type="fixed">
@@ -81,4 +107,10 @@
         </geometry>
       </visual>
+      <collision>
+        <geometry>
+          <cylinder radius="0.2" length="1.0"/>
+        </geometry>
+          <origin xyz="0.0 0.0 0.55" rpy="0 0 0"/>
+      </collision>
     </link>
     <joint name="tv_table_joint" type="fixed">
@@ -93,4 +125,9 @@
         </geometry>
       </visual>
+      <collision>
+        <geometry>
+          <box size="0.35 2.7 0.35"/>
+        </geometry>
+      </collision>
     </link>
     <joint name="tv_52_link" type="fixed">
@@ -105,4 +142,9 @@
         </geometry>
       </visual>
+      <collision>
+        <geometry>
+          <box size="1.2 0.1 0.7"/>
+        </geometry>
+      </collision>
     </link>
     <joint name="recorder_joint" type="fixed">
@@ -117,4 +159,9 @@
         </geometry>
       </visual>
+      <collision>
+        <geometry>
+          <box size="0.25 0.45 0.1"/>
+        </geometry>
+      </collision>
     </link>
     <joint name="sofa_joint" type="fixed">
@@ -129,4 +176,9 @@
         </geometry>
       </visual>
+      <collision>
+        <geometry>
+          <box size="0.8 2.35 0.77"/>
+        </geometry>
+      </collision>
     </link>
     <joint name="sofa_table_joint" type="fixed">
@@ -141,9 +193,14 @@
         </geometry>
       </visual>
+      <collision>
+        <geometry>
+          <box size="0.5 1.3 0.43"/>
+        </geometry>
+      </collision>
     </link>
     <joint name="carpet_joint" type="fixed">
       <parent link="bsen_room_link"/>
       <child link="carpet_link"/>
-      <origin xyz="9.9 2.9 0.1" rpy="0 0 0"/>
+      <origin xyz="9.9 2.9 0.01" rpy="0 0 0"/>
     </joint>
     <link name="carpet_link">
@@ -153,4 +210,9 @@
         </geometry>
       </visual>
+      <collision>
+        <geometry>
+          <box size="1.76 2.55 0.01"/>
+        </geometry>
+      </collision>
     </link>
     <joint name="drawer_joint" type="fixed">
@@ -165,4 +227,9 @@
         </geometry>
       </visual>
+      <collision>
+        <geometry>
+          <box size="0.6 0.4 0.6"/>
+        </geometry>
+      </collision>
     </link>
     <joint name="bed_joint" type="fixed">
@@ -177,4 +244,9 @@
         </geometry>
       </visual>
+      <collision>
+        <geometry>
+          <box size="2.2 1.88 0.2"/>
+        </geometry>
+      </collision>
     </link>
     <joint name="wardrobe_joint" type="fixed">
@@ -189,4 +261,9 @@
         </geometry>
       </visual>
+      <collision>
+        <geometry>
+          <box size="0.7 0.95 2.56"/>
+        </geometry>
+      </collision>
     </link>
     <joint name="workdesk_joint" type="fixed">
@@ -201,4 +278,9 @@
         </geometry>
       </visual>
+      <collision>
+        <geometry>
+          <box size="0.65 2.44 0.7"/>
+        </geometry>
+      </collision>
     </link>
     <joint name="tv_multi_joint" type="fixed">
@@ -213,4 +295,9 @@
         </geometry>
       </visual>
+      <collision>
+        <geometry>
+          <box size="2.5 0.2 1.4"/>
+        </geometry>
+      </collision>
     </link>
     <joint name="intelingent_shelf_joint" type="fixed">
@@ -225,4 +312,9 @@
         </geometry>
       </visual>
+      <collision>
+        <geometry>
+          <box size="0.3 0.5 0.9"/>
+        </geometry>
+      </collision>
     </link>
     <xacro:environments_sim/>

File: tms_rp/rostms_description/urdf/objects.urdf.xacro (robot description, xacro)
@@ -33,4 +33,10 @@
         <origin xyz="0.0 0.0 0.3978" rpy="0 0 0"/>
       </visual>
+      <collision>
+        <geometry>
+          <cylinder radius="0.35" length="0.8"/>
+        </geometry>
+        <origin xyz="0.0 0.0 0.3978" rpy="0 0 0"/>
+      </collision>
     </link>
   </xacro:macro>
@@ -64,4 +70,10 @@
         <origin xyz="0.0 0.0 0.51" rpy="0.0 0.0 0.0"/>
       </visual>
+      <collision>
+        <geometry>
+          <cylinder radius="0.35" length="1.1"/>
+        </geometry>
+        <origin xyz="0.0 0.0 0.51" rpy="0.0 0.0 0.0"/>
+      </collision>
     </link>
     <!-- refrigerator -->
@@ -93,4 +105,10 @@
         <origin xyz="0.0 0.0 0.56" rpy="0 0 0"/>
       </visual>
+      <collision>
+        <geometry>
+          <box size="0.6 0.5 1.1"/>
+        </geometry>
+        <origin xyz="0.0 0.0 0.56" rpy="0 0 0"/>
+      </collision>
     </link>
     <!-- Add meeting_chair -->
@@ -125,6 +143,12 @@
           <mesh filename="package://environmental_model/model/wagon.dae"/>
         </geometry>
-        <origin xyz="0. 0. 0.5" rpy="0 0 0"/>
+        <origin xyz="0. 0. 0.3" rpy="0 0 0"/>
       </visual>
+      <collision>
+        <geometry>
+          <box size="0.6 0.4 0.7"/>
+        </geometry>
+        <origin xyz="0. 0. 0.3" rpy="0 0 0"/>
+      </collision>
     </link>
     <objects_sim/>
