Commit message: change rviz model position

File: tms_rp/rostms_description/urdf/environments.urdf.xacro (robot description, xacro)
@@ -65,5 +65,5 @@
       <parent link="bsen_room_link"/>
       <child link="kitchen_link"/>
-      <origin xyz="9.26 5.9 0.4855" rpy="0 0 -1.57079633"/>
+      <origin xyz="9.05 5.87 0.4855" rpy="0 0 -1.57079633"/>
     </joint>
     <link name="kitchen_link">
@@ -125,5 +125,5 @@
       <parent link="bsen_room_link"/>
       <child link="tv_table_link"/>
-      <origin xyz="11.1 2.9 0.175" rpy="0 0 0"/>
+      <origin xyz="14.25 2.5 0.175" rpy="0 0 0"/>
     </joint>
     <link name="tv_table_link">
@@ -139,42 +139,8 @@
       </collision>
     </link>
-    <joint name="tv_52_link" type="fixed">
-      <parent link="bsen_room_link"/>
-      <child link="tv_52_link"/>
-      <origin xyz="11.2 2.9 0.7085" rpy="0 0 -1.57079633"/>
-    </joint>
-    <link name="tv_52_link">
-      <visual>
-        <geometry>
-          <mesh filename="package://environmental_model/model/tv_52.dae"/>
-        </geometry>
-      </visual>
-      <collision>
-        <geometry>
-          <box size="1.2 0.1 0.7"/>
-        </geometry>
-      </collision>
-    </link>
-    <joint name="recorder_joint" type="fixed">
-      <parent link="bsen_room_link"/>
-      <child link="recorder_link"/>
-      <origin xyz="11.1 2.9 0.3805" rpy="0 0 3.14159265"/>
-    </joint>
-    <link name="recorder_link">
-      <visual>
-        <geometry>
-          <mesh filename="package://environmental_model/model/recorder.dae"/>
-        </geometry>
-      </visual>
-      <collision>
-        <geometry>
-          <box size="0.25 0.45 0.1"/>
-        </geometry>
-      </collision>
-    </link>
     <joint name="sofa_joint" type="fixed">
       <parent link="bsen_room_link"/>
       <child link="sofa_link"/>
-      <origin xyz="9.1 2.9 0.395" rpy="0 0 0"/>
+      <origin xyz="11.75 2.6 0.395" rpy="0 0 0"/>
     </joint>
     <link name="sofa_link">
@@ -193,5 +159,5 @@
       <parent link="bsen_room_link"/>
       <child link="sofa_table_link"/>
-      <origin xyz="10.2 2.9 0.235" rpy="0 0 0"/>
+      <origin xyz="12.7 2.5 0.235" rpy="0 0 0"/>
     </joint>
     <link name="sofa_table_link">
@@ -207,8 +173,25 @@
       </collision>
     </link>
+    <joint name="bed_joint" type="fixed">
+      <parent link="bsen_room_link"/>
+      <child link="bed_link"/>
+      <origin xyz="10.35 2.7 0.235" rpy="0 0 0"/>
+    </joint>
+    <link name="bed_link">
+      <visual>
+        <geometry>
+          <mesh filename="package://environmental_model/model/paramount_bed.dae"/>
+        </geometry>
+      </visual>
+      <collision>
+        <geometry>
+          <box size="0.5 1.3 0.43"/>
+        </geometry>
+      </collision>
+    </link>
     <joint name="carpet_joint" type="fixed">
       <parent link="bsen_room_link"/>
       <child link="carpet_link"/>
-      <origin xyz="9.9 2.9 0.01" rpy="0 0 0"/>
+      <origin xyz="12.3 2.6 0.01" rpy="0 0 0"/>
     </joint>
     <link name="carpet_link">
@@ -227,5 +210,5 @@
       <parent link="bsen_room_link"/>
       <child link="drawer_link"/>
-      <origin xyz="12.93 5.8 0.303" rpy="0 0 -1.57079633"/>
+      <origin xyz="12.72 5.8 0.303" rpy="0 0 -1.57079633"/>
     </joint>
     <link name="drawer_link">
@@ -241,25 +224,8 @@
       </collision>
     </link>
-    <joint name="bed_joint" type="fixed">
-      <parent link="bsen_room_link"/>
-      <child link="bed_link"/>
-      <origin xyz="12.48 2.3 0.2075" rpy="0 0 0"/>
-    </joint>
-    <link name="bed_link">
-      <visual>
-        <geometry>
-          <mesh filename="package://environmental_model/model/bed.dae"/>
-        </geometry>
-      </visual>
-      <collision>
-        <geometry>
-          <box size="2.2 1.88 0.2"/>
-        </geometry>
-      </collision>
-    </link>
     <joint name="wardrobe_joint" type="fixed">
       <parent link="bsen_room_link"/>
       <child link="wardrobe_link"/>
-      <origin xyz="13.7 5.9 1.3" rpy="0 0 -1.57079633"/>
+      <origin xyz="13.46 5.9 1.3" rpy="0 0 -1.57079633"/>
     </joint>
     <link name="wardrobe_link">
@@ -278,5 +244,5 @@
       <parent link="bsen_room_link"/>
       <child link="workdesk_link"/>
-      <origin xyz="12.05 5.9 0.5" rpy="0 0 -1.57079633"/>
+      <origin xyz="11.80 5.9 0.5" rpy="0 0 -1.57079633"/>
     </joint>
     <link name="workdesk_link">
@@ -295,5 +261,5 @@
       <parent link="bsen_room_link"/>
       <child link="tv_multi_link"/>
-      <origin xyz="14.37 2.2 1.0" rpy="0 0 -1.57079633"/>
+      <origin xyz="14.37 2.2 1.45" rpy="0 0 -1.57079633"/>
     </joint>
     <link name="tv_multi_link">
@@ -312,5 +278,5 @@
       <parent link="bsen_room_link"/>
       <child link="intelingent_shelf_link"/>
-      <origin xyz="11.56 3.520 0.445" rpy="0 0 0"/>
+      <origin xyz="11.48 4.220 0.445" rpy="0 0 0"/>
     </joint>
     <link name="intelingent_shelf_link">

Commit message: modifed refrigerator model

File: tms_rp/rostms_description/urdf/environments.urdf.xacro (robot description, xacro)
@@ -292,4 +292,21 @@
       </collision>
     </link>
+    <joint name="refrigerator_joint" type="fixed">
+      <parent link="bsen_room_link"/>
+      <child link="refrigerator_link"/>
+      <origin xyz="7.0 5.52 0.0" rpy="0 0 -1.57079633"/>
+    </joint>
+    <link name="refrigerator_link">
+      <visual>
+        <geometry>
+          <mesh filename="package://environmental_model/model/refrigerator.dae"/>
+        </geometry>
+      </visual>
+      <collision>
+        <geometry>
+          <box size="0.3 0.5 0.9"/>
+        </geometry>
+      </collision>
+    </link>
     <xacro:environments_sim/>
   </xacro:macro>

File: tms_rp/rostms_description/urdf/objects.urdf.xacro (robot description, xacro)
@@ -78,5 +78,5 @@
     </link>
     <!-- refrigerator -->
-    <link name="refrigerator_x_link"/>
+<!--     <link name="refrigerator_x_link"/>
     <joint name="refrigerator_x_joint" type="prismatic">
       <parent link="world_link"/>
@@ -111,5 +111,5 @@
         <origin xyz="0.0 0.0 0.56" rpy="0 0 0"/>
       </collision>
-    </link>
+    </link> -->
     <!-- Add meeting_chair -->
     <xacro:meeting_chair_link num="1"/>

Commit message: change model data position

File: tms_rp/rostms_description/urdf/environments.urdf.xacro (robot description, xacro)
@@ -65,5 +65,5 @@
       <parent link="bsen_room_link"/>
       <child link="kitchen_link"/>
-      <origin xyz="9.05 5.87 0.4855" rpy="0 0 -1.57079633"/>
+      <origin xyz="9.03 5.87 0.4855" rpy="0 0 -1.57079633"/>
     </joint>
     <link name="kitchen_link">
@@ -244,5 +244,5 @@
       <parent link="bsen_room_link"/>
       <child link="workdesk_link"/>
-      <origin xyz="11.80 5.9 0.5" rpy="0 0 -1.57079633"/>
+      <origin xyz="11.80 5.9 0.35" rpy="0 0 -1.57079633"/>
     </joint>
     <link name="workdesk_link">
@@ -278,5 +278,5 @@
       <parent link="bsen_room_link"/>
       <child link="intelingent_shelf_link"/>
-      <origin xyz="11.48 4.220 0.445" rpy="0 0 0"/>
+      <origin xyz="11.65 3.970 0.005" rpy="0 0 0"/>
     </joint>
     <link name="intelingent_shelf_link">

Commit message: model change .refrigerator .meeting_door .kitchen

File: tms_rp/rostms_description/urdf/environments.urdf.xacro (robot description, xacro)
@@ -65,5 +65,5 @@
       <parent link="bsen_room_link"/>
       <child link="kitchen_link"/>
-      <origin xyz="9.03 5.87 0.4855" rpy="0 0 -1.57079633"/>
+      <origin xyz="9.09 5.907 0.0" rpy="0 0 -1.57079633"/>
     </joint>
     <link name="kitchen_link">
@@ -295,5 +295,5 @@
       <parent link="bsen_room_link"/>
       <child link="refrigerator_link"/>
-      <origin xyz="7.0 5.52 0.0" rpy="0 0 -1.57079633"/>
+      <origin xyz="6.94 5.53 -0.01" rpy="0 0 -1.57079633"/>
     </joint>
     <link name="refrigerator_link">
@@ -303,4 +303,21 @@
         </geometry>
       </visual>
+    </link>
+    <joint name="meeting_door_joint" type="fixed">
+      <parent link="bsen_room_link"/>
+      <child link="meeting_door_link"/>
+      <origin xyz="1.94 3.035 1.31" rpy="0 0 3.14159"/>
+    </joint>
+    <link name="meeting_door_link">
+      <visual>
+        <geometry>
+          <mesh filename="package://environmental_model/model/meeting_door.dae"/>
+        </geometry>
+      </visual>
+      <collision>
+        <geometry>
+          <box size="0.03 1.23 0.9"/>
+        </geometry>
+      </collision>
     </link>
     <xacro:environments_sim/>
