Commit message: integrated all bringup launch file into one component

File: tms_rp/rostms_description/urdf/all_components_with_moveit.urdf (robot description, URDF)
Before this commit: robot rostms, 68 links, 67 joints
Links:
- link bsen_celling_link: geometry collision mesh filename=package://environmental_model/model/bsen_celling.dae; visual mesh filename=package://environmental_model/model/bsen_celling.dae
- link bsen_room_link: mass 1 -> None
- link bsen_wall_link: geometry collision box size=0.1 0.1 0.1; visual mesh filename=package://environmental_model/model/bsen_wall.dae
Joints:
- joint wall_joint: origin xyz=0. 0. 0. rpy=0 0 0 -> xyz=0 0 0 rpy=0 0 0

Commit message: updated tms_db_reader

File: tms_rp/rostms_description/urdf/all_components_with_moveit.urdf (robot description, URDF)
Before this commit: robot rostms, 74 links, 73 joints
Links:
- removed link recorder_link
- removed link refrigerator_x_link
- removed link refrigerator_y_link
- removed link tv_52_link
- added link cancoffee_link; visual mesh filename=package://environmental_model/model/cancoffee.dae
- added link cancoffee_pitch_link
- added link cancoffee_x_link
- added link cancoffee_y_link
- added link cancoffee_yaw_link
- added link cancoffee_z_link
- added link greentea_bottle_link; visual mesh filename=package://environmental_model/model/greentea_bottle.dae
- added link greentea_bottle_pitch_link
- added link greentea_bottle_x_link
- added link greentea_bottle_y_link
- added link greentea_bottle_yaw_link
- added link greentea_bottle_z_link
- added link soysauce_bottle_black_link; visual mesh filename=package://environmental_model/model/soysauce_bottle_black.d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
- added link soysauce_bottle_black_pitch_link
- added link soysauce_bottle_black_x_link
- added link soysauce_bottle_black_y_link
- added link soysauce_bottle_black_yaw_link
- added link soysauce_bottle_black_z_link
- added link wheelchair_link; collision box size=0.6 0.5 1.1; visual mesh filename=package://environmental_model/model/wheelchair.dae
- added link wheelchair_x_link
- added link wheelchair_y_link
- link bed_link: geometry collision box size=0.5 1.3 0.43; visual mesh filename=package://environmental_model/model/paramount_bed.dae
- link refrigerator_link: geometry collision box size=0.3 0.5 0.9; visual mesh filename=package://environmental_model/model/refrigerator.dae
Joints:
- removed joint recorder_joint
- removed joint refrigerator_x_joint
- removed joint refrigerator_y_joint
- removed joint refrigerator_yaw_joint
- removed joint tv_52_link
- added joint cancoffee_pitch_joint: type continuous, parent cancoffee_yaw_link, child cancoffee_pitch_link, origin xyz=0 0 0 rpy=0 0 0, axis 0 1 0
- added joint cancoffee_roll_joint: type continuous, parent cancoffee_pitch_link, child cancoffee_link, origin xyz=0 0 0 rpy=0 0 0, axis 1 0 0
- added joint cancoffee_x_joint: type prismatic, parent world_link, child cancoffee_x_link, origin xyz=0 0 0 rpy=0 0 0, limit lower=0. upper=15. effort=1000.0 velocity=0.5
- added joint cancoffee_y_joint: type prismatic, parent cancoffee_x_link, child cancoffee_y_link, origin xyz=0 0 0 rpy=0 0 1.57079633, limit lower=0. upper=8. effort=1000.0 velocity=0.5
- added joint cancoffee_yaw_joint: type continuous, parent cancoffee_z_link, child cancoffee_yaw_link, origin xyz=0 0 0 rpy=-1.57079633 0 -1.57079633, axis 0 0 1
- added joint cancoffee_z_joint: type prismatic, parent cancoffee_y_link, child cancoffee_z_link, origin xyz=0 0 0 rpy=0 -1.57079633 0, limit lower=0. upper=3. effort=1000.0 velocity=0.5
- added joint greentea_bottle_pitch_joint: type continuous, parent greentea_bottle_yaw_link, child greentea_bottle_pitch_link, origin xyz=0 0 0 rpy=0 0 0, axis 0 1 0
- added joint greentea_bottle_roll_joint: type continuous, parent greentea_bottle_pitch_link, child greentea_bottle_link, origin xyz=0 0 0 rpy=0 0 0, axis 1 0 0
- added joint greentea_bottle_x_joint: type prismatic, parent world_link, child greentea_bottle_x_link, origin xyz=0 0 0 rpy=0 0 0, limit lower=0. upper=15. effort=1000.0 velocity=0.5
- added joint greentea_bottle_y_joint: type prismatic, parent greentea_bottle_x_link, child greentea_bottle_y_link, origin xyz=0 0 0 rpy=0 0 1.57079633, limit lower=0. upper=8. effort=1000.0 velocity=0.5
- added joint greentea_bottle_yaw_joint: type continuous, parent greentea_bottle_z_link, child greentea_bottle_yaw_link, origin xyz=0 0 0 rpy=-1.57079633 0 -1.57079633, axis 0 0 1
- added joint greentea_bottle_z_joint: type prismatic, parent greentea_bottle_y_link, child greentea_bottle_z_link, origin xyz=0 0 0 rpy=0 -1.57079633 0, limit lower=0. upper=3. effort=1000.0 velocity=0.5
- added joint refrigerator_joint: type fixed, parent bsen_room_link, child refrigerator_link, origin xyz=7.0 5.52 0.0 rpy=0 0 -1.57079633
- added joint soysauce_bottle_black_pitch_joint: type continuous, parent soysauce_bottle_black_yaw_link, child soysauce_bottle_black_pitch_link, origin xyz=0 0 0 rpy=0 0 0, axis 0 1 0
- added joint soysauce_bottle_black_roll_joint: type continuous, parent soysauce_bottle_black_pitch_link, child soysauce_bottle_black_link, origin xyz=0 0 0 rpy=0 0 0, axis 1 0 0
- added joint soysauce_bottle_black_x_joint: type prismatic, parent world_link, child soysauce_bottle_black_x_link, origin xyz=0 0 0 rpy=0 0 0, limit lower=0. upper=15. effort=1000.0 velocity=0.5
- added joint soysauce_bottle_black_y_joint: type prismatic, parent soysauce_bottle_black_x_link, child soysauce_bottle_black_y_link, origin xyz=0 0 0 rpy=0 0 1.57079633, limit lower=0. upper=8. effort=1000.0 velocity=0.5
- added joint soysauce_bottle_black_yaw_joint: type continuous, parent soysauce_bottle_black_z_link, child soysauce_bottle_black_yaw_link, origin xyz=0 0 0 rpy=-1.57079633 0 -1.57079633, axis 0 0 1
- added joint soysauce_bottle_black_z_joint: type prismatic, parent soysauce_bottle_black_y_link, child soysauce_bottle_black_z_link, origin xyz=0 0 0 rpy=0 -1.57079633 0, limit lower=0. upper=3. effort=1000.0 velocity=0.5
- added joint wheelchair_x_joint: type prismatic, parent world_link, child wheelchair_x_link, origin xyz=0 0 0 rpy=0 0 0, limit lower=0. upper=15. effort=1000.0 velocity=5.0
- added joint wheelchair_y_joint: type prismatic, parent wheelchair_x_link, child wheelchair_y_link, origin xyz=0 0 0 rpy=0 0 1.57079633, limit lower=0. upper=8. effort=1000.0 velocity=5.0
- added joint wheelchair_yaw_joint: type continuous, parent wheelchair_y_link, child wheelchair_link, origin xyz=0 0 0 rpy=0 0 0, axis 0 0 1
- joint bed_joint: origin xyz=12.48 2.3 0.2075 rpy=0 0 0 -> xyz=10.35 2.7 0.235 rpy=0 0 0
- joint carpet_joint: origin xyz=9.9 2.9 0.01 rpy=0 0 0 -> xyz=12.3 2.6 0.01 rpy=0 0 0
- joint drawer_joint: origin xyz=12.93 5.8 0.303 rpy=0 0 -1.57079633 -> xyz=12.72 5.8 0.303 rpy=0 0 -1.57079633
- joint intelingent_shelf_joint: origin xyz=11.56 3.520 0.445 rpy=0 0 0 -> xyz=11.65 3.970 0.005 rpy=0 0 0
- joint kitchen_joint: origin xyz=9.26 5.9 0.4855 rpy=0 0 -1.57079633 -> xyz=9.03 5.87 0.4855 rpy=0 0 -1.57079633
- joint sofa_joint: origin xyz=9.1 2.9 0.395 rpy=0 0 0 -> xyz=11.75 2.6 0.395 rpy=0 0 0
- joint sofa_table_joint: origin xyz=10.2 2.9 0.235 rpy=0 0 0 -> xyz=12.7 2.5 0.235 rpy=0 0 0
- joint tv_multi_joint: origin xyz=14.37 2.2 1.0 rpy=0 0 -1.57079633 -> xyz=14.37 2.2 1.45 rpy=0 0 -1.57079633
- joint tv_table_joint: origin xyz=11.1 2.9 0.175 rpy=0 0 0 -> xyz=14.25 2.5 0.175 rpy=0 0 0
- joint wardrobe_joint: origin xyz=13.7 5.9 1.3 rpy=0 0 -1.57079633 -> xyz=13.46 5.9 1.3 rpy=0 0 -1.57079633
- joint workdesk_joint: origin xyz=12.05 5.9 0.5 rpy=0 0 -1.57079633 -> xyz=11.80 5.9 0.35 rpy=0 0 -1.57079633

Commit message: modified refrigerator model

File: tms_rp/rostms_description/urdf/all_components_with_moveit.urdf (robot description, URDF)
Before this commit: robot rostms, 91 links, 90 joints
Links:
- link cancoffee_link: geometry collision cylinder length=0.001 radius=0.001; visual mesh filename=package://environmental_model/model/cancoffee.dae
- link chipstar_red_link: geometry collision cylinder length=0.001 radius=0.001; visual mesh filename=package://environmental_model/model/chipstar_red.dae
- link greentea_bottle_link: geometry collision cylinder length=0.001 radius=0.001; visual mesh filename=package://environmental_model/model/greentea_bottle.dae
- link soysauce_bottle_black_link: geometry collision cylinder length=0.001 radius=0.001; visual mesh filename=package://environmental_model/model/soysauce_bottle_black.d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

File: tms_rp/rostms_description/urdf/objects.urdf.xacro (robot description, xacro)
@@ -202,4 +202,10 @@
         <origin rpy="0 0 0" xyz="0. 0. 0."/>
       </visual>
+      <collision>
+        <geometry>
+          <cylinder radius="0.001" length="0.001"/>
+        </geometry>
+        <origin xyz="0 0 0" rpy="0. 0. 0."/>
+      </collision>
     </link>
     <!-- greentea_bottle -->
@@ -252,4 +258,10 @@
         <origin rpy="0 0 0" xyz="0. 0. 0."/>
       </visual>
+      <collision>
+        <geometry>
+          <cylinder radius="0.001" length="0.001"/>
+        </geometry>
+        <origin xyz="0 0 0" rpy="0. 0. 0."/>
+      </collision>
     </link>
     <!-- cancoffee -->
@@ -302,4 +314,10 @@
         <origin rpy="0 0 0" xyz="0. 0. 0."/>
       </visual>
+      <collision>
+        <geometry>
+          <cylinder radius="0.001" length="0.001"/>
+        </geometry>
+        <origin xyz="0 0 0" rpy="0. 0. 0."/>
+      </collision>
     </link>
     <!-- soysauce_bottle_black -->
@@ -352,4 +370,10 @@
         <origin rpy="0 0 0" xyz="0. 0. 0."/>
       </visual>
+      <collision>
+        <geometry>
+          <cylinder radius="0.001" length="0.001"/>
+        </geometry>
+        <origin xyz="0 0 0" rpy="0. 0. 0."/>
+      </collision>
     </link>
     <objects_sim/>

Commit message: pick up object from refrigerator

File: tms_rp/rostms_description/urdf/all_components_with_moveit.urdf (robot description, URDF)
Before this commit: robot rostms, 91 links, 90 joints
Links:
- added link meeting_door_link; collision box size=0.03 1.23 0.9; visual mesh filename=package://environmental_model/model/meeting_door.dae
- added link refrigerator_door_link; collision cylinder length=0.001 radius=0.001; visual mesh filename=package://environmental_model/model/refrigerator_door.dae
Joints:
- added joint meeting_door_joint: type fixed, parent bsen_room_link, child meeting_door_link, origin xyz=1.94 3.035 1.31 rpy=0 0 3.14159
- added joint refrigerator_door_joint: type continuous, parent refrigerator_link, child refrigerator_door_link, origin xyz=-0.035 0.45 1.06 rpy=0 0 0, axis 0 0 1
- joint refrigerator_joint: origin xyz=7.0 5.52 0.0 rpy=0 0 -1.57079633 -> xyz=6.94 5.53 -0.01 rpy=0 0 -1.57079633

File: tms_rp/rostms_description/urdf/environments.urdf.xacro (robot description, xacro)
@@ -65,5 +65,5 @@
       <parent link="bsen_room_link"/>
       <child link="kitchen_link"/>
-      <origin xyz="9.09 5.907 0.0" rpy="0 0 -1.57079633"/>
+      <origin xyz="9.03 5.87 0.4855" rpy="0 0 -1.57079633"/>
     </joint>
     <link name="kitchen_link">
@@ -304,4 +304,22 @@
       </visual>
     </link>
+    <joint name="refrigerator_door_joint" type="continuous">
+      <parent link="refrigerator_link"/>
+      <child link="refrigerator_door_link"/>
+      <origin rpy="0 0 0" xyz="-0.035 0.45 1.06"/>
+      <axis xyz="0 0 1"/>
+    </joint>
+    <link name="refrigerator_door_link">
+      <visual>
+        <geometry>
+          <mesh filename="package://environmental_model/model/refrigerator_door.dae"/>
+        </geometry>
+      </visual>
+      <collision>
+        <geometry>
+          <cylinder radius="0.001" length="0.001"/>
+        </geometry>
+      </collision>
+    </link>
     <joint name="meeting_door_joint" type="fixed">
       <parent link="bsen_room_link"/>

Commit message: updated refrigerator collision model

File: tms_rp/rostms_description/urdf/all_components_with_moveit.urdf (robot description, URDF)
Before this commit: robot rostms, 93 links, 92 joints
Links:
- link refrigerator_link: geometry collision box size=0.5 0.47 0.05; visual mesh filename=package://environmental_model/model/refrigerator.dae

File: tms_rp/rostms_description/urdf/environments.urdf.xacro (robot description, xacro)
@@ -303,4 +303,10 @@
         </geometry>
       </visual>
+      <collision>
+        <geometry>
+          <box size="0.5 0.47 0.05"/>
+        </geometry>
+        <origin xyz="-0.32 0.235 1.09" rpy="0 0 0"/>
+      </collision>
     </link>
     <joint name="refrigerator_door_joint" type="continuous">

Commit message: bugfix

File: tms_rp/rostms_description/urdf/all_components_with_moveit.urdf (robot description, URDF)
Before this commit: robot rostms, 93 links, 92 joints
Links:
- link refrigerator_link: geometry visual mesh filename=package://environmental_model/model/refrigerator.dae

File: tms_rp/rostms_description/urdf/environments.urdf.xacro (robot description, xacro)
@@ -303,10 +303,10 @@
         </geometry>
       </visual>
-      <collision>
+      <!-- <collision>
         <geometry>
           <box size="0.5 0.47 0.05"/>
         </geometry>
         <origin xyz="-0.32 0.235 1.09" rpy="0 0 0"/>
-      </collision>
+      </collision> -->
     </link>
     <joint name="refrigerator_door_joint" type="continuous">

Commit message: add tms_ur_listener

File: tms_rp/rostms_description/urdf/all_components_with_moveit.urdf (robot description, URDF)
Before this commit: robot rostms, 93 links, 92 joints
Links:
- link refrigerator_link: geometry collision box size=0.5 0.47 0.05; visual mesh filename=package://environmental_model/model/refrigerator.dae

File: tms_rp/rostms_description/urdf/environments.urdf.xacro (robot description, xacro)
@@ -303,10 +303,10 @@
         </geometry>
       </visual>
-      <!-- <collision>
+      <collision>
         <geometry>
           <box size="0.5 0.47 0.05"/>
         </geometry>
         <origin xyz="-0.32 0.235 1.09" rpy="0 0 0"/>
-      </collision> -->
+      </collision>
     </link>
     <joint name="refrigerator_door_joint" type="continuous">
