Commit message: tms_ss_kinect_v2: add skeleton_state_publisher

File: tms_ss/tms_ss_kinect_v2/urdf/skeleton.urdf (robot description, URDF)
Before this commit: robot Human, 15 links, 14 joints
Links:
- removed link base_link
- added link Body; visual mesh filename=package://tms_ss_kinect_v2/model/male/Body.dae
- added link LeftElbowVirtual
- added link LeftHipVirtual1
- added link LeftHipVirtual2
- added link LeftKneeVirtual
- added link LeftShoulderVirtual1
- added link LeftShoulderVirtual2
- added link LeftWristVirtual
- added link NeckVirtual
- added link RightElbowVirtual
- added link RightHipVirtual1
- added link RightHipVirtual2
- added link RightKneeVirtual
- added link RightShoulderVirtual1
- added link RightShoulderVirtual2
- added link RightWristVirtual
Joints:
- removed joint AnkleLeft
- removed joint AnkleRight
- removed joint CervicalSpine
- removed joint ElbowLeft
- removed joint ElbowRight
- removed joint HipLeft
- removed joint HipRight
- removed joint KneeLeft
- removed joint KneeRight
- removed joint ShoulderLeft
- removed joint ShoulderRight
- removed joint SpineShoulder
- removed joint WristLeft
- removed joint WristRight
- added joint L_ARM_JOINT1: type continuous, parent Body, child LeftShoulderVirtual1
- added joint L_ARM_JOINT2: type continuous, parent LeftShoulderVirtual1, child LeftShoulderVirtual2
- added joint L_ARM_JOINT3: type continuous, parent LeftShoulderVirtual2, child LeftArm1
- added joint L_ARM_JOINT4: type continuous, parent LeftArm1, child LeftElbowVirtual
- added joint L_ARM_JOINT5: type continuous, parent LeftElbowVirtual, child LeftArm2
- added joint L_ARM_JOINT6: type continuous, parent LeftArm2, child LeftWristVirtual
- added joint L_ARM_JOINT7: type continuous, parent LeftWristVirtual, child LeftHand1
- added joint L_LEG_JOINT1: type continuous, parent Body, child LeftHipVirtual1
- added joint L_LEG_JOINT2: type continuous, parent LeftHipVirtual1, child LeftHipVirtual2
- added joint L_LEG_JOINT3: type continuous, parent LeftHipVirtual2, child LeftLeg1
- added joint L_LEG_JOINT4: type continuous, parent LeftLeg1, child LeftKneeVirtual
- added joint L_LEG_JOINT5: type continuous, parent LeftKneeVirtual, child LeftLeg2
- added joint L_LEG_JOINT6: type continuous, parent LeftLeg2, child LeftFoot
- added joint NECK_JOINT0: type continuous, parent Body, child Neck
- added joint NECK_JOINT1: type continuous, parent Neck, child NeckVirtual
- added joint NECK_JOINT2: type continuous, parent NeckVirtual, child Head
- added joint R_ARM_JOINT1: type continuous, parent Body, child RightShoulderVirtual1
- added joint R_ARM_JOINT2: type continuous, parent RightShoulderVirtual1, child RightShoulderVirtual2
- added joint R_ARM_JOINT3: type continuous, parent RightShoulderVirtual2, child RightArm1
- added joint R_ARM_JOINT4: type continuous, parent RightArm1, child RightElbowVirtual
- added joint R_ARM_JOINT5: type continuous, parent RightElbowVirtual, child RightArm2
- added joint R_ARM_JOINT6: type continuous, parent RightArm2, child RightWristVirtual
- added joint R_ARM_JOINT7: type continuous, parent RightWristVirtual, child RightHand1
- added joint R_LEG_JOINT1: type continuous, parent Body, child RightHipVirtual1
- added joint R_LEG_JOINT2: type continuous, parent RightHipVirtual1, child RightHipVirtual2
- added joint R_LEG_JOINT3: type continuous, parent RightHipVirtual2, child RightLeg1
- added joint R_LEG_JOINT4: type continuous, parent RightLeg1, child RightKneeVirtual
- added joint R_LEG_JOINT5: type continuous, parent RightKneeVirtual, child RightLeg2
- added joint R_LEG_JOINT6: type continuous, parent RightLeg2, child RightFoot

Commit message: tms_ss_kinect_v2: create movable human model

File: tms_ss/tms_ss_kinect_v2/urdf/skeleton.urdf (robot description, URDF)
Before this commit: robot Human, 30 links, 29 joints
Joints:
- joint L_ARM_JOINT1: origin (none) -> xyz=-0.185 0 1.39 rpy=0 0 0
- joint L_ARM_JOINT4: origin (none) -> xyz=-0.215 0 0 rpy=0 0 0
- joint L_ARM_JOINT6: origin (none) -> xyz=-0.22 0 0 rpy=0 0 0
- joint L_LEG_JOINT1: origin (none) -> xyz=-0.072 0 0.85 rpy=0 0 0
- joint L_LEG_JOINT4: origin (none) -> xyz=0.0 0 -0.3 rpy=0 0 0
- joint L_LEG_JOINT6: origin (none) -> xyz=0.0 0 -0.42 rpy=0 0 0
- joint NECK_JOINT0: origin (none) -> xyz=0 0 1.45 rpy=0 0 0
- joint NECK_JOINT1: origin (none) -> xyz=0 0.04 0.03 rpy=0 0 0
- joint R_ARM_JOINT1: origin (none) -> xyz=0.185 0 1.39 rpy=0 0 0
- joint R_ARM_JOINT4: origin (none) -> xyz=0.215 0 0 rpy=0 0 0
- joint R_ARM_JOINT6: origin (none) -> xyz=0.22 0 0 rpy=0 0 0
- joint R_LEG_JOINT1: origin (none) -> xyz=0.072 0 0.85 rpy=0 0 0
- joint R_LEG_JOINT4: origin (none) -> xyz=0.0 0 -0.3 rpy=0 0 0
- joint R_LEG_JOINT6: origin (none) -> xyz=0.0 0 -0.42 rpy=0 0 0

Commit message: tms_ss_kinect_v2: set joint coordinate and modify to view multiple skeletons

File: tms_ss/tms_ss_kinect_v2/urdf/skeleton.urdf (robot description, URDF)
Before this commit: robot Human, 30 links, 29 joints
Joints:
- joint L_ARM_JOINT1: axis (none) -> -1.0 0.0 0.0; origin xyz=-0.185 0 1.39 rpy=0 0 0 -> xyz=-0.185 0 0.29 rpy=0.0 0.0 0.0
- joint L_ARM_JOINT2: axis (none) -> 0.0 1.0 0.0; origin (none) -> xyz=0.0 0.0 0.0 rpy=0 4.71238898038 0
- joint L_ARM_JOINT3: axis (none) -> 1.0 0.0 0.0
- joint L_ARM_JOINT4: axis (none) -> 0.0 0.0 1.0; origin xyz=-0.215 0 0 rpy=0 0 0 -> xyz=-0.215 0 0 rpy=0 0 0.0
- joint L_LEG_JOINT1: axis (none) -> -1.0 0.0 0.0; origin xyz=-0.072 0 0.85 rpy=0 0 0 -> xyz=-0.072 0 -0.25 rpy=0 0 0
- joint L_LEG_JOINT2: axis (none) -> 0.0 1.0 0.0
- joint L_LEG_JOINT3: axis (none) -> 0.0 0.0 1.0
- joint L_LEG_JOINT4: axis (none) -> 0.0 0.0 -1.0
- joint NECK_JOINT0: origin xyz=0 0 1.45 rpy=0 0 0 -> xyz=0 0 0.35 rpy=0 0 0
- joint R_ARM_JOINT1: axis (none) -> -1.0 0.0 0.0; origin xyz=0.185 0 1.39 rpy=0 0 0 -> xyz=0.185 0 0.29 rpy=0 0 0
- joint R_ARM_JOINT2: axis (none) -> 0.0 1.0 0.0; origin (none) -> xyz=0.0 0.0 0.0 rpy=0 1.57079632679 0
- joint R_ARM_JOINT3: axis (none) -> -1.0 0.0 0.0
- joint R_ARM_JOINT4: axis (none) -> 0.0 0.0 -1.0; origin xyz=0.215 0 0 rpy=0 0 0 -> xyz=0.215 0 0 rpy=0 0 0.0
- joint R_LEG_JOINT1: axis (none) -> -1.0 0.0 0.0; origin xyz=0.072 0 0.85 rpy=0 0 0 -> xyz=0.072 0 -0.25 rpy=0 0 0
- joint R_LEG_JOINT2: axis (none) -> 0.0 1.0 0.0
- joint R_LEG_JOINT3: axis (none) -> 0.0 0.0 1.0
- joint R_LEG_JOINT4: axis (none) -> -1.0 0.0 0.0

Commit message: tms_ss_kinect_v2: can show multiple skeletons in rViz

File: tms_ss/tms_ss_kinect_v2/urdf/skeleton.urdf (robot description, URDF)
Before this commit: robot Human, 30 links, 29 joints
Joints:
- joint L_LEG_JOINT4: axis 0.0 0.0 -1.0 -> -1.0 0.0 0.0
