Commit message: added stand-alone mode of smartpal in gazebo

File: tms_rp/smartpal5_gazebo/urdf/smartpal_gazebo.urdf.xacro (robot description, xacro)
@@ -61,5 +61,5 @@
   </link>
   <!-- Lumbar -->
-  <joint name="lumbar_lower_joint" type="revolute">
+  <joint name="lumbar_lower_joint" type="fixed">
     <parent link="base_link"/>
   	<child link="lumbar_lower_link"/>
@@ -88,5 +88,5 @@
   	</inertial>
   </link>
-  <joint name="lumbar_upper_joint" type="revolute">
+  <joint name="lumbar_upper_joint" type="fixed">
   	<parent link="lumbar_lower_link"/>
   	<child link="lumbar_upper_link"/>
