Commit message: tms_ss_kinect_v2: devide package

File: tms_rp/skeleton_description/urdf/checker_box.urdf (robot description, URDF)
Before this commit: robot Kinect_v2, 1 links, 0 joints
Links:
- removed link base_link
- added link Box; visual mesh filename=package://skeleton_description/model/checker_box/checker_bo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

File: tms_rp/skeleton_description/urdf/kinect_v2.urdf (robot description, URDF)
Before this commit: robot CheckerBox, 1 links, 0 joints
Links:
- removed link Box
- added link base_link; visual mesh filename=package://skeleton_description/model/kinect_v2/kinect_v2.dae

File: tms_rp/skeleton_description/urdf/skeleton.urdf (robot description, URDF)
Before this commit: robot Human, 30 links, 29 joints
Links:
- link Body: geometry visual mesh filename=package://skeleton_description/model/male/Body.dae
- link Head: geometry visual mesh filename=package://skeleton_description/model/male/Head.dae
- link LeftArm1: geometry visual mesh filename=package://skeleton_description/model/male/LeftArm1.dae
- link LeftArm2: geometry visual mesh filename=package://skeleton_description/model/male/LeftArm2.dae
- link LeftFoot: geometry visual mesh filename=package://skeleton_description/model/male/LeftFoot.dae
- link LeftHand1: geometry visual mesh filename=package://skeleton_description/model/male/LeftHand1.dae
- link LeftLeg1: geometry visual mesh filename=package://skeleton_description/model/male/LeftLeg1.dae
- link LeftLeg2: geometry visual mesh filename=package://skeleton_description/model/male/LeftLeg2.dae
- link Neck: geometry visual mesh filename=package://skeleton_description/model/male/Neck.dae
- link RightArm1: geometry visual mesh filename=package://skeleton_description/model/male/RightArm1.dae
- link RightArm2: geometry visual mesh filename=package://skeleton_description/model/male/RightArm2.dae
- link RightFoot: geometry visual mesh filename=package://skeleton_description/model/male/RightFoot.dae
- link RightHand1: geometry visual mesh filename=package://skeleton_description/model/male/RightHand1.dae
- link RightLeg1: geometry visual mesh filename=package://skeleton_description/model/male/RightLeg1.dae
- link RightLeg2: geometry visual mesh filename=package://skeleton_description/model/male/RightLeg2.dae
