Commit message: Pump changes 1

File: tms_rp/skeleton_description/urdf/skeleton/model_002.urdf (robot description, URDF)
Before this commit: robot Human, 30 links, 29 joints
Joints:
- joint L_ARM_JOINT1: axis -1.0 0.0 0.0 -> 0.0 0.0 1.0
- joint L_ARM_JOINT2: origin xyz=-0.0 0.0 0.0 rpy=0 4.71238898038 0 -> (none)
- joint L_ARM_JOINT4: origin xyz=-0 0 -0.215 rpy=0 -1.57079632679 0.0 -> xyz=-0.215 0 0 rpy=0 0 0

Commit message: for checking calculation: 1

File: tms_rp/skeleton_description/urdf/skeleton/model_002.urdf (robot description, URDF)
Before this commit: robot Human, 30 links, 29 joints
Joints:
- joint L_ARM_JOINT2: origin xyz=-0.0 0.0 0.0 rpy=0 4.71238898038 0 -> xyz=-0.0 0.0 0.0 rpy=0 0 0
- joint L_ARM_JOINT4: origin xyz=-0 0 -0.215 rpy=0 -1.57079632679 0.0 -> xyz=0.215 0 0 rpy=0 0 0
- joint L_ARM_JOINT6: origin xyz=-0.22 0 0.0 rpy=0 0 0 -> xyz=0.22 0 0.0 rpy=0 0 0

Commit message: calc_joint_angles: calculate about left arm

File: tms_rp/skeleton_description/urdf/skeleton/model_002.urdf (robot description, URDF)
Before this commit: robot Human, 30 links, 29 joints
Joints:
- joint L_ARM_JOINT2: origin xyz=-0.0 0.0 0.0 rpy=0 0 0 -> (none)

Commit message: skeleton_description: fix some minor error

File: tms_rp/skeleton_description/urdf/skeleton/model_002.urdf (robot description, URDF)
Before this commit: robot Human, 30 links, 29 joints
Joints:
- joint L_LEG_JOINT1: axis -1.0 0.0 0.0 -> 0.0 0.0 1.0
- joint L_LEG_JOINT3: axis 0.0 0.0 1.0 -> 1.0 0.0 0.0
- joint L_LEG_JOINT4: axis -1.0 0.0 0.0 -> 0.0 0.0 1.0
- joint R_ARM_JOINT1: axis -1.0 0.0 0.0 -> 0.0 0.0 1.0
- joint R_ARM_JOINT3: axis -1.0 0.0 0.0 -> 1.0 0.0 0.0
- joint R_ARM_JOINT4: axis 0.0 0.0 -1.0 -> 0.0 0.0 1.0
- joint R_LEG_JOINT1: axis -1.0 0.0 0.0 -> 0.0 0.0 1.0
- joint R_LEG_JOINT3: axis 0.0 0.0 1.0 -> 1.0 0.0 0.0
- joint R_LEG_JOINT4: axis -1.0 0.0 0.0 -> 0.0 0.0 1.0

Commit message: skeleton_description: fixed calculation

File: tms_rp/skeleton_description/urdf/skeleton/model_002.urdf (robot description, URDF)
Before this commit: robot Human, 30 links, 29 joints
Joints:
- joint R_ARM_JOINT2: origin xyz=-0.0 0.0 0.0 rpy=0 1.57079632679 0 -> xyz=-0.0 0.0 0.0 rpy=0 0 0
- joint R_ARM_JOINT4: origin xyz=0 0 0.215 rpy=0 -1.57079632679 0.0 -> xyz=0.215 0 0 rpy=0 0 0
