Commit message: [fix] add wheelchair 3D data

File: tms_rc/tms_rc_mimamorukun/mimamorukun_control/urdf/wheelchair.urdf.xacro (robot description, xacro)
@@ -26,5 +26,5 @@
   <visual>
     <geometry>
-      <mesh filename="package://environmental_model/model/refrigerator.dae"/>
+      <mesh filename="package://environmental_model/model/wheelchair.dae"/>
     </geometry>
     <origin xyz="0.0 0.0 0.56" rpy="0 0 0"/>
